File: pcb_main/rev.A/zxevo1010_main.kicad_pcb (KiCad board)
At the start: 2 copper layers, 100 x 100 mm, 209 parts, among them J1 Mini-DIN-6, J10 TE 041021-4, J13 Conn_02x05_Odd_Even, J16 MEM2055-00-190-01-A, J17 B2B-XH-A, J2 USB_B_Micro, J22 Conn_02x05_Odd_Even, J3 Mini-DIN-6, J4 PJ-320, J5 Conn_02x05_Odd_Even, J6 Conn_02x30_Row_Letter_First, J8 Conn_02x05_Odd_Even, J9 DB15_Female_HighDensity_Mount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, Q1 BC856, Q2 BC856, Q3 BC847, Q6 BC847, SW3 SW_Push, SW5 SW_Push, SW6 SW_Push, U1 39SF040, U10 GM71C(S)18163CT, U11 CH340X, U12 LMV358IDR, U13 PCF8583T, U14 LP2985-3.3, U15 74LVC1G04DB, U16 74LVC1G04DB, U17 74LVC1G04DB, U18 74LVC1G04DB, U19 CD4069UBM, U2 EP1K50QC208, U20 74LVC1G04DB, U21 EPM3128ATC100, U22 LP2985-3.3, U23 ADV7125-lqfp48, U24 FT812, U3 Z80CPU_QFP, U4 74HCT245PW, U5 ICS501, U6 ATmega128, U7 GM71C(S)18163CT, U8 1117-3.3, U9 1117-2.5, Y1 14 MHz, Y2 11.059 Mhz, Y3 32768 Hz, Y4 8 MHz

Commit message: wip pcbs rev.A
Parts:
- removed JP2: SolderJumper_2_Open, Jumper:SolderJumper-2_P1.3mm_Open_RoundedPad1.0x1.5mm
- removed Q3: BC847, Package_TO_SOT_SMD:SOT-23
- removed R19: 1k, Resistor_SMD:R_0603_1608Metric_Pad0.98x0.95mm_HandSolder
- removed R20, R42, R43: 75, Resistor_SMD:R_0603_1608Metric_Pad0.98x0.95mm_HandSolder
- removed R65, R66: 47k, Resistor_SMD:R_0603_1608Metric_Pad0.98x0.95mm_HandSolder
- removed R67, R95: 10k, Resistor_SMD:R_0603_1608Metric_Pad0.98x0.95mm_HandSolder
- removed U4: 74HCT245PW, Package_SO:TSSOP-20_4.4x6.5mm_P0.65mm
- added C42: 18p, Capacitor_SMD:C_0603_1608Metric_Pad1.08x0.95mm_HandSolder, B.Cu at (128.6, 33.9)
- added C43: 10u, Capacitor_Tantalum_SMD:CP_EIA-3216-18_Kemet-A_Pad1.58x1.35mm_HandSolder, B.Cu at (126.7, 33.9)
- added R6: 120, Resistor_SMD:R_0603_1608Metric_Pad0.98x0.95mm_HandSolder, B.Cu at (156.2, 56.6)
- C24, C27: value 10u -> 18p; footprint Capacitor_Tantalum_SMD:CP_EIA-3216-18_Kemet-A_Pad1.58x1.35mm_HandSolder -> Capacitor_SMD:C_0603_1608Metric_Pad1.08x0.95mm_HandSolder
- C26, C30, C32, C35, C50, C53, C74, U10: moved to B.Cu
- R15: value 240 -> 1k
- R16, R7: value 430 -> 1k
- R17: value 240 -> 24k
- R18: value 430 -> 24k
- R2: value 240 -> 120
- R21, R22, R23: value 100 -> 75
- R24: value 10k -> 1k
- moved Y4 47.7 mm to (167.7, 67.8)
- moved C38 47.7 mm to (167.7, 66.4)
- moved C37 47.7 mm to (167.7, 69.3)
- moved C36 47.2 mm to (157.8, 73.7)
- moved R1 47.2 mm to (156.2, 73.7)
- moved U21 47.2 mm to (144.7, 70.1)
- moved U23 47.2 mm to (160.4, 77.7), turned to 0 degrees
- moved R5 45.9 mm to (161.8, 69.1)
- moved C34 45.9 mm to (164.3, 66.9)
- moved C33 45.9 mm to (164.3, 63.5)
- moved U24 45.9 mm to (160.4, 64.7)
- moved C17 45.2 mm to (165.5, 103.3)
- moved U11 45.2 mm to (164.4, 102.1)
- moved C53 42.1 mm to (175.8, 27.5)
- moved C27 42.1 mm to (131.6, 33.9), turned to -90 degrees
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Connections:
- C24 pad 1: /TOP_IN_L -> Net-(C24-Pad1)
- C24 pad 2: Net-(C24-Pad2) -> GND
- C27 pad 1: /TOP_IN_R -> Net-(C27-Pad1)
- C27 pad 2: Net-(C27-Pad2) -> GND
- J13 pad 3: /TDO_FPGA -> /TDO_CPLD
- J8 pad 2: /TOP_IN_L -> /MIXER_L
- J8 pad 8: /TOP_IN_R -> /MIXER_R
- J9 pad 1: /VGA_R -> /V_R
- J9 pad 13: /VGA_HS -> /V_HS_OUT
- J9 pad 14: /VGA_VS -> /V_VS_OUT
- J9 pad 15: Net-(JP2-A) -> unconnected-(J9-Pad15)
- J9 pad 2: /VGA_G -> /V_G
- J9 pad 3: /VGA_B -> /V_B
- R15 pad 1: /VR+ -> Net-(C27-Pad1)
- R15 pad 2: /VGA_R -> Net-(C24-Pad1)
- R16 pad 1: /VR- -> /FT_AU_L
- R16 pad 2: /VGA_R -> Net-(C27-Pad1)
- R17 pad 1: /VB+ -> /MIXER_L
- R17 pad 2: /VGA_B -> Net-(C43-Pad2)
- R18 pad 1: /VB- -> /MIXER_R
- R18 pad 2: /VGA_B -> Net-(C43-Pad2)
- R2 pad 1: /VG+ -> /V_VS_OUT
- R2 pad 2: /VGA_G -> /V_VS
- R21 pad 2: /VGA_B -> /V_B
- R22 pad 2: /VGA_G -> /V_G
- R23 pad 2: /VGA_R -> /V_R
- R49 pad 2: Net-(U12A--) -> /MIXER_L
- R50 pad 2: Net-(U12B--) -> /MIXER_R
- R55 pad 1: Net-(U12A--) -> /MIXER_L
- R58 pad 1: Net-(U12B--) -> /MIXER_R
- R7 pad 1: /VG- -> Net-(C24-Pad1)
- R7 pad 2: /VGA_G -> Net-(U24-AUDIO_L)
- U12 pad 2: Net-(U12A--) -> /MIXER_L
- U12 pad 6: Net-(U12B--) -> /MIXER_R
- U2 pad 100: unconnected-(U2-IO_100-Pad100) -> /M_SEL
- U2 pad 101: unconnected-(U2-IO_101-Pad101) -> /~{FT_CS}
- U2 pad 103: unconnected-(U2-IO_103-Pad103) -> /FT_MOSI
- U2 pad 104: unconnected-(U2-IO_104-Pad104) -> /FT_SCK
- U2 pad 111: unconnected-(U2-IO_111-Pad111) -> /O_CLK
- U2 pad 112: unconnected-(U2-IO_112-Pad112) -> /O_VS
- U2 pad 113: unconnected-(U2-IO_113-Pad113) -> /O_HS
- U2 pad 120: /VVSYNC -> unconnected-(U2-IO_120-Pad120)
- U2 pad 121: /VHSYNC -> unconnected-(U2-IO_121-Pad121)
- U2 pad 122: /VCSYNC -> unconnected-(U2-IO_122-Pad122)
- U2 pad 125: /V_B- -> unconnected-(U2-IO_125-Pad125)
- U2 pad 126: /V_B+ -> unconnected-(U2-IO_126-Pad126)
- U2 pad 127: /V_G- -> unconnected-(U2-IO_127-Pad127)
- U2 pad 128: /V_G+ -> unconnected-(U2-IO_128-Pad128)
- U2 pad 131: /V_R- -> unconnected-(U2-IO_131-Pad131)
- U2 pad 132: /V_R+ -> unconnected-(U2-IO_132-Pad132)
- U2 pad 71: unconnected-(U2-IO_71-Pad71) -> /O_G3
- U2 pad 73: unconnected-(U2-IO_73-Pad73) -> /O_G1
- U2 pad 74: unconnected-(U2-IO_74-Pad74) -> /O_G4
- U2 pad 75: unconnected-(U2-IO_75-Pad75) -> /O_G0
- U2 pad 83: unconnected-(U2-IO_83-Pad83) -> /O_B0
- U2 pad 85: unconnected-(U2-IO_85-Pad85) -> /O_R4
- U2 pad 86: unconnected-(U2-IO_86-Pad86) -> /O_B1
- U2 pad 87: unconnected-(U2-IO_87-Pad87) -> /O_R3
- U2 pad 88: unconnected-(U2-IO_88-Pad88) -> /O_B2
- U2 pad 89: unconnected-(U2-IO_89-Pad89) -> /O_R2
- U2 pad 90: unconnected-(U2-IO_90-Pad90) -> /O_B3
- U2 pad 92: unconnected-(U2-IO_92-Pad92) -> /O_R1
- U2 pad 93: unconnected-(U2-IO_93-Pad93) -> /O_B4
- U2 pad 94: unconnected-(U2-IO_94-Pad94) -> /O_R0
- U2 pad 95: unconnected-(U2-IO_95-Pad95) -> /PAL_SEL
- U2 pad 96: unconnected-(U2-IO_96-Pad96) -> /O_G2
- U2 pad 99: unconnected-(U2-IO_99-Pad99) -> /FT_MISO
- U21 pad 15: unconnected-(U21-TMS-Pad15) -> /TMS_FPGA
- U21 pad 4: unconnected-(U21-TDI-Pad4) -> /TDO_FPGA
- U21 pad 49: unconnected-(U21-I/O-Pad49) -> /V_HS
- U21 pad 50: unconnected-(U21-I/O-Pad50) -> /V_VS
- U21 pad 62: unconnected-(U21-TCK-Pad62) -> /TCK_FPGA
- U21 pad 73: unconnected-(U21-TDO-Pad73) -> /TDO_CPLD
- U23 pad 28: unconnected-(U23-IOB-Pad28) -> /V_B
- U23 pad 32: unconnected-(U23-IOG-Pad32) -> /V_G
- U23 pad 34: unconnected-(U23-IOR-Pad34) -> /V_R
- U24 pad 3: /FT_AU_L -> Net-(U24-AUDIO_L)
- Y1 pad 1: Net-(U5-X1) -> Net-(U5-X2)
- Y1 pad 2: Net-(U5-X2) -> Net-(U5-X1)
Routing:
- net /ADV_CLK: track 0.00 -> 29.6 mm
- net /ADV_B7: track 0.00 -> 27.9 mm
- net /FT_VS: track 0.00 -> 27.8 mm
- net /ADV_B6: track 0.00 -> 26.6 mm
- net /FT_HS: track 0.00 -> 26.5 mm
- net /ADV_B5: track 0.00 -> 25.3 mm
- net /FT_CLK: track 0.00 -> 24.8 mm
- net /ADV_B4: track 0.00 -> 24.0 mm
- net /ADV_B3: track 0.00 -> 22.7 mm
- net /FT_B6: track 0.00 -> 22.0 mm
- net /ADV_B2: track 0.00 -> 20.9 mm
- net /FT_B5: track 0.00 -> 20.7 mm
- net /ADV_B1: track 0.00 -> 19.6 mm
- net /FT_B4: track 0.00 -> 18.9 mm
- net /ADV_B0: track 0.00 -> 17.8 mm
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
Commit message: wip pcbs rev.A
Parts:
- removed R35: 680, Resistor_SMD:R_0603_1608Metric_Pad0.98x0.95mm_HandSolder
- added C44: 100n, Capacitor_SMD:C_0603_1608Metric_Pad1.08x0.95mm_HandSolder, B.Cu at (135.2, 102.7)
- added C45: 100n, Capacitor_SMD:C_0603_1608Metric_Pad1.08x0.95mm_HandSolder, B.Cu at (130.3, 112.6)
- added C46: 100n, Capacitor_SMD:C_0603_1608Metric_Pad1.08x0.95mm_HandSolder, B.Cu at (120.3, 112.6)
- added C47: 100n, Capacitor_SMD:C_0603_1608Metric_Pad1.08x0.95mm_HandSolder, B.Cu at (115.2, 87.8)
- added C48: 100n, Capacitor_SMD:C_0603_1608Metric_Pad1.08x0.95mm_HandSolder, B.Cu at (110.4, 97.7)
- added C49: 100n, Capacitor_SMD:C_0603_1608Metric_Pad1.08x0.95mm_HandSolder, B.Cu at (135.2, 97.7)
- added C51: 100n, Capacitor_SMD:C_0603_1608Metric_Pad1.08x0.95mm_HandSolder, B.Cu at (125.3, 112.6)
- added C52: 100n, Capacitor_SMD:C_0603_1608Metric_Pad1.08x0.95mm_HandSolder, B.Cu at (118.0, 65.4)
- added C54: 100n, Capacitor_SMD:C_0603_1608Metric_Pad1.08x0.95mm_HandSolder, B.Cu at (130.3, 87.8)
- added C55: 100n, Capacitor_SMD:C_0603_1608Metric_Pad1.08x0.95mm_HandSolder, B.Cu at (110.4, 92.7)
- added C56: 100n, Capacitor_SMD:C_0603_1608Metric_Pad1.08x0.95mm_HandSolder, B.Cu at (110.4, 102.7)
- added C57: 100n, Capacitor_SMD:C_0603_1608Metric_Pad1.08x0.95mm_HandSolder, B.Cu at (115.3, 112.6)
- added C58: 100n, Capacitor_SMD:C_0603_1608Metric_Pad1.08x0.95mm_HandSolder, B.Cu at (102.0, 107.2)
- added C59: 100n, Capacitor_SMD:C_0603_1608Metric_Pad1.08x0.95mm_HandSolder, B.Cu at (189.7, 121.5)
- added C60: 100n, Capacitor_SMD:C_0603_1608Metric_Pad1.08x0.95mm_HandSolder, B.Cu at (178.6, 108.6)
- added C61: 100n, Capacitor_SMD:C_0603_1608Metric_Pad1.08x0.95mm_HandSolder, B.Cu at (110.4, 107.7)
- added C62: 100n, Capacitor_SMD:C_0603_1608Metric_Pad1.08x0.95mm_HandSolder, B.Cu at (177.3, 97.6)
- added C63: 100n, Capacitor_SMD:C_0603_1608Metric_Pad1.08x0.95mm_HandSolder, B.Cu at (158.9, 110.4)
- added C64: 100n, Capacitor_SMD:C_0603_1608Metric_Pad1.08x0.95mm_HandSolder, B.Cu at (144.7, 114.1)
- added C65: 100n, Capacitor_SMD:C_0603_1608Metric_Pad1.08x0.95mm_HandSolder, B.Cu at (147.1, 93.2)
- added C66: 100n, Capacitor_SMD:C_0603_1608Metric_Pad1.08x0.95mm_HandSolder, B.Cu at (152.0, 93.2)
- added C67: 100n, Capacitor_SMD:C_0603_1608Metric_Pad1.08x0.95mm_HandSolder, B.Cu at (156.9, 93.2)
- added C69: 100n, Capacitor_SMD:C_0603_1608Metric_Pad1.08x0.95mm_HandSolder, B.Cu at (163.9, 103.3)
- added C70: 100n, Capacitor_SMD:C_0603_1608Metric_Pad1.08x0.95mm_HandSolder, B.Cu at (129.4, 116.8)
- added C71: 100n, Capacitor_SMD:C_0603_1608Metric_Pad1.08x0.95mm_HandSolder, B.Cu at (132.7, 121.5)
- added C72: 100n, Capacitor_SMD:C_0603_1608Metric_Pad1.08x0.95mm_HandSolder, B.Cu at (111.1, 120.6)
- added C73: 100n, Capacitor_SMD:C_0603_1608Metric_Pad1.08x0.95mm_HandSolder, B.Cu at (130.6, 136.6)
- added C75: 100n, Capacitor_SMD:C_0603_1608Metric_Pad1.08x0.95mm_HandSolder, B.Cu at (126.6, 136.6)
- added C76: 100n, Capacitor_SMD:C_0603_1608Metric_Pad1.08x0.95mm_HandSolder, B.Cu at (113.2, 136.6)
- added C77: 100n, Capacitor_SMD:C_0603_1608Metric_Pad1.08x0.95mm_HandSolder, B.Cu at (144.7, 64.1)
- added C78: 100n, Capacitor_SMD:C_0603_1608Metric_Pad1.08x0.95mm_HandSolder, B.Cu at (150.7, 70.1)
- added C79: 100n, Capacitor_SMD:C_0603_1608Metric_Pad1.08x0.95mm_HandSolder, B.Cu at (138.7, 70.1)
- added C80: 100n, Capacitor_SMD:C_0603_1608Metric_Pad1.08x0.95mm_HandSolder, B.Cu at (144.7, 76.1)
- added C81: 100n, Capacitor_SMD:C_0603_1608Metric_Pad1.08x0.95mm_HandSolder, B.Cu at (161.9, 66.3)
- added C82: 1u, Capacitor_SMD:C_0603_1608Metric_Pad1.08x0.95mm_HandSolder, B.Cu at (160.4, 66.3)
- added C83: 1u, Capacitor_SMD:C_0603_1608Metric_Pad1.08x0.95mm_HandSolder, B.Cu at (161.4, 79.9)
- added C85: 100n, Capacitor_SMD:C_0603_1608Metric_Pad1.08x0.95mm_HandSolder, B.Cu at (161.4, 78.4)
- added C87: 100n, Capacitor_SMD:C_0603_1608Metric_Pad1.08x0.95mm_HandSolder, B.Cu at (157.8, 79.9)
- added C88: 10u, Capacitor_SMD:C_0805_2012Metric_Pad1.18x1.45mm_HandSolder, B.Cu at (127.0, 59.0)
- added F1: 0.2A, Fuse:Fuse_1812_4532Metric_Pad1.30x3.40mm_HandSolder, B.Cu at (109.0, 142.4)
- added Q3: BC856, Package_TO_SOT_SMD:SOT-23, B.Cu at (120.7, 144.5)
- added R43: 10k, Resistor_SMD:R_0603_1608Metric_Pad0.98x0.95mm_HandSolder, B.Cu at (130.7, 84.5)
- C14, C15, R12, R13, R8, R9: moved to B.Cu
- C35, C50: value 1u -> 100n
- LOGO1: footprint mygraphic:black-mage-6.7x9.5 -> mygraphic:black-mage-12.5x8.6-r
- U1: value 39SF040 -> 29F040-K
- U10: value GM71C(S)18163CT -> HY5118160; moved to F.Cu
- U3: value Z80CPU_QFP -> Z84C0020FEC
- U7: value GM71C(S)18163CT -> HY5118160; moved to B.Cu
- moved C50 91.0 mm to (135.2, 107.7), turned to 0 degrees
- moved C30 90.5 mm to (106.8, 71.6), turned to 0 degrees
- moved C32 83.7 mm to (125.3, 87.8)
- moved LOGO1 83.5 mm to (122.8, 100.2)
- moved C53 82.0 mm to (120.2, 87.8), turned to 90 degrees
- moved C35 79.5 mm to (135.2, 92.7), turned to 0 degrees
- moved Q1 13.3 mm to (116.5, 144.5)
- moved Q2 13.3 mm to (129.8, 144.5)
- moved R3 13.3 mm to (113.5, 144.5)
- moved R4 13.3 mm to (126.8, 144.5)
- moved D6 13.2 mm to (114.3, 141.8)
- moved D7 13.2 mm to (127.6, 141.8)
- moved U13 11.7 mm to (169.8, 128.3), turned to 180 degrees
- moved R75 11.4 mm to (105.3, 77.9)
- moved R5 9.59 mm to (152.3, 70.1), turned to 90 degrees
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Connections:
- C11 pad 1: GNDA -> GND
- C19 pad 2: GNDA -> GND
- C28 pad 1: GNDA -> GND
- C29 pad 2: GNDA -> GND
- C31 pad 2: GNDA -> GND
- C32 pad 1: GND -> +2V5
- C32 pad 2: +2V5 -> GND
- C35 pad 1: GND -> +2V5
- C35 pad 2: +2V5 -> GND
- C5 pad 1: GNDA -> GND
- C50 pad 1: GND -> +3V3
- C50 pad 2: +3V3 -> GND
- C53 pad 1: GND -> +3V3
- C53 pad 2: +3V3 -> GND
- C6 pad 1: GNDA -> GND
- C7 pad 1: GNDA -> GND
- J4 pad R2: GNDA -> GND
- J4 pad S: GNDA -> GND
- J8 pad 3: GNDA -> GND
- J8 pad 4: GNDA -> GND
- J8 pad 5: GNDA -> GND
- J8 pad 6: GNDA -> GND
- J9 pad 0: GNDA -> GND
- J9 pad 10: GNDA -> GND
- J9 pad 5: GNDA -> GND
- J9 pad 6: GNDA -> GND
- J9 pad 7: GNDA -> GND
- J9 pad 8: GNDA -> GND
- L2 pad 1: +3V3_2 -> +3V3
- R1 pad 1: GNDA -> GND
- R11 pad 1: GNDA -> GND
- R21 pad 1: GNDA -> GND
- R22 pad 1: GNDA -> GND
- R23 pad 1: GNDA -> GND
- R27 pad 1: +5V_FUSE -> +5V_JOYSTICK
- R28 pad 1: +3V3_2 -> +3V3
- R29 pad 1: +5V_FUSE -> +5V_JOYSTICK
- R30 pad 1: +5V_FUSE -> +5V_JOYSTICK
- R31 pad 1: +3V3_2 -> +3V3
- R32 pad 1: +3V3_2 -> +3V3
- R36 pad 1: +5V_FUSE -> +5V_JOYSTICK
- R38 pad 1: +5V_FUSE -> +5V_JOYSTICK
- R46 pad 1: +5V_FUSE -> +5V_JOYSTICK
- R47 pad 1: +5V_FUSE -> +5V_JOYSTICK
- R53 pad 1: +3V3_2 -> +3V3
- R54 pad 1: GNDA -> GND
- R57 pad 1: GNDA -> GND
- R78 pad 1: +3V3_2 -> +3V3
- R90 pad 2: GNDA -> GND
- R91 pad 2: GNDA -> GND
- R92 pad 2: GNDA -> GND
- U12 pad 4: GNDA -> GND
- U14 pad 2: GNDA -> GND
- U15 pad 1: (no net) -> unconnected-(U15-NC-Pad1)
- U16 pad 1: (no net) -> unconnected-(U16-NC-Pad1)
- U17 pad 1: (no net) -> unconnected-(U17-NC-Pad1)
- U18 pad 1: (no net) -> unconnected-(U18-NC-Pad1)
- U2 pad 149: /~{IORQ2} -> unconnected-(U2-IO_149-Pad149)
- U2 pad 182: /~{SPI_CS} -> /~{SPICS}
- U2 pad 62: unconnected-(U2-IO_62/LOCK-Pad62) -> Net-(U2-IO_62/LOCK)
- U2 pad 63: unconnected-(U2-IO_63-Pad63) -> +3V3
- U2 pad 64: unconnected-(U2-IO_64-Pad64) -> +3V3
- U2 pad 68: unconnected-(U2-IO_68-Pad68) -> +3V3
- U2 pad 80: /~{IORQGE2} -> GND
- U20 pad 1: (no net) -> unconnected-(U20-NC-Pad1)
- U20 pad 3: GNDA -> GND
- U22 pad 2: GNDA -> GND
- U23 pad 1: GNDA -> GND
- U23 pad 12: GNDA -> GND
- U23 pad 14: GNDA -> GND
- U23 pad 15: GNDA -> GND
- U23 pad 2: GNDA -> GND
- U23 pad 25: GNDA -> GND
- U23 pad 26: GNDA -> GND
- U23 pad 27: GNDA -> GND
- U23 pad 31: GNDA -> GND
- U23 pad 33: GNDA -> GND
- U23 pad 39: GNDA -> GND
- U23 pad 40: GNDA -> GND
Routing:
- net /~{WR}: track 0.00 -> 26.9 mm
- net /~{RD}: track 0.00 -> 26.4 mm
- net /RES: track 0.00 -> 26.0 mm
- net /SDDO: track 0.00 -> 25.6 mm
- net /SDDI: track 0.00 -> 25.6 mm
- net /~{WAIT}: track 0.00 -> 25.4 mm
- net /~{SDCS}: track 0.00 -> 25.0 mm
- net /~{RRAS0}: track 0.00 -> 24.9 mm, vias 0 -> 2
- net /~{M1}: track 0.00 -> 24.8 mm
- net /~{RWE}: track 0.00 -> 24.4 mm, vias 0 -> 1
- net /RD0: track 0.00 -> 24.0 mm, vias 0 -> 1
- net /~{RFSH}: track 0.00 -> 23.1 mm
- net /RD1: track 0.00 -> 23.1 mm, vias 0 -> 1
- net /RA0: track 0.00 -> 22.9 mm, vias 0 -> 1
- net /~{IORQ1}: track 0.00 -> 22.7 mm
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- added copper zone on B.Cu, net +2V5
- added copper zone on F.Cu, net +3V3
Other:
- board text added: "PCB Rev.${REVISION} Eugene Lozovoy 2024 Original design by NedoPC VDAC2 design by TSL"
- board text added: "ZXEVO.1010"
- board text removed: "1010"
- board text removed: "PCB Rev.${REVISION} Eugene Lozovoy 2024"
- board text removed: "ZXEVO"

Commit message: wip pcb rev.A
Parts:
- C25: moved to B.Cu
- U2: footprint Package_QFP:LQFP-208_28x28mm_P0.5mm -> PCM_Package_QFP_AKL:LQFP-208_28x28mm_P0.5mm
- moved C4 57.6 mm to (110.7, 128.2), turned to 180 degrees
- moved Y2 56.6 mm to (110.7, 126.7), turned to 90 degrees
- moved C17 56.3 mm to (111.7, 120.2)
- moved C69 56.3 mm to (110.2, 120.2)
- moved U11 56.3 mm to (110.7, 119.0)
- moved C3 55.8 mm to (110.7, 125.2), turned to 0 degrees
- moved C76 45.7 mm to (107.2, 91.2), turned to 90 degrees
- moved C63 45.5 mm to (115.8, 124.7), turned to 180 degrees
- moved R33 45.5 mm to (150.4, 79.9), turned to 180 degrees
- moved C16 44.6 mm to (115.8, 123.2), turned to 0 degrees
- moved C65 42.7 mm to (189.7, 97.0), turned to -90 degrees
- moved U15 41.9 mm to (188.9, 96.9), turned to -90 degrees
- moved C55 41.4 mm to (151.0, 84.5), turned to 90 degrees
- moved R14 41.1 mm to (140.2, 80.3), turned to 180 degrees
- moved R76 41.1 mm to (188.2, 97.0), turned to -90 degrees
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Connections:
- J22 pad 5: +5V_FUSE -> +5V_JOYSTICK
Routing:
- net +3V3: track 0.00 -> 56.4 mm, vias 0 -> 12
- net /CLKZ_OUT: track 0.00 -> 50.2 mm, vias 0 -> 1
- net +2V5: track 0.00 -> 37.1 mm, vias 0 -> 12
- net /~{IORQ}: track 0.00 -> 36.1 mm
- net /~{MREQ}: track 0.00 -> 35.1 mm
- net /~{NMI}: track 0.00 -> 34.3 mm
- net /~{INT}: track 0.00 -> 32.5 mm
- net /~{ROMOE}: track 19.4 -> 51.4 mm
- net /D7: track 0.00 -> 31.7 mm
- net /~{ROMWE}: track 19.1 -> 50.3 mm
- net /D6: track 0.00 -> 30.8 mm
- net /D5: track 0.00 -> 30.0 mm
- net /ROMPG2: track 18.8 -> 48.7 mm
- net /D4: track 0.00 -> 29.4 mm
- net /ROMPG3: track 18.5 -> 47.6 mm
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Other:
- board text added: "Original design by NedoPC"
- board text added: "PCB Rev.${REVISION} Eugene Lozovoy 2024"
- board text added: "VDAC2 design by TSL"
- board text removed: "PCB Rev.${REVISION} Eugene Lozovoy 2024 Original design by NedoPC VDAC2 design by TSL"

Commit message: wip pcb rev.A
Parts:
- J5: footprint Connector_PinHeader_2.54mm:PinHeader_2x05_P2.54mm_Vertical -> Connector_PinHeader_2.54mm:PinHeader_2x03_P2.54mm_Vertical
- J8: footprint Connector_PinHeader_2.54mm:PinHeader_2x04_P2.54mm_Vertical -> Connector_PinHeader_2.54mm:PinHeader_2x03_P2.54mm_Vertical
- U24: footprint Package_DFN_QFN:QFN-56-1EP_8x8mm_P0.5mm_EP4.3x4.3mm -> my:QFN-56-1EP_8x8mm_P0.5mm_EP4.3x4.3mm
- U3: footprint my:TQFP-44_14x14mm_P0.8mm -> my:Z80_FEC_VEC
- moved BT1 82.8 mm to (100.2, 93.1), turned to -90 degrees
- moved C59 27.8 mm to (189.9, 93.7)
- moved R77 27.8 mm to (188.4, 93.7)
- moved U16 27.8 mm to (189.1, 93.7)
- moved R37 27.8 mm to (191.5, 93.7)
- moved R64 26.8 mm to (181.1, 118.3), turned to 0 degrees
- moved C58 25.7 mm to (126.6, 114.8), turned to -90 degrees
- moved C1 25.2 mm to (112.9, 115.8), turned to 90 degrees
- moved Y1 24.7 mm to (111.2, 114.8), turned to 0 degrees
- moved C2 24.6 mm to (114.4, 115.8), turned to 90 degrees
- moved U5 24.0 mm to (123.6, 114.8), turned to 180 degrees
- moved R25 20.1 mm to (121.3, 113.0), turned to 180 degrees
- moved C67 18.8 mm to (189.9, 83.1)
- moved R85 18.8 mm to (188.4, 83.1)
- moved U17 18.8 mm to (189.2, 83.1)
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Connections:
- J5 pad 1: /SPICK -> /PRGDO
- J5 pad 2: GND -> +5V
- J5 pad 3: /PRGDO -> /SPICK
- J5 pad 4: +5V -> /PRGDI
- J5 pad 6: unconnected-(J5-Pin_6-Pad6) -> GND
- J8 pad 5: GND -> /TAPE_IN
- J8 pad 6: GND -> /MIXER_R
Routing:
- net /~{RFSH}: track 33.8 -> 110.3 mm, vias 0 -> 2
- net /~{M1}: track 32.8 -> 105.7 mm, vias 0 -> 3
- net /~{WAIT}: track 32.3 -> 94.9 mm, vias 0 -> 3
- net /~{WR}: track 30.4 -> 93.0 mm, vias 0 -> 3
- net /~{RD}: track 31.1 -> 92.5 mm, vias 0 -> 1
- net /D0: track 26.1 -> 85.0 mm, vias 0 -> 4
- net /D1: track 27.1 -> 85.3 mm, vias 0 -> 4
- net /D7: track 31.7 -> 86.2 mm, vias 0 -> 2
- net /D2: track 27.9 -> 80.9 mm, vias 0 -> 4
- net /A13: track 20.8 -> 72.7 mm, vias 0 -> 2
- net /A8: track 16.6 -> 65.8 mm, vias 0 -> 2
- net /A9: track 17.3 -> 65.0 mm, vias 0 -> 2
- net /A12: track 20.0 -> 67.6 mm, vias 0 -> 2
- net /A11: track 19.1 -> 65.8 mm, vias 0 -> 2
- net /D6: track 30.8 -> 76.5 mm, vias 0 -> 2
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