File: pcb_main/rev.A/zxevo1010_main.kicad_pcb (KiCad board)
At the start: 2 copper layers, 100 x 100 mm, 248 parts, among them J10 Conn_02x30_Row_Letter_First, J11 TE 041021-4, J12 MEM2055-00-190-01-A, J13 Conn_02x05_Odd_Even, J14 Conn_02x05_Odd_Even, J2 B2B-XH-A, J3 Mini-DIN-6, J4 USB_B_Micro, J5 Conn_02x05_Odd_Even, J6 Mini-DIN-6, J7 DB15_Female_HighDensity_Mount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, J8 PJ-320, J9 Conn_02x05_Odd_Even, Q1 BC847, Q2 BC856, Q3 BC856, Q4 BC856, SW2 SW_Push, SW3 SW_Push, SW4 SW_Push, U1 CH340X, U10 74LVC2G04DB, U11 EPM3128ATC100, U12 29F040-K, U13 74LVC2G04DB, U14 LP2985-3.3, U15 LMV358IDR, U16 ATmega128, U17 Z84C0020FEC, U18 PCF8583T, U19 CD4069UBM, U2 HY5118160, U20 1117-3.3, U21 1117-2.5, U22 LP2985-3.3, U23 LP2985-3.3, U24 1117-3.3, U3 HY5118160, U4 ICS501, U5 74LVC2G04DB, U6 EP1K50QC208, U7 ADV7125-lqfp48, U8 74LVC2G04DB, U9 FT812, Y1 14 MHz, Y2 8 MHz, Y3 11.059 Mhz, Y4 32768 Hz

Commit message: wip pcb rev.A (almost done)
Parts:
- U10, U13, U5, U8: value 74LVC2G04DB -> SN74LVC2G04DBVR
Changed lines of the file:
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@@
 			)
 		)
-		(property "Value" "74LVC2G04DB"
-			(at 2.25 0 180)
+		(property "Value" "SN74LVC2G04DBVR"
+			(at 2.05 -2.15 180)
 			(layer "F.Fab")
 			(effects
@@
 			(effects
 				(font
-					(size 1.1 0.75)
-					(thickness 0.14)
+					(size 1.1 0.6)
+					(thickness 0.11)
 				)
 			)
@@
 			)
 		)
-		(property "Value" "74LVC2G04DB"
-			(at 3.1 2.9 0)
+		(property "Value" "SN74LVC2G04DBVR"
+			(at 5.15 2.9 0)
 			(layer "F.Fab")
 			(effects
@@
 			(effects
 				(font
-					(size 1.1 0.8)
-					(thickness 0.14)
+					(size 1.1 0.6)
+					(thickness 0.11)
 				)
 			)
@@
 			)
 		)
-		(property "Value" "74LVC2G04DB"
+		(property "Value" "SN74LVC2G04DBVR"
 			(at 0.025 3.25 0)
 			(layer "F.Fab")
@@
 			(effects
 				(font
-					(size 1.1 0.8)
-					(thickness 0.14)
+					(size 1.1 0.6)
+					(thickness 0.11)
 				)
 			)
@@
 			)
 		)
-		(property "Value" "74LVC2G04DB"
+		(property "Value" "SN74LVC2G04DBVR"
 			(at 0 2.9 90)
 			(layer "F.Fab")
@@
 			(effects
 				(font
-					(size 1.1 0.8)
-					(thickness 0.14)
+					(size 1.1 0.6)
+					(thickness 0.11)
 				)
 			)
@@
 		)
 		(property "Value" "LP2985-3.3"
-			(at 2.4 -2.9 0)
+			(at 2.2 -2.9 0)
 			(layer "F.Fab")
 			(effects
@@
 				(face "ZX Spectrum 7")
 				(size 0.97 0.97)
-				(thickness 0.2)
+				(thickness 0.194)
+				(bold yes)
 			)
 		)
@@
 				(face "ZX Spectrum 7")
 				(size 0.97 0.97)
-				(thickness 0.2)
+				(thickness 0.194)
+				(bold yes)
 			)
 		)
@@
 				(face "ZX Spectrum 7")
 				(size 0.97 0.97)
-				(thickness 0.2)
+				(thickness 0.194)
+				(bold yes)
 			)
 		)

Commit message: wip pcb rev.A
Parts:
- C12, C17: moved to B.Cu
- C13, C16: value 10u -> 100u; footprint Capacitor_Tantalum_SMD:CP_EIA-3216-18_Kemet-A_Pad1.58x1.35mm_HandSolder -> Capacitor_Tantalum_SMD:CP_EIA-6032-28_Kemet-C_Pad2.25x2.35mm_HandSolder; moved to F.Cu
- C32, C43: footprint Capacitor_SMD:CP_Elec_5x5.9 -> Capacitor_Tantalum_SMD:CP_EIA-6032-28_Kemet-C_Pad2.25x2.35mm_HandSolder
- C6: value 4.7u -> 100n
- R1, R11, R12, R2: value 4.7k -> 10k
- R19: value 530 -> 10k
- R36, R38: value 24k -> 47k
- R39, R53: value 47 -> 51
- R45, R60: value 4.7k -> 8.2k
- R51, R69, R70, R71: value 10k -> 1k
- R52, R58: value 24k -> 27k
- U12: value 29F040-K -> 29F040
- U7: value ADV7125-lqfp48 -> ADV7125
- moved R81 35.2 mm to (144.3, 80.3), turned to 180 degrees
- moved C13 14.5 mm to (118.3, 61.9), turned to 180 degrees
- moved C16 14.4 mm to (118.3, 65.6), turned to 180 degrees
- moved C19 8.83 mm to (112.8, 68.3), turned to 180 degrees
- moved R54 7.87 mm to (112.8, 69.8), turned to 0 degrees
- moved R38 6.64 mm to (120.7, 63.2), turned to 180 degrees
- moved C20 5.97 mm to (112.8, 65.3), turned to 180 degrees
- moved C11 5.85 mm to (118.3, 67.8), turned to 180 degrees
- moved R55 5.52 mm to (112.8, 66.8), turned to 0 degrees
- moved R58 5.23 mm to (120.7, 64.7), turned to 180 degrees
- moved R56 4.67 mm to (112.8, 63.8), turned to 0 degrees
- moved R87 4.39 mm to (108.6, 68.7), turned to 0 degrees
- moved R36 4.04 mm to (120.7, 60.2), turned to 180 degrees
- moved C21 4.01 mm to (112.8, 62.3), turned to 180 degrees
- moved R59 3.91 mm to (131.9, 56.2), turned to 0 degrees
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Connections:
- R65 pad 2: /~{SPICS} -> /SPICK
- R81 pad 1: +5V_2 -> +2V5
- U13 pad 1: /~{BEEP} -> /BEEP
Routing:
- net Net-(C16-Pad2): track 3.94 -> 23.4 mm, vias 0 -> 1
- net Net-(C13-Pad2): track 4.43 -> 22.2 mm, vias 0 -> 1
- net GND: track 94.9 -> 82.2 mm, vias 393 -> 400
- net +5V_2: track 210.0 -> 200.8 mm
- net +3V3_AUDIO: track 38.4 -> 30.3 mm, vias 4 -> 5
- net Net-(C13-Pad1): track 8.79 -> 2.36 mm, vias 2 -> 1
- net +5V: track 516.1 -> 509.7 mm
- net Net-(C17-Pad2): track 3.48 -> 9.50 mm, vias 1 -> 0
- net /~{BEEP}: track 7.26 -> 1.30 mm
- net Net-(C16-Pad1): track 7.02 -> 11.3 mm, vias 2 -> 1
- net /MIXER_R: track 40.5 -> 37.2 mm, vias 2 -> 3
- net /A4: track 84.0 -> 80.8 mm
- net Net-(D5-A): track 6.47 -> 3.63 mm
- net /A3: track 84.7 -> 81.9 mm
- net +2V5: track 57.0 -> 59.8 mm, vias 16 -> 17
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