File: pcb_main/rev.A/zxevo1010_main.kicad_pcb (KiCad board)
At the start: 2 copper layers, 100 x 100 mm, 248 parts, among them J10 Conn_02x30_Row_Letter_First, J11 TE 041021-4, J12 MEM2055-00-190-01-A, J13 Conn_02x05_Odd_Even, J14 Conn_02x05_Odd_Even, J2 B2B-XH-A, J3 Mini-DIN-6, J4 USB_B_Micro, J5 Conn_02x05_Odd_Even, J6 Mini-DIN-6, J7 DB15_Female_HighDensity_Mount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, J8 PJ-320, J9 Conn_02x05_Odd_Even, Q1 BC847, Q2 BC856, Q3 BC856, Q4 BC856, SW2 SW_Push, SW3 SW_Push, SW4 SW_Push, U1 CH340X, U10 SN74LVC2G04DBVR, U11 EPM3128ATC100, U12 29F040, U13 SN74LVC2G04DBVR, U14 LP2985-3.3, U15 LMV358IDR, U16 ATmega128, U17 Z84C0020FEC, U18 PCF8583T, U19 CD4069UBM, U2 HY5118160, U20 1117-3.3, U21 1117-2.5, U22 LP2985-3.3, U23 LP2985-3.3, U24 1117-3.3, U3 HY5118160, U4 ICS501, U5 SN74LVC2G04DBVR, U6 EP1K50QC208, U7 ADV7125, U8 SN74LVC2G04DBVR, U9 FT812, Y1 14 MHz, Y2 8 MHz, Y3 11.059 Mhz, Y4 32768 Hz

Commit message: wip pcb rev.A
Parts:
- C37, C40, C90: value 100n -> 10n
Routing:
- net GND: track 82.2 -> 84.6 mm
Changed lines of the file:
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@@
 		(tags "SOIC SO")
 		(property "Reference" "U15"
-			(at 4.7 3.425 90)
+			(at 4.7 3.125 90)
 			(layer "F.SilkS")
 			(effects
@@
 		)
 		(property "ValueSilk" "${VALUE}"
-			(at 4.7 -1.475 90)
+			(at 4.7 -1.175 90)
 			(layer "F.SilkS")
 			(effects
 				(font
-					(size 1.1 0.8)
-					(thickness 0.14)
+					(size 1.1 0.65)
+					(thickness 0.12)
+					(bold yes)
 				)
 			)
@@
 			)
 		)
-		(property "Value" "100n"
-			(at 3.8125 0 180)
+		(property "Value" "10n"
+			(at 2.7625 0 180)
 			(layer "B.Fab")
 			(effects
@@
 			)
 		)
-		(property "Value" "100n"
+		(property "Value" "10n"
 			(at -0.3875 -2.75 0)
 			(layer "B.Fab")
@@
 			)
 		)
-		(property "Value" "100n"
-			(at 1.7 -1.3 0)
+		(property "Value" "10n"
+			(at 1.7 -0.86 0)
 			(layer "B.Fab")
 			(effects
@@
 	)
 	(segment
+		(start 126.614273 99.485727)
+		(end 126.55 99.55)
+		(width 0.15)
+		(layer "F.Cu")
+		(net 1)
+	)
+	(segment
 		(start 160.55 68.6625)
 		(end 159.3625 68.6625)
@@
 	)
 	(segment
+		(start 128.825 99.65)
+		(end 127.283942 99.65)
+		(width 0.15)
+		(layer "F.Cu")
+		(net 1)
+	)
+	(segment
 		(start 150.3875 74.325)
 		(end 150.3875 75.4)
@@
 	)
 	(segment
+		(start 127.119669 99.485727)
+		(end 126.614273 99.485727)
+		(width 0.15)
+		(layer "F.Cu")
+		(net 1)
+	)
+	(segment
 		(start 152.9 75.4125)
 		(end 150.4 75.4125)
@@
 	)
 	(segment
+		(start 127.283942 99.65)
+		(end 127.119669 99.485727)
+		(width 0.15)
+		(layer "F.Cu")
+		(net 1)
+	)
+	(segment
 		(start 152.8875 72.3625)
 		(end 152.8875 71.939184)
@@
 	)
 	(segment
-		(start 128.148656 100.15)
-		(end 127.698656 99.7)
+		(start 127.978322 99.979666)
+		(end 128.148656 100.15)
+		(width 0.15)
+		(layer "F.Cu")
+		(net 90)
+	)
+	(segment
+		(start 126.933267 99.979666)
+		(end 127.978322 99.979666)
 		(width 0.15)
 		(layer "F.Cu")
@@
 	)
 	(segment
-		(start 127.698656 99.7)
-		(end 126.95 99.7)
+		(start 126.902206 100.010727)
+		(end 126.933267 99.979666)
 		(width 0.15)
 		(layer "F.Cu")
@@
 	)
 	(via
-		(at 126.95 99.7)
+		(at 126.902206 100.010727)
 		(size 0.6)
 		(drill 0.3)
@@
 	)
 	(segment
-		(start 126.95 99.7)
-		(end 127.0375 99.7)
+		(start 126.902206 100.010727)
+		(end 126.902206 99.835294)
 		(width 0.15)
 		(layer "B.Cu")
@@
 	)
 	(segment
-		(start 127.0375 99.7)
+		(start 126.902206 99.835294)
 		(end 127.8125 98.925)
 		(width 0.15)

Commit message: wip pcb rev.A
Parts:
- Y3: value 11.059 Mhz -> 11.059 MHz
Other:
- board text added: "VDAC's CPLD"
Changed lines of the file:
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@@
 			)
 		)
+		(property "K" "K"
+			(at -0.76 2.15 0)
+			(layer "F.SilkS")
+			(effects
+				(font
+					(size 1.1 0.6)
+					(thickness 0.14)
+				)
+			)
+		)
+		(property "A" "A"
+			(at 3.24 2.15 0)
+			(layer "F.SilkS")
+			(effects
+				(font
+					(size 1.1 0.6)
+					(thickness 0.14)
+				)
+			)
+		)
 		(property ki_fp_filters "LED* LED_SMD:* LED_THT:*")
 		(sheetname "Root")
@@
 			)
 		)
+		(property "K" "K"
+			(at -0.75 2.15 0)
+			(layer "F.SilkS")
+			(effects
+				(font
+					(size 1.1 0.6)
+					(thickness 0.14)
+				)
+			)
+		)
+		(property "A" "A"
+			(at 3.25 2.15 0)
+			(layer "F.SilkS")
+			(effects
+				(font
+					(size 1.1 0.6)
+					(thickness 0.14)
+				)
+			)
+		)
 		(property ki_fp_filters "LED* LED_SMD:* LED_THT:*")
 		(sheetname "Root")
@@
 			)
 		)
+		(property "K" "K"
+			(at -0.7875 2.15 0)
+			(layer "F.SilkS")
+			(effects
+				(font
+					(size 1.1 0.6)
+					(thickness 0.14)
+				)
+			)
+		)
+		(property "A" "A"
+			(at 3.2625 2.15 0)
+			(layer "F.SilkS")
+			(effects
+				(font
+					(size 1.1 0.6)
+					(thickness 0.14)
+				)
+			)
+		)
 		(property ki_fp_filters "LED* LED_SMD:* LED_THT:*")
 		(sheetname "Root")
@@
 			)
 		)
-		(property "Value" "11.059 Mhz"
+		(property "Value" "11.059 MHz"
 			(at 2.775 0 180)
 			(layer "F.Fab")
@@
 		)
 	)
+	(gr_text "VDAC's CPLD"
+		(at 152.8875 66.0317 0)
+		(layer "F.SilkS")
+		(effects
+			(font
+				(size 1.1 0.8)
+				(thickness 0.14)
+				(bold yes)
+			)
+			(justify top)
+		)
+	)
