File: pcb_main/rev.A/zxevo1010_main.kicad_sch (KiCad schematic)
At the start: 210 parts, among them J1 Mini-DIN-6, J10 TE 041021-4, J13 Conn_02x05_Odd_Even, J16 MEM2055-00-190-01-A, J17 B2B-XH-A, J18 XHP-2, SXH-002T-P0.6, J2 USB_B_Micro, J22 Conn_02x05_Odd_Even, J3 Mini-DIN-6, J4 PJ-320, J5 Conn_02x05_Odd_Even, J6 Conn_02x30_Row_Letter_First, J8 Conn_02x05_Odd_Even, J9 DB15_Female_HighDensity_Mount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, Q1 BC856, Q2 BC856, Q3 BC847, Q6 BC847, SW1 PB05A, SW3 SW_Push, SW5 SW_Push, SW6 SW_Push, U1 39SF040, U10 GM71C(S)18163CT, U11 CH340X, U12 LMV358IDR, U13 PCF8583T, U14 LP2985-3.3, U15 74LVC1G04DB, U16 74LVC1G04DB, U17 74LVC1G04DB, U18 74LVC1G04DB, U19 CD4069UBM, U2 EP1K50QC208, U20 74LVC1G04DB, U21 EPM3128ATC100, U22 LP2985-3.3, U23 ADV7125-lqfp48, U24 FT812, U3 Z80CPU_QFP, U4 74HCT245PW, U5 ICS501, U6 ATmega128, U7 GM71C(S)18163CT, U8 1117-3.3, U9 1117-2.5, Y1 14 MHz, Y2 11.059 Mhz, Y3 32768 Hz, Y4 8 MHz

Commit message: wip pcbs rev.A
Parts:
- removed C24, C27: 10u, Capacitor_Tantalum_SMD:CP_EIA-3216-18_Kemet-A_Pad1.58x1.35mm_HandSolder, symbol Device:C_Polarized
- removed JP2: SolderJumper_2_Open, Jumper:SolderJumper-2_P1.3mm_Open_RoundedPad1.0x1.5mm, symbol Jumper:SolderJumper_2_Open
- removed Q3: BC847, Package_TO_SOT_SMD:SOT-23, symbol Transistor_BJT:BC847
- removed R19: 1k, Resistor_SMD:R_0603_1608Metric_Pad0.98x0.95mm_HandSolder, symbol Device:R
- removed R20, R42, R43: 75, Resistor_SMD:R_0603_1608Metric_Pad0.98x0.95mm_HandSolder, symbol Device:R
- removed R65, R66: 47k, Resistor_SMD:R_0603_1608Metric_Pad0.98x0.95mm_HandSolder, symbol Device:R
- removed R67, R95: 10k, Resistor_SMD:R_0603_1608Metric_Pad0.98x0.95mm_HandSolder, symbol Device:R
- removed U4: 74HCT245PW, Package_SO:TSSOP-20_4.4x6.5mm_P0.65mm, symbol 74xx:74LS245
- added C24, C27, C42: 18p, Capacitor_SMD:C_0603_1608Metric_Pad1.08x0.95mm_HandSolder, symbol Device:C
- added C43: 10u, Capacitor_Tantalum_SMD:CP_EIA-3216-18_Kemet-A_Pad1.58x1.35mm_HandSolder, symbol Device:C_Polarized
- added R6: 120, Resistor_SMD:R_0603_1608Metric_Pad0.98x0.95mm_HandSolder, symbol Device:R
- R15: value 240 -> 1k
- R16, R7: value 430 -> 1k
- R17: value 240 -> 24k
- R18: value 430 -> 24k
- R2: value 240 -> 120
- R21, R22, R23: value 100 -> 75
- R24: value 10k -> 1k
Connections:
- net TOP_IN_L is gone; now on net MIXER_L: J8.2 (Pin_2)
- net TOP_IN_R is gone; now on net MIXER_R: J8.8 (Pin_8)
- net VB+ is gone; now on net MIXER_L: R17.1
- net VB- is gone; now on net MIXER_R: R18.1
- net VGA_VS is gone; now on net V_VS_OUT: J9.14
- net VR- is gone; now on net FT_AU_L: R16.1
- net FT_AU_L: now also C42.1, C43.1; no longer U24.3 (AUDIO_L)
- net FT_MISO: now also U2.99 (IO_99)
- net FT_MOSI: now also U2.103 (IO_103)
- net FT_SCK: now also U2.104 (IO_104)
- net GND: now also C24.2, C27.2, C42.2
- net M_SEL: now also U2.100 (IO_100)
- net O_B0: now also U2.83 (IO_83)
- net O_B1: now also U2.86 (IO_86)
- net O_B2: now also U2.88 (IO_88)
- net O_B3: now also U2.90 (IO_90)
- net O_B4: now also U2.93 (IO_93)
- net O_CLK: now also U2.111 (IO_111)
- net O_G0: now also U2.75 (IO_75)
- net O_G1: now also U2.73 (IO_73)
- net O_G2: now also U2.96 (IO_96)
- net O_G3: now also U2.71 (IO_71)
- net O_G4: now also U2.74 (IO_74)
- net O_HS: now also U2.113 (IO_113)
- net O_R0: now also U2.94 (IO_94)
- net O_R1: now also U2.92 (IO_92)
- net O_R2: now also U2.89 (IO_89)
- net O_R3: now also U2.87 (IO_87)
- net O_R4: now also U2.85 (IO_85)
- net O_VS: now also U2.112 (IO_112)
- net PAL_SEL: now also U2.95 (IO_95)
- net TCK_FPGA: now also U21.62 (TCK)
- net TDO_FPGA: now also U21.4 (TDI); no longer J13.3 (Pin_3)
- net TMS_FPGA: now also U21.15 (TMS)
- net ~{FT_CS}: now also U2.101 (IO_101)
- net MIXER_R: now reaches R50.2, R58.1, U12.6 (-)
- net MIXER_L: now reaches R49.2, R55.1, U12.2 (-)
- net at C2.2, U5.1 (X1): now also Y1.2; no longer Y1.1
- net at C1.2, U5.8 (X2): now also Y1.1; no longer Y1.2
- net V_B: now reaches U23.28 (IOB)
- net V_B: now also J9.3, R21.2
- net V_G: now reaches U23.32 (IOG)
- net V_G: now also J9.2, R22.2
- net V_R: now reaches U23.34 (IOR)
- net V_R: now also J9.1, R23.2
- net V_HS: now reaches U21.49 (I/O)
- net V_HS: now also R6.2
- net V_VS: now reaches U21.50 (I/O)
- net V_VS: now also R2.2
- net TDO_CPLD: now reaches U21.73 (TDO)
- net TDO_CPLD: now also J13.3 (Pin_3)
- net VCSYNC: no longer names the net of U2.122 (IO_122)
- net VG+ renamed V_VS_OUT
- net VG-: no longer names the net of R7.1
- net VG-: now also R15.2, C24.1
- net VGA_B: no longer names the net of R17.2, R18.2
- net VGA_B: now also C43.2; no longer J9.3, R21.2
- removed net VGA_G: J9.2, R2.2, R22.2, R7.2
- net VGA_HS renamed V_HS_OUT
- net V_HS_OUT: now also R6.1
- removed net VGA_R: J9.1, R15.2, R16.2, R23.2
- net VHSYNC: no longer names the net of U2.121 (IO_121)
- net VR+: no longer names the net of R15.1
- net VR+: now also R16.2, C27.1
- net VVSYNC: no longer names the net of U2.120 (IO_120)
- net V_B+: no longer names the net of U2.126 (IO_126)
- net V_B-: no longer names the net of U2.125 (IO_125)
- net V_G+: no longer names the net of U2.128 (IO_128)
- net V_G-: no longer names the net of U2.127 (IO_127)
- net V_R+: no longer names the net of U2.132 (IO_132)
- net V_R-: no longer names the net of U2.131 (IO_131)
- new net: R7.2, U24.3 (AUDIO_L)
- no-connect marks 83 -> 87
Other:
- note removed: "VGA"
- moved on the sheet: C17, C33, C34, C36, C37, C38, J17, J2, J9, JP3, R1, R21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

Commit message: wip pcbs rev.A
Parts:
- removed R35: 680, Resistor_SMD:R_0603_1608Metric_Pad0.98x0.95mm_HandSolder, symbol Device:R
- added C44, C45, C46, C47, C48, C49, C51, C52, C54, C55, C56, C57, C58, C59, C60, C61, C62, C63, C64, C65, C66, C67, C69, C70, C71, C72, C73, C75, C76, C77, C78, C79, C80, C81, C85, C87: 100n, Capacitor_SMD:C_0603_1608Metric_Pad1.08x0.95mm_HandSolder, symbol Device:C
- added C82, C83: 1u, Capacitor_SMD:C_0603_1608Metric_Pad1.08x0.95mm_HandSolder, symbol Device:C
- added C88: 10u, Capacitor_SMD:C_0805_2012Metric_Pad1.18x1.45mm_HandSolder, symbol Device:C
- added F1: 0.2A, Fuse:Fuse_1812_4532Metric_Pad1.30x3.40mm_HandSolder, symbol Device:Polyfuse
- added Q3: BC856, Package_TO_SOT_SMD:SOT-23, symbol Transistor_BJT:BC856
- added R43: 10k, Resistor_SMD:R_0603_1608Metric_Pad0.98x0.95mm_HandSolder, symbol Device:R
- C35, C50: value 1u -> 100n
- J16: now not fitted; now left out of the parts list
- U1: value 39SF040 -> 29F040-K
- U10, U7: value GM71C(S)18163CT -> HY5118160
- U3: value Z80CPU_QFP -> Z84C0020FEC
Connections:
- net +3V3_2 is gone; now on net +3V3: L2.1, R28.1, R31.1, R32.1, R53.1, R78.1
- net GNDA is gone; now on net GND: C11.1, C19.2, C28.1, C29.2, C31.2, C5.1, C6.1, C7.1, J4.R2, J4.S, J8.3 (Pin_3), J8.4 (Pin_4), J8.5 (Pin_5), J8.6 (Pin_6), J9.0, J9.10, J9.5, J9.6, J9.7, J9.8, R1.1, R11.1, R21.1, R22.1, R23.1, R54.1, R57.1, R90.2, R91.2, R92.2, U12.4 (V-), U14.2 (GND), U20.3 (GND), U22.2 (GND), U23.1 (GND), U23.12 (~{SYNC}), U23.14 (GND), U23.15 (GND), U23.2 (GND), U23.25 (GND), U23.26 (GND), U23.27 (~{IOB}), U23.31 (~{IOG}), U23.33 (~{IOR}), U23.39 (GND), U23.40 (GND)
- net ~{IORQGE2} is gone; now on net GND: U2.80 (Dedicated_Input)
- net ~{SPI_CS} is gone; now on net ~{SPICS}: U2.182 (Dedicated_Input)
- net +2V5: now also C32.1, C35.1, C44.1, C45.1, C46.1, C47.1, C48.1, C61.1; no longer C32.2, C35.2
- net +3V3: now also C50.1, C53.1, U2.63 (IO_63), U2.64 (IO_64), U2.68 (IO_68), C49.1, C51.1, C54.1, C55.1, C56.1, C57.1, C77.1, C78.1, C79.1, C80.1, C81.1, C82.1, R43.1; no longer C50.2, C53.2
- net +3V3_AUDIO: now also C52.1, C88.2
- net +3V3_VIDEO: now also C83.1, C85.1, C87.1
- net +5V: now also C58.2, C59.2, C60.2, C62.2, C63.2, C64.2, C65.2, C66.2, C67.2, C69.2, C70.2, C71.2, C72.2, C73.2, C75.2, C76.2, F1.1
- net +5V_FUSE: no longer R27.1, R29.1, R30.1, R36.1, R38.1, R46.1, R47.1
- net GND: now also C32.2, C35.2, C50.2, C53.2, C44.2, C45.2, C46.2, C47.2, C48.2, C49.2, C51.2, C52.2, C54.2, C55.2, C56.2, C57.2, C58.1, C59.1, C60.1, C61.2, C62.1, C63.1, C64.1, C65.1, C66.1, C67.1, C69.1, C70.1, C71.1, C72.1, C73.1, C75.1, C76.1, C77.2, C78.2, C79.2, C80.2, C81.2, C82.2, C83.2, C85.2, C87.2, C88.1, Q3.3 (C); no longer C32.1, C35.1, C50.1, C53.1
- net PRGDI: now also Q3.1 (B)
- net at Q1.2 (E), R3.1: now also Q3.2 (E)
- net at U2.62 (IO_62/LOCK): now also R43.2
- net ~{IORQ2}: no longer names the net of U2.149 (IO_149)
- new net +5V_JOYSTICK: F1.2, R27.1, R29.1, R30.1, R36.1, R38.1, R46.1, R47.1
- no-connect marks 87 -> 93
Other:
- note added: "JTAG & ISP"
- note added: "NemoBus"
- note removed: "Debug & ISP"
- moved on the sheet: BT1, C1, C10, C11, C12, C13, C14, C15, C16, C17, C18, C19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

Commit message: wip pcb rev.A
Parts:
- U2: footprint Package_QFP:LQFP-208_28x28mm_P0.5mm -> PCM_Package_QFP_AKL:LQFP-208_28x28mm_P0.5mm
Connections:
- net +5V_FUSE: no longer J22.5 (Pin_5)
- net +5V_JOYSTICK: now also J22.5 (Pin_5)
Changed lines of the file:
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@@
 	(text "Tape"
 		(exclude_from_sim no)
-		(at 209.296 405.638 0)
+		(at 200.406 405.638 0)
 		(effects
 			(font
@@
 			)
 		)
-		(property "Footprint" "Package_QFP:LQFP-208_28x28mm_P0.5mm"
+		(property "Footprint" "PCM_Package_QFP_AKL:LQFP-208_28x28mm_P0.5mm"
 			(at 62.23 145.415 0)
 			(effects
@@
 	)
 	(symbol
-		(lib_id "power:+5V")
-		(at 382.27 50.8 0)
-		(unit 1)
-		(exclude_from_sim no)
-		(in_bom yes)
-		(on_board yes)
-		(dnp no)
-		(property "Reference" "#PWR078"
-			(at 382.27 54.61 0)
-			(effects
-				(font
-					(size 1 1)
-				)
-				(hide yes)
-			)
-		)
-		(property "Value" "+5V_FUSE"
-			(at 383.794 46.736 0)
-			(effects
-				(font
-					(size 1 1)
-				)
-			)
-		)
-		(property "Footprint" ""
-			(at 382.27 50.8 0)
-			(effects
-				(font
-					(size 1.27 1.27)
-				)
-				(hide yes)
-			)
-		)
-		(property "Datasheet" ""
-			(at 382.27 50.8 0)
-			(effects
-				(font
-					(size 1.27 1.27)
-				)
-				(hide yes)
-			)
-		)
-		(property "Description" "Power symbol creates a global label with name \"+5V\""
-			(at 382.27 50.8 0)
-			(effects
-				(font
-					(size 1.27 1.27)
-				)
-				(hide yes)
-			)
-		)
-		(pin "1"
-		)
-		(instances
-			(project "zxevo1010"
-				(path "/895fa090-e1df-4200-a112-cb7c4b9368aa"
-					(reference "#PWR078")
-					(unit 1)
-				)
-			)
-		)
-	)
-	(symbol
 		(lib_id "power:GND")
 		(at 318.77 481.33 0)
@@
 					(unit 1)
 				)
+			)
+		)
+	)
+	(symbol
+		(lib_id "power:+5V")
+		(at 382.27 50.8 0)
+		(unit 1)
+		(exclude_from_sim no)
+		(in_bom yes)
+		(on_board yes)
+		(dnp no)
+		(property "Reference" "#PWR078"
+			(at 382.27 54.61 0)
+			(effects
+				(font
+					(size 1 1)
+				)
+				(hide yes)
+			)
+		)
+		(property "Value" "+5V_JOYSTICK"
+			(at 382.27 46.99 0)
+			(effects
+				(font
+					(size 1 1)
+				)
+			)
+		)
+		(property "Footprint" ""
+			(at 382.27 50.8 0)
+			(effects
+				(font
+					(size 1.27 1.27)
+				)
+				(hide yes)
+			)
+		)
+		(property "Datasheet" ""
+			(at 382.27 50.8 0)
+			(effects
+				(font
+					(size 1.27 1.27)
+				)
+				(hide yes)
+			)
+		)
+		(property "Description" "Power symbol creates a global label with name \"+5V\""
+			(at 382.27 50.8 0)
+			(effects
+				(font
+					(size 1.27 1.27)
+				)
+				(hide yes)
+			)
+		)
+		(pin "1"
+		)
+		(instances
+			(project "zxevo1010_main"
+				(path "/895fa090-e1df-4200-a112-cb7c4b9368aa"
+					(reference "#PWR078")
+					(unit 1)
+				)

Commit message: wip pcb rev.A
Parts:
- J5: footprint Connector_PinHeader_2.54mm:PinHeader_2x05_P2.54mm_Vertical -> Connector_PinHeader_2.54mm:PinHeader_2x03_P2.54mm_Vertical; symbol Connector_Generic:Conn_02x05_Odd_Even -> Connector_Generic:Conn_02x03_Odd_Even
- J8: footprint Connector_PinHeader_2.54mm:PinHeader_2x04_P2.54mm_Vertical -> Connector_PinHeader_2.54mm:PinHeader_2x03_P2.54mm_Vertical; symbol Connector_Generic:Conn_02x04_Odd_Even -> Connector_Generic:Conn_02x03_Odd_Even
- U24: footprint Package_DFN_QFN:QFN-56-1EP_8x8mm_P0.5mm_EP4.3x4.3mm -> my:QFN-56-1EP_8x8mm_P0.5mm_EP4.3x4.3mm
- U3: footprint my:TQFP-44_14x14mm_P0.8mm -> my:Z80_FEC_VEC; ValueAlt (none) -> Z84C0020VEC
Connections:
- net +5V: now also J5.2 (Pin_2); no longer J5.4 (Pin_4)
- net GND: now also J5.6 (Pin_6); no longer J5.10 (Pin_10), J5.2 (Pin_2), J8.5 (Pin_5), J8.6 (Pin_6)
- net MIXER_R: now also J8.6 (Pin_6); no longer J8.8 (Pin_8)
- net PRGDI: now also J5.4 (Pin_4); no longer J5.9 (Pin_9)
- net PRGDO: now also J5.1 (Pin_1); no longer J5.3 (Pin_3)
- net SPICK: now also J5.3 (Pin_3); no longer J5.1 (Pin_1)
- net TAPE_IN: now also J8.5 (Pin_5); no longer J8.7 (Pin_7)
- no-connect marks 93 -> 90
Other:
- moved on the sheet: R12, R13, R14, R33, R8, R9, U2

Commit message: wip pcb rev.A
Connections:
- net GND: now also SW5.1, SW6.1; no longer SW5.2, SW6.2
- net NMIKEY: now also SW5.2; no longer SW5.1
- net ~{SOFTRST}: now also SW6.2; no longer SW6.1
- net at C2.2, U5.1 (X1): now also Y1.1; no longer Y1.2
- net at C1.2, U5.8 (X2): now also Y1.2; no longer Y1.1
Changed lines of the file:
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@@
 		(lib_id "Device:Crystal")
 		(at 204.47 129.54 0)
+		(mirror y)
 		(unit 1)
 		(exclude_from_sim no)
@@
 		(lib_id "Switch:SW_Push")
 		(at 345.44 307.34 90)
-		(mirror x)
 		(unit 1)
 		(exclude_from_sim no)
@@
 		)
 		(property "Value" "SW_Push"
-			(at 341.63 309.2449 90)
+			(at 341.63 305.4351 90)
 			(effects
 				(font
@@
 		(lib_id "Switch:SW_Push")
 		(at 335.28 307.34 90)
-		(mirror x)
 		(unit 1)
 		(exclude_from_sim no)
@@
 		)
 		(property "Value" "SW_Push"
-			(at 331.47 309.2449 90)
+			(at 331.47 305.4351 90)
 			(effects
 				(font

Commit message: wip pcb rev.A
Parts:
- removed C65: 100n, Capacitor_SMD:C_0603_1608Metric_Pad1.08x0.95mm_HandSolder, symbol Device:C
- removed L2: 1u, Inductor_SMD:L_0805_2012Metric_Pad1.15x1.40mm_HandSolder, symbol Device:L
- removed U15, U16, U17, U18, U20: 74LVC1G04DB, Package_TO_SOT_SMD:SOT-23-5_HandSoldering, symbol 74xGxx:74LVC1G04
- added C89: 100n, Capacitor_SMD:C_0603_1608Metric_Pad1.08x0.95mm_HandSolder, symbol Device:C
- added C91: 10u, Capacitor_SMD:C_0805_2012Metric_Pad1.18x1.45mm_HandSolder, symbol Device:C
- added C92: 100u, Capacitor_SMD:CP_Elec_5x5.9, symbol Device:C_Polarized
- added U15, U16, U20, U25: 74LVC2G04, Package_TO_SOT_SMD:SOT-23-6_Handsoldering, symbol 74xGxx:74LVC2G04
- added U4: 1117-3.3, Package_TO_SOT_SMD:SOT-223-3_TabPin2, symbol Regulator_Linear:AZ1117-3.3
- C24, C27, C42: value 18p -> 4.7n
- C32, C35, C44, C45, C46, C47, C48, C49, C50, C51, C53, C54, C55, C56, C57, C61: footprint Capacitor_SMD:C_0603_1608Metric_Pad1.08x0.95mm_HandSolder -> Capacitor_SMD:C_0805_2012Metric_Pad1.18x1.45mm_HandSolder
- U13: footprint Package_SO:SOIC-8_3.9x4.9mm_P1.27mm -> my:SOT176-1
- Y2, Y4: footprint Crystal:Crystal_SMD_SeikoEpson_TSX3225-4Pin_3.2x2.5mm_HandSoldering -> my:Crystal_SMD_3225-4Pin_3.2x2.5mm_HandSoldering
Connections:
- net +3V3: no longer R28.1, R31.1, R32.1, R53.1, R78.1
- net +3V3_AUDIO: now also U25.5 (VCC)
- net +5V: now also C89.2, C91.2, U15.5 (VCC), U16.5 (VCC), U20.5 (VCC), U4.3 (VI)
- net CLKZ_OUT: now also U16.1
- net CSROM: now also U15.1
- net FT_AU_L: now also U24.3 (AUDIO_L), U25.3; no longer C42.1, C43.1, R16.1
- net GND: now also U24.15 (GPIO3), C89.1, C91.1, C92.2, U15.2 (GND), U15.3, U16.2 (GND), U16.3, U20.2 (GND), U25.2 (GND), U4.1 (GND)
- net RES: now also U20.3
- net ~{BEEP}: now also U25.1
- net ~{CSROM}: now also U15.6
- net ~{ROMPG0}: now also U20.1
- net at R86.1: now also U20.4
- net at R76.2: now also U20.6
- net at R52.2: now also U25.6
- net at R87.2, R88.2: now also U16.6
- net at R7.2: now also U25.4; no longer U24.3 (AUDIO_L)
- net SD_VDD renamed +3V3_SD
- net +3V3_SD: now also R28.1, R31.1, R32.1, R53.1, R78.1, C92.1, U4.2 (VO)
- new net: C42.1, C43.1, R16.1
- no-connect marks 90 -> 91
Other:
- moved on the sheet: C24, C25, C27, C32, C35, C42, C44, C45, C46, C47, C48, C52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

Commit message: wip pcb rev.A. Main board almost done
Parts:
- removed C26, C74: 10u, Capacitor_SMD:C_0805_2012Metric_Pad1.18x1.45mm_HandSolder, symbol Device:C
- added C89: 10u, Capacitor_SMD:C_0805_2012Metric_Pad1.18x1.45mm_HandSolder, symbol Device:C
- added C90: 100n, Capacitor_SMD:C_0603_1608Metric_Pad1.08x0.95mm_HandSolder, symbol Device:C
- added C91: 22u, Capacitor_Tantalum_SMD:CP_EIA-3216-18_Kemet-A_Pad1.58x1.35mm_HandSolder, symbol Device:C_Polarized
- added R91: 51, Resistor_SMD:R_0603_1608Metric_Pad0.98x0.95mm_HandSolder, symbol Device:R
- added U14: LP2985-3.3, Package_TO_SOT_SMD:SOT-23-5_HandSoldering, symbol Regulator_Linear:LP2985-3.3
- C14: renamed from C11; value 10u -> 1u
- D1: value LED -> LED_Green
- D2: renamed from D6; value LED -> LED_Blue
- D3: renamed from D7; value LED -> LED_Red
- J5: renamed from J22; Desc Joystick_HDR -> JOY; p1 (none) -> U; p10 (none) -> GND; p2 (none) -> D; p3 (none) -> L; p4 (none) -> R; p5 (none) -> +5; p6 (none) -> F1; p7 (none) -> F2; p8 (none) -> GND; p9 (none) -> F3
- R45: renamed from R49; value 8.2k -> 4.7k
- R60: renamed from R50; value 8.2k -> 4.7k
- U10: renamed from U16; value 74LVC2G04 -> 74LVC2G04DB
- U13: renamed from U25; value 74LVC2G04 -> 74LVC2G04DB
- U5: renamed from U20; value 74LVC2G04 -> 74LVC2G04DB
- U8: renamed from U15; value 74LVC2G04 -> 74LVC2G04DB
- renumbered C17 to C1, C33 to C10, C22 to C11, C23 to C12, C12 to C13, C16 to C15, C13 to C16, C43 to C17, C24 to C19, C14 to C2, C27 to C20, C42 to C21, C4 to C22, C3 to C23, C9 to C24, C10 to C25, C8 to C26, C20 to C27, C19 to C28, C21 to C29, C15 to C3, C39 to C30, C86 to C31, C40 to C32, C41 to C33, C84 to C34, C68 to C35, C7 to C36, C5 to C37, C29 to C38, C28 to C39, C1 to C4, C6 to C40, C31 to C41, C91 to C42, C92 to C43, C30 to C44, C58 to C45, C59 to C46, C60 to C47, C62 to C48, C63 to C49, C2 to C5, C64 to C50, C66 to C51, C67 to C52, C69 to C53, C70 to C54, C71 to C55, C72 to C56, C73 to C57, C75 to C58, C76 to C59, C36 to C6, C89 to C60, C49 to C61, C50 to C62, C51 to C63, C53 to C64, C54 to C65, C55 to C66, C56 to C67, C57 to C68, C77 to C69, C37 to C7, C78 to C70, C79 to C71, C80 to C72, C81 to C73, C82 to C74, C25 to C75, C32 to C76, C35 to C77, C44 to C78, C45 to C79, C38 to C8, C46 to C80, C47 to C81, C48 to C82, C61 to C83, C88 to C84, C52 to C85, C83 to C86, C85 to C87, C87 to C88, C34 to C9, D3 to D4, D8 to D6, F2 to F1, F1 to F2, H3 to H2, H2 to H3, J18 to J1, J6 to J10, J10 to J11, J16 to J12, J5 to J14, J17 to J2, J1 to J3, J2 to J4, J3 to J6, J9 to J7, J4 to J8, J8 to J9, JP3 to JP1, Q6 to Q1, Q3 to Q2, Q1 to Q3, Q2 to Q4, R81 to R1, R33 to R10, R44 to R11, R48 to R12, R14 to R13, R25 to R14, R76 to R15, R21 to R16, R22 to R17, R23 to R18, R5 to R19, R82 to R2, R77 to R20, R2 to R21, R43 to R22, R13 to R23, R6 to R24, R87 to R25, R88 to R26, R1 to R27, R85 to R28, R86 to R29, R27 to R3, R12 to R30, R9 to R31, R8 to R32, R34 to R33, R37 to R34, R10 to R35, R55 to R36, R52 to R37, R58 to R38, R51 to R39, R29 to R4, R11 to R40, R54 to R41, R79 to R42, R83 to R43, R84 to R44, R71 to R46, R59 to R47, R60 to R48, R61 to R49, R30 to R5, R62 to R50, R63 to R51, R17 to R52, R56 to R53, R7 to R54, R15 to R55, R16 to R56, R80 to R57, R18 to R58, R57 to R59, R38 to R6, R72 to R61, R64 to R62, R69 to R63, R70 to R64, R26 to R65, R45 to R66, R3 to R67, R4 to R68, R98 to R69, R36 to R7, R97 to R70, R96 to R71, R68 to R72, R39 to R73, R40 to R74, R41 to R75, R78 to R76, R53 to R77, R32 to R78, R28 to R79, R46 to R8, R31 to R80, R24 to R81, R89 to R82, R90 to R83, R91 to R84, R73 to R85, R74 to R86, R93 to R87, R92 to R88, R75 to R89, R47 to R9, R94 to R90, SW3 to SW2, SW5 to SW3, SW6 to SW4, U11 to U1, U21 to U11, U1 to U12, U12 to U15, U6 to U16, U3 to U17, U13 to U18, U7 to U2, U8 to U20, U9 to U21, U14 to U22, U22 to U23, U4 to U24, U10 to U3, U5 to U4, U2 to U6, U23 to U7, U24 to U9, Y4 to Y2, Y2 to Y3, Y3 to Y4
Connections:
- net +3V3: no longer C69.1, C70.1, C71.1, C72.1, C73.1, C74.1, R19.2, U11.18 (VCCIO), U11.3 (VCCIO), U11.34 (VCCIO), U11.39 (VCCINT), U11.51 (VCCIO), U11.66 (VCCIO), U11.82 (VCCIO), U11.91 (VCCINT), U9.11 (VCCIO1), U9.14 (PD_N), U9.19 (VCC), U9.21 (VCC), U9.22 (VCCIO2)
- net +5V: now also C89.2, U14.1 (VIN), U14.3 (ON/~{OFF})
- net FT_SCK: now also R91.1; no longer U6.104 (IO)
- net GND: now also C89.1, C90.1, C91.2, U14.2 (GND)
- net +3V3_VIDEO renamed +3V3A_VDAC
- new net: C90.2, U14.4 (BP)
- new net: R91.2, U6.104 (IO)
- new net +3V3_VDAC: C69.1, C70.1, C71.1, C72.1, C73.1, C74.1, C91.1, R19.2, U11.18 (VCCIO), U11.3 (VCCIO), U11.34 (VCCIO), U11.39 (VCCINT), U11.51 (VCCIO), U11.66 (VCCIO), U11.82 (VCCIO), U11.91 (VCCINT), U14.5 (VOUT), U9.11 (VCCIO1), U9.14 (PD_N), U9.19 (VCC), U9.21 (VCC), U9.22 (VCCIO2)
Other:
- moved on the sheet: C17, C36, C37, C38, C39, C40, C41, C42, C43, C61, C62, C63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

Commit message: wip pcb rev.A
Parts:
- added F2: 0.2A, Fuse:Fuse_1812_4532Metric_Pad1.30x3.40mm_HandSolder, symbol Device:Polyfuse
- added R92: 0, Resistor_SMD:R_1206_3216Metric, symbol Device:R
- renumbered F2 to F3
Connections:
- net +5V: now also R92.1; no longer C31.2, C34.2, C36.2, C44.2, C45.2, C54.2, C55.2, C56.2, C57.2, C58.2, C59.2, R81.1, U19.14 (VDD), U2.1 (VCC), U2.25 (VCC), U2.6 (VCC), U20.3 (VI), U21.3 (VI), U22.1 (VIN), U22.3 (ON/~{OFF}), U3.1 (VCC), U3.25 (VCC), U3.6 (VCC), U4.2 (VDD), U4.7 (OE)
- net +5V_FUSE renamed +5V_FUSE1
- net +5V_FUSE1: no longer J3.4, JP1.2 (B), R1.2, R2.2
- new net +5V_2: C31.2, C34.2, C36.2, C44.2, C45.2, C54.2, C55.2, C56.2, C57.2, C58.2, C59.2, F2.1, R81.1, R92.2, U19.14 (VDD), U2.1 (VCC), U2.25 (VCC), U2.6 (VCC), U20.3 (VI), U21.3 (VI), U22.1 (VIN), U22.3 (ON/~{OFF}), U3.1 (VCC), U3.25 (VCC), U3.6 (VCC), U4.2 (VDD), U4.7 (OE)
- new net +5V_FUSE2: F2.2, J3.4, JP1.2 (B), R1.2, R2.2
Other:
- moved on the sheet: C10, C30, C31, C32, C33, C34, C35, C36, C37, C38, C39, C40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
