File: pcb_main/rev.A/zxevo1010_main.kicad_sch (KiCad schematic)
At the start: 249 parts, among them J1 XHP-2, SXH-002T-P0.6, J10 Conn_02x30_Row_Letter_First, J11 TE 041021-4, J12 MEM2055-00-190-01-A, J13 Conn_02x05_Odd_Even, J14 Conn_02x05_Odd_Even, J2 B2B-XH-A, J3 Mini-DIN-6, J4 USB_B_Micro, J5 Conn_02x05_Odd_Even, J6 Mini-DIN-6, J7 DB15_Female_HighDensity_Mount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, J8 PJ-320, J9 Conn_02x05_Odd_Even, Q1 BC847, Q2 BC856, Q3 BC856, Q4 BC856, SW1 PB05A, SW2 SW_Push, SW3 SW_Push, SW4 SW_Push, U1 CH340X, U10 74LVC2G04DB, U11 EPM3128ATC100, U12 29F040-K, U13 74LVC2G04DB, U14 LP2985-3.3, U15 LMV358IDR, U16 ATmega128, U17 Z84C0020FEC, U18 PCF8583T, U19 CD4069UBM, U2 HY5118160, U20 1117-3.3, U21 1117-2.5, U22 LP2985-3.3, U23 LP2985-3.3, U24 1117-3.3, U3 HY5118160, U4 ICS501, U5 74LVC2G04DB, U6 EP1K50QC208, U7 ADV7125-lqfp48, U8 74LVC2G04DB, U9 FT812, Y1 14 MHz, Y2 8 MHz, Y3 11.059 Mhz, Y4 32768 Hz

Commit message: wip pcb rev.A
Connections:
- net R10 renamed RD10
- net R11 renamed RD11
- net R12 renamed RD12
Changed lines of the file:
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@@
 		)
 	)
-	(label "R10"
+	(label "RD10"
 		(at 209.55 58.42 180)
 		(fields_autoplaced yes)
@@
 		)
 	)
-	(label "R12"
+	(label "RD12"
 		(at 209.55 63.5 180)
 		(fields_autoplaced yes)
@@
 		)
 	)
-	(label "R11"
+	(label "RD11"
 		(at 260.35 60.96 180)
 		(fields_autoplaced yes)
@@
 		)
 	)
-	(label "R11"
+	(label "RD11"
 		(at 142.24 219.71 180)
 		(fields_autoplaced yes)
@@
 		)
 	)
-	(label "R12"
+	(label "RD12"
 		(at 260.35 63.5 180)
 		(fields_autoplaced yes)
@@
 		)
 	)
-	(label "R11"
+	(label "RD11"
 		(at 209.55 60.96 180)
 		(fields_autoplaced yes)
@@
 		)
 	)
-	(label "R12"
+	(label "RD12"
 		(at 142.24 224.79 180)
 		(fields_autoplaced yes)
@@
 		)
 	)
-	(label "R10"
+	(label "RD10"
 		(at 260.35 58.42 180)
 		(fields_autoplaced yes)
@@
 		)
 	)
-	(label "R10"
+	(label "RD10"
 		(at 142.24 214.63 180)
 		(fields_autoplaced yes)

Commit message: wip pcb rev.A (almost done)
Parts:
- U10, U13, U5, U8: value 74LVC2G04DB -> SN74LVC2G04DBVR
Changed lines of the file:
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@@
 		(dnp no)
 		(property "Reference" "U8"
-			(at 254.762 146.304 0)
+			(at 261.62 150.876 0)
 			(effects
 				(font
@@
 			)
 		)
-		(property "Value" "74LVC2G04DB"
-			(at 255.016 148.336 0)
+		(property "Value" "SN74LVC2G04DBVR"
+			(at 261.874 152.908 0)
 			(effects
 				(font
@@
 			)
 		)
-		(property "Value" "74LVC2G04DB"
+		(property "Value" "SN74LVC2G04DBVR"
 			(at 420.116 462.026 0)
 			(effects
@@
 			)
 		)
-		(property "Value" "74LVC2G04DB"
+		(property "Value" "SN74LVC2G04DBVR"
 			(at 414.274 497.078 0)
 			(effects
@@
 		(dnp no)
 		(property "Reference" "U13"
-			(at 404.622 266.954 0)
+			(at 412.75 271.272 0)
 			(effects
 				(font
@@
 			)
 		)
-		(property "Value" "74LVC2G04DB"
-			(at 404.876 268.986 0)
+		(property "Value" "SN74LVC2G04DBVR"
+			(at 413.004 273.558 0)
 			(effects
 				(font
@@
 		(dnp no)
 		(property "Reference" "U5"
-			(at 254.762 125.984 0)
+			(at 261.62 130.556 0)
 			(effects
 				(font
@@
 			)
 		)
-		(property "Value" "74LVC2G04DB"
-			(at 255.016 128.016 0)
+		(property "Value" "SN74LVC2G04DBVR"
+			(at 261.874 132.588 0)
 			(effects
 				(font
@@
 			)
 		)
-		(property "Value" "74LVC2G04DB"
+		(property "Value" "SN74LVC2G04DBVR"
 			(at 420.116 477.266 0)
 			(effects
@@
 		(dnp no)
 		(property "Reference" "U5"
-			(at 254.762 186.944 0)
+			(at 261.62 191.516 0)
 			(effects
 				(font
@@
 			)
 		)
-		(property "Value" "74LVC2G04DB"
-			(at 255.016 188.976 0)
+		(property "Value" "SN74LVC2G04DBVR"
+			(at 261.874 193.548 0)
 			(effects
 				(font
@@
 		(dnp no)
 		(property "Reference" "U13"
-			(at 405.892 304.038 0)
+			(at 414.02 308.356 0)
 			(effects
 				(font
@@
 			)
 		)
-		(property "Value" "74LVC2G04DB"
-			(at 406.146 305.816 0)
+		(property "Value" "SN74LVC2G04DBVR"
+			(at 414.274 310.388 0)
 			(effects
 				(font
@@
 			)
 		)
-		(property "Value" "74LVC2G04DB"
+		(property "Value" "SN74LVC2G04DBVR"
 			(at 400.304 497.078 0)
 			(effects
@@
 			)
 		)
-		(property "Value" "74LVC2G04DB"
+		(property "Value" "SN74LVC2G04DBVR"
 			(at 442.214 497.078 0)
 			(effects
@@
 			)
 		)
-		(property "Value" "74LVC2G04DB"
+		(property "Value" "SN74LVC2G04DBVR"
 			(at 428.244 497.078 0)
 			(effects
@@
 		(dnp no)
 		(property "Reference" "U10"
-			(at 254.762 166.624 0)
+			(at 261.62 171.196 0)
 			(effects
 				(font
@@
 			)
 		)
-		(property "Value" "74LVC2G04DB"
-			(at 255.016 168.656 0)
+		(property "Value" "SN74LVC2G04DBVR"
+			(at 261.874 173.228 0)
 			(effects
 				(font

Commit message: wip pcb rev.A
Parts:
- C13, C16: value 10u -> 100u; footprint Capacitor_Tantalum_SMD:CP_EIA-3216-18_Kemet-A_Pad1.58x1.35mm_HandSolder -> Capacitor_Tantalum_SMD:CP_EIA-6032-28_Kemet-C_Pad2.25x2.35mm_HandSolder
- C32, C43: footprint Capacitor_SMD:CP_Elec_5x5.9 -> Capacitor_Tantalum_SMD:CP_EIA-6032-28_Kemet-C_Pad2.25x2.35mm_HandSolder
- C6: value 4.7u -> 100n
- R1, R11, R12, R2: value 4.7k -> 10k
- R19: value 530 -> 10k
- R36, R38: value 24k -> 47k
- R39, R53: value 47 -> 51
- R45, R60: value 4.7k -> 8.2k
- R51, R69, R70, R71: value 10k -> 1k
- R52, R58: value 24k -> 27k
- U12: value 29F040-K -> 29F040
- U14, U22, U23: ValueAlt (none) -> LD3985M33R
- U7: value ADV7125-lqfp48 -> ADV7125
Connections:
- net +2V5: now also R81.1
- net +5V_2: no longer R81.1
- net BEEP: now also U13.1
- net SPICK: now also R65.2
- net ~{BEEP}: no longer U13.1
- net ~{SPICS}: no longer R65.2
Other:
- note added: "Possible opamp replacements: - MCP6002T-I/SN - TP8542ARZ"
- note removed: "Possible opamp replacements: - MCP6002T-I/SN - TP8542ARZ - MC4558"
- moved on the sheet: C4, C5, J11, J12, R14, R53, R76, R77, R78, R79, R80, U10C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

Commit message: wip pcb rev.A
Parts:
- C37, C40, C90: value 100n -> 10n
Other:
- note added: "Possible opamp replacements: - AD8606ARZ - OPA2348AIDR - MCP6022T-I/SN - MCP6002T-I/SN - TP8606ARZ - TP8542ARZ"
- note removed: "Possible opamp replacements: - MCP6002T-I/SN - TP8542ARZ"
Changed lines of the file:
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@@
 		)
 	)
-	(text_box "        | IN Vpp | R kOhm | OUT Vpp\nBeeper  | 3.3    | 49     | 0.6\nFT812   | 3.3    | 30     | 0.9\nSAM2695 | 2.8    | 22     | 1.0\nVS1053b | 2.1    | 18     | 1.0\nNeoGS   | 5.9    | 47     | 1.0\nPSG     | 5.9    | 47     | 1.0"
+	(text_box "        | IN Vpp | R kOhm | OUT Vpp\nBeeper  | 3.3    | 49     | 0.6\nFT812   | 3.3    | 30     | 0.9\nSAM2695 | 2.8    | 22     | 1.0\nVS1053b | 2.1    | 18     | 1.0\nNeoGS   | 0.9    | 8.2    | 0.9\nPSG     | 0.9    | 8.2    | 0.9"
 		(exclude_from_sim no)
 		(at 542.29 299.72 0)
@@
 		)
 	)
-	(text "Possible opamp replacements:\n- MCP6002T-I/SN\n- TP8542ARZ"
+	(text "Possible opamp replacements:\n- AD8606ARZ\n- OPA2348AIDR\n- MCP6022T-I/SN\n- MCP6002T-I/SN\n- TP8606ARZ\n- TP8542ARZ"
 		(exclude_from_sim no)
-		(at 518.16 257.048 0)
+		(at 524.51 254.508 0)
 		(effects
 			(font
@@
 		(dnp no)
 		(property "Reference" "R74"
-			(at 382.7781 375.1591 0)
+			(at 382.778 374.65 0)
 			(effects
 				(font
@@
 		)
 		(property "Value" "10k"
-			(at 382.7781 377.4578 0)
+			(at 382.778 376.9487 0)
 			(effects
 				(font
@@
 			)
 		)
-		(property "Value" "100n"
+		(property "Value" "10n"
 			(at 209.55 491.49 0)
 			(effects
@@
 			)
 		)
-		(property "Value" "100n"
+		(property "Value" "10n"
 			(at 257.81 491.49 0)
 			(effects
@@
 			)
 		)
-		(property "Value" "100n"
+		(property "Value" "10n"
 			(at 161.29 491.49 0)
 			(effects
@@
 		(dnp no)
 		(property "Reference" "R75"
-			(at 390.3981 375.1591 0)
+			(at 390.398 374.65 0)
 			(effects
 				(font
@@
 		)
 		(property "Value" "10k"
-			(at 390.3981 377.4578 0)
+			(at 390.398 376.9487 0)
 			(effects
 				(font
@@
 		(dnp no)
 		(property "Reference" "R73"
-			(at 375.1581 375.1591 0)
+			(at 375.158 374.65 0)
 			(effects
 				(font
@@
 		)
 		(property "Value" "10k"
-			(at 375.1581 377.4578 0)
+			(at 375.158 376.9487 0)
 			(effects
 				(font

Commit message: wip pcb rev.A
Parts:
- Y3: value 11.059 Mhz -> 11.059 MHz
Changed lines of the file:
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@@
 			)
 		)
-		(property "Value" "11.059 Mhz"
+		(property "Value" "11.059 MHz"
 			(at 52.07 303.53 0)
 			(effects

Commit message: pcb rev.A final versions
Parts:
- added R93, R94: 5.1k, Resistor_SMD:R_0603_1608Metric_Pad0.98x0.95mm_HandSolder, symbol Device:R
- C37, C40, C90: now not fitted
- J4: value USB_B_Micro -> USB Type C; footprint Connector_USB:USB_Micro-B_Molex-105017-0001 -> my:USB_C_Receptacle_HRO_TYPE-C-31-M-12_dangling; symbol Connector:USB_B_Micro -> Connector:USB_C_Receptacle_USB2.0_16P
- J8: value PJ-320 -> PJ-322; footprint my:PJ-320A_D -> my:PJ-322
- SW1: value PB05A -> RWB-101
- SW2, SW3, SW4: value SW_Push -> Push angle button, 6x6x7mm or 6x6x8mm
- U14, U22, U23: value LP2985-3.3 -> TPS7A2033PDBVR; ValueAlt LD3985M33R -> NCP114ASN330T1G, LP2985-3.3, LD3985M33R
Connections:
- net GND: now also J4.A1 (GND), J4.A12 (GND), J4.B1 (GND), J4.B12 (GND), J4.S1 (SHIELD), R93.1, R94.1; no longer J4.5 (GND), J4.6 (Shield)
- net UDN: now also J4.A7 (D-), J4.B7 (D-); no longer J4.2 (D-)
- net UDP: now also J4.A6 (D+), J4.B6 (D+); no longer J4.3 (D+)
- net at J2.2 (Pin_2): now also J4.A4 (VBUS), J4.A9 (VBUS), J4.B4 (VBUS), J4.B9 (VBUS); no longer J4.1 (VBUS)
- new net: J4.A5 (CC1), R93.2
- new net: J4.B5 (CC2), R94.2
- no-connect marks 91 -> 92
Other:
- moved on the sheet: C1, J2, U1
