File: pcb_top/rev.A/zxevo1010_top.kicad_pcb (KiCad board)
At the start: 2 copper layers, 100 x 80.8 mm, 91 parts, among them J1 Conn_01x04, J6 Conn_02x30_Row_Letter_First, U1 ESP-12E, U12 YM2203, U13 YM3014B, U14 YM2203, U15 YM3014B, U16 LMV358IDR, U17 LMV358IDR, U2 CY62167ELL, U3 EPM3256ATC144, U4 Z84C0020FEC, U5 SAM2695, U6 27C512, U7 74HCT245D, U8 74AHCT1G125DB, U9 LMV358IDR

Commit message: wip pcbs rev.A
Parts:
- removed C14, C21: 10u, Capacitor_SMD:CP_Elec_4x5.4
- removed C15: 100n, Capacitor_SMD:C_0603_1608Metric_Pad1.08x0.95mm_HandSolder
- removed R14: 27k, Resistor_SMD:R_0603_1608Metric_Pad0.98x0.95mm_HandSolder
- removed R18, R26: 10k, Resistor_SMD:R_0603_1608Metric_Pad0.98x0.95mm_HandSolder
- removed R19: 10K, Resistor_SMD:R_0603_1608Metric_Pad0.98x0.95mm_HandSolder
- removed U9: LMV358IDR, Package_SO:SOIC-8_3.9x4.9mm_P1.27mm
- added J2: Conn_02x05_Odd_Even, Connector_PinHeader_2.54mm:PinHeader_2x05_P2.54mm_Vertical, B.Cu at (103.9, 92.8)
- added Q1: BSS138, Package_TO_SOT_SMD:SOT-23, F.Cu at (68.7, 108.8)
- added R7: 10k, Resistor_SMD:R_0603_1608Metric_Pad0.98x0.95mm_HandSolder, F.Cu at (64.0, 107.7)
- J1: value Conn_01x04 -> Conn_02x05_Odd_Even; footprint Connector_PinHeader_2.54mm:PinHeader_1x04_P2.54mm_Vertical -> Connector_PinHeader_2.54mm:PinHeader_2x04_P2.54mm_Vertical
- R11: value 47k -> 4.7k
- moved R11 8.24 mm to (64.0, 110.2)
- moved J1 3.34 mm to (103.9, 61.8)
Connections:
- J1 pad 1: /SND_L -> /TAPE_OUT
- J1 pad 2: GNDA -> /MIXER_L
- J1 pad 4: /SND_R -> GNDA
- R10 pad 1: Net-(U9A--) -> /MIXER_L
- R11 pad 1: Net-(U9A-+) -> Net-(Q1-S)
- R11 pad 2: unconnected-(R11-Pad2) -> +3V3_2
- R12 pad 1: Net-(U9A--) -> /MIXER_L
- R13 pad 1: Net-(U9A--) -> /MIXER_L
- R15 pad 1: Net-(U9A--) -> /MIXER_L
- R17 pad 1: Net-(U9A--) -> /MIXER_L
- R20 pad 1: Net-(U9A--) -> /MIXER_L
- R21 pad 1: Net-(U9A--) -> /MIXER_L
- R22 pad 1: Net-(U9A--) -> /MIXER_L
- R23 pad 1: Net-(U9B--) -> /MIXER_R
- R25 pad 1: Net-(U9B--) -> /MIXER_R
- R27 pad 1: Net-(U9B--) -> /MIXER_R
- R28 pad 1: Net-(U9B--) -> /MIXER_R
- R29 pad 1: Net-(U9B--) -> /MIXER_R
- R30 pad 1: Net-(U9B--) -> /MIXER_R
- R31 pad 1: Net-(U9B--) -> /MIXER_R
- R32 pad 1: Net-(U9B--) -> /MIXER_R
- R34 pad 1: Net-(U9B--) -> /MIXER_R
- R8 pad 1: Net-(U9A--) -> /MIXER_L
- U1 pad 21: /ESP_RX -> Net-(Q1-S)
- U1 pad 7: /ESP_CTS -> Net-(U1-GPIO13)

Commit message: wip pcb rev.A
Parts:
- removed C30: 10u, Capacitor_SMD:CP_Elec_4x5.4
- removed C32: 100n, Capacitor_SMD:C_0603_1608Metric_Pad1.08x0.95mm_HandSolder
- added C14: 10u, Capacitor_SMD:C_0805_2012Metric_Pad1.18x1.45mm_HandSolder, B.Cu at (212.3, 72.6)
- added C15: 22u, Capacitor_Tantalum_SMD:CP_EIA-3216-18_Kemet-A_Pad1.58x1.35mm_HandSolder, B.Cu at (212.7, 95.2)
- added C21: 22u, Capacitor_Tantalum_SMD:CP_EIA-3216-18_Kemet-A_Pad1.58x1.35mm_HandSolder, B.Cu at (212.7, 70.3)
- added D1: LED, LED_SMD:LED_0603_1608Metric_Pad1.05x0.95mm_HandSolder, F.Cu at (180.8, 114.8)
- added J3: Conn_02x05_Odd_Even, Connector_PinHeader_2.54mm:PinHeader_2x05_P2.54mm_Vertical, F.Cu at (100.9, 72.5)
- added J4: PJ-320, my:PJ-320A_D, F.Cu at (127.0, 52.0)
- added JP2: SolderJumper_2_Bridged, Jumper:SolderJumper-2_P1.3mm_Bridged_RoundedPad1.0x1.5mm, F.Cu at (215.9, 134.7)
- added R14: 51, Resistor_SMD:R_0603_1608Metric_Pad0.98x0.95mm_HandSolder, B.Cu at (141.0, 120.9)
- added R16: 6.8k, Resistor_SMD:R_0603_1608Metric_Pad0.98x0.95mm_HandSolder, B.Cu at (163.6, 122.5)
- added R18: 6.8k, Resistor_SMD:R_0603_1608Metric_Pad0.98x0.95mm_HandSolder, B.Cu at (160.2, 122.5)
- added R19: 51, Resistor_SMD:R_0603_1608Metric_Pad0.98x0.95mm_HandSolder, B.Cu at (141.0, 116.4)
- added R24: 6.8k, Resistor_SMD:R_0603_1608Metric_Pad0.98x0.95mm_HandSolder, B.Cu at (105.3, 77.6)
- added R26: 6.8k, Resistor_SMD:R_0603_1608Metric_Pad0.98x0.95mm_HandSolder, B.Cu at (105.3, 81.0)
- added R35: 10k, Resistor_SMD:R_0603_1608Metric_Pad0.98x0.95mm_HandSolder, B.Cu at (105.3, 74.2)
- added R44: 6.8k, Resistor_SMD:R_0603_1608Metric_Pad0.98x0.95mm_HandSolder, B.Cu at (150.7, 142.9)
- added R45: 1K, Resistor_SMD:R_0603_1608Metric_Pad0.98x0.95mm_HandSolder, B.Cu at (154.9, 117.8)
- added R46: 6.8k, Resistor_SMD:R_0603_1608Metric_Pad0.98x0.95mm_HandSolder, B.Cu at (169.2, 122.5)
- added R47: 6.8k, Resistor_SMD:R_0603_1608Metric_Pad0.98x0.95mm_HandSolder, B.Cu at (172.6, 122.5)
- added R48: 51, Resistor_SMD:R_0603_1608Metric_Pad0.98x0.95mm_HandSolder, B.Cu at (112.7, 113.3)
- added R49: 51, Resistor_SMD:R_0603_1608Metric_Pad0.98x0.95mm_HandSolder, B.Cu at (120.5, 113.3)
- added R50: 51, Resistor_SMD:R_0603_1608Metric_Pad0.98x0.95mm_HandSolder, B.Cu at (119.0, 113.3)
- added R51: 51, Resistor_SMD:R_0603_1608Metric_Pad0.98x0.95mm_HandSolder, B.Cu at (141.0, 119.4)
- added R52: 51, Resistor_SMD:R_0603_1608Metric_Pad0.98x0.95mm_HandSolder, B.Cu at (141.0, 117.8)
- added R53: 6.8k, Resistor_SMD:R_0603_1608Metric_Pad0.98x0.95mm_HandSolder, B.Cu at (215.4, 116.3)
- added R54: 6.8k, Resistor_SMD:R_0603_1608Metric_Pad0.98x0.95mm_HandSolder, B.Cu at (215.4, 111.8)
- added R55: 6.8k, Resistor_SMD:R_0603_1608Metric_Pad0.98x0.95mm_HandSolder, B.Cu at (215.4, 124.7)
- added R56: 6.8k, Resistor_SMD:R_0603_1608Metric_Pad0.98x0.95mm_HandSolder, B.Cu at (215.4, 120.5)
- added R57: 1k, Resistor_SMD:R_0603_1608Metric_Pad0.98x0.95mm_HandSolder, B.Cu at (174.6, 131.4)
- added R58: 6.8k, Resistor_SMD:R_0603_1608Metric_Pad0.98x0.95mm_HandSolder, B.Cu at (122.2, 95.7)
- added R59: 1M, Resistor_SMD:R_0603_1608Metric_Pad0.98x0.95mm_HandSolder, B.Cu at (118.3, 107.6)
- added R63: 3.3k, Resistor_SMD:R_0805_2012Metric_Pad1.20x1.40mm_HandSolder, B.Cu at (114.1, 84.0)
- added U10: EPM3064ATC100, Package_QFP:TQFP-100_14x14mm_P0.5mm, F.Cu at (137.9, 107.5)
- added U11: EP1K30TC144, Package_QFP:TQFP-144_20x20mm_P0.5mm, F.Cu at (166.9, 110.5)
- added U18: MAX809LEUR, Package_TO_SOT_SMD:SOT-23, F.Cu at (215.9, 131.3)
- added U19: TDA1543T, Package_SO:SOIC-16W_7.5x10.3mm_P1.27mm, F.Cu at (119.3, 82.6)
- added U20: ESP32-WROOM-32, RF_Module:ESP32-WROOM-32, F.Cu at (116.1, 163.8)
- added U21: 74ACT245, Package_SO:TSSOP-20_4.4x6.5mm_P0.65mm, F.Cu at (184.5, 100.0)
- added U22: 74LXC245, Package_SO:TSSOP-20_4.4x6.5mm_P0.65mm, F.Cu at (149.5, 119.8)
- added U23: MA8201, Package_QFP:MQFP-44_10x10mm_P0.8mm, F.Cu at (118.3, 97.3)
- added U24: EPM3064ATC100, Package_QFP:TQFP-100_14x14mm_P0.5mm, F.Cu at (178.9, 73.5)
- added U25: 1117-3.3, Package_TO_SOT_SMD:SOT-223-3_TabPin2, F.Cu at (214.4, 70.3)
- added U26: 1117-2.5, Package_TO_SOT_SMD:SOT-223-3_TabPin2, F.Cu at (214.4, 78.6)
- added U27: 1117-3.3, Package_TO_SOT_SMD:SOT-223-3_TabPin2, F.Cu at (214.4, 86.9)
- added U28: 1117-1.8, Package_TO_SOT_SMD:SOT-223-3_TabPin2, F.Cu at (214.4, 95.2)
- added U9: VS1053b, Package_QFP:LQFP-48_7x7mm_P0.5mm, F.Cu at (118.3, 97.3)
- added X1: 20 MHz, my:Oscillator_SMD_7050_7.0x5.0mm, F.Cu at (114.8, 116.8)
- added X2: 24 MHz, my:Oscillator_SMD_7050_7.0x5.0mm, F.Cu at (121.9, 116.8)
- added Y1: 12 MHz, Crystal:Crystal_SMD_SeikoEpson_TSX3225-4Pin_3.2x2.5mm_HandSoldering, F.Cu at (134.6, 69.5)
- added Y2: 14 MHz, Crystal:Crystal_SMD_SeikoEpson_TSX3225-4Pin_3.2x2.5mm_HandSoldering, F.Cu at (118.3, 107.6)
- C1, C3: value 10n -> 100n; moved to B.Cu
- C10, C31: footprint Capacitor_SMD:CP_Elec_4x5.4 -> Capacitor_SMD:C_0805_2012Metric_Pad1.18x1.45mm_HandSolder; moved to B.Cu
- C11, C12, C13, C16, C17, C18, C19, C20, C22, C23, C24, C25, C27, C9: footprint Capacitor_SMD:CP_Elec_4x5.4 -> Capacitor_Tantalum_SMD:CP_EIA-3216-18_Kemet-A_Pad1.58x1.35mm_HandSolder
- C2, C4: value 10n -> 10u; footprint Capacitor_SMD:C_0603_1608Metric_Pad1.08x0.95mm_HandSolder -> Capacitor_SMD:C_0805_2012Metric_Pad1.18x1.45mm_HandSolder; moved to B.Cu
- C26: value 10u -> 100n; footprint Capacitor_SMD:CP_Elec_4x5.4 -> Capacitor_SMD:C_0805_2012Metric_Pad1.18x1.45mm_HandSolder; moved to B.Cu
- C28: value 100n -> 10u; footprint Capacitor_SMD:C_0603_1608Metric_Pad1.08x0.95mm_HandSolder -> Capacitor_SMD:C_0805_2012Metric_Pad1.18x1.45mm_HandSolder; moved to B.Cu
- C29, C33: value 2.2n -> 22u; footprint Capacitor_SMD:C_0603_1608Metric_Pad1.08x0.95mm_HandSolder -> Capacitor_Tantalum_SMD:CP_EIA-3216-18_Kemet-A_Pad1.58x1.35mm_HandSolder; moved to B.Cu
- C5: value 100n -> 22p
- C6: value 10u -> 22p; footprint Capacitor_SMD:C_0805_2012Metric_Pad1.18x1.45mm_HandSolder -> Capacitor_SMD:C_0603_1608Metric_Pad1.08x0.95mm_HandSolder
- C7: value 100n -> 33p
- C8: value 10u -> 33p; footprint Capacitor_SMD:C_0805_2012Metric_Pad1.18x1.45mm_HandSolder -> Capacitor_SMD:C_0603_1608Metric_Pad1.08x0.95mm_HandSolder
- J1: footprint Connector_PinHeader_2.54mm:PinHeader_2x04_P2.54mm_Vertical -> Connector_PinSocket_2.54mm:PinSocket_2x03_P2.54mm_Vertical
- J2: footprint Connector_PinHeader_2.54mm:PinHeader_2x05_P2.54mm_Vertical -> Connector_PinSocket_2.54mm:PinSocket_2x03_P2.54mm_Vertical
- Q1, R1, R10, R11, R12, R13, R15, R17, R2, R20, R21, R22, R23, R25, R27, R28, R29, R30, R31, R32, R34, R7, R8: moved to B.Cu
- R3, R4, R43, R5, R6: value 1k -> 6.8k; moved to B.Cu
- R33, R36, R9: value 3.3k -> 6.8k; moved to B.Cu
- R37: value 470 -> 1k; moved to B.Cu
- R38: value 1k -> 100; moved to B.Cu
- R39, R40, R41: value 3.3k -> 1k; moved to B.Cu
- R42: value 470 -> 6.8k; moved to B.Cu
- U12, U14: value YM2203 -> 74AHCT1G125DB; footprint Package_DIP:DIP-40_W15.24mm_Socket -> Package_TO_SOT_SMD:SOT-23-5_HandSoldering
- U13: value YM3014B -> 74AHCT1G125DB; footprint Package_DIP:DIP-8_W7.62mm_Socket -> Package_TO_SOT_SMD:SOT-23-5_HandSoldering
- U15: value YM3014B -> YMF288-M; footprint Package_DIP:DIP-8_W7.62mm_Socket -> Package_SO:SOP-28_8.4x18.16mm_P1.27mm
- U16: value LMV358IDR -> YMF288-M; footprint Package_SO:SOIC-8_3.9x4.9mm_P1.27mm -> Package_SO:SOP-28_8.4x18.16mm_P1.27mm
- U17: value LMV358IDR -> TDA1543; footprint Package_SO:SOIC-8_3.9x4.9mm_P1.27mm -> Package_DIP:DIP-8_W7.62mm
- U2: value CY62167ELL -> CY62167EV30LL-45ZXI
- U3: value EPM3256ATC144 -> CY62167EV30LL-45ZXI; footprint PCM_Package_QFP_AKL:TQFP-144_20x20mm_P0.5mm -> Package_SO:TSOP-I-48_18.4x12mm_P0.5mm
- U6: value 27C512 -> 29F040
- U7: value 74HCT245D -> 74LVC1G04DB; footprint Package_SO:SOIC-20W_7.5x12.8mm_P1.27mm -> Package_TO_SOT_SMD:SOT-23-5_HandSoldering
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Connections:
- net /~{RFSH} renamed /~{ZXRFSH}
- C1 pad 1: /DACCH3 -> GND
- C1 pad 2: GNDA -> Net-(U5-VCM)
- C10 pad 1: Net-(U13-Mp) -> GND
- C10 pad 2: GNDA -> +5V
- C2 pad 1: /DACCH2 -> GND
- C2 pad 2: GNDA -> Net-(U5-VCM)
- C26 pad 1: Net-(U13-Rb) -> /MA_RCAP
- C28 pad 1: Net-(U13-Rb) -> GND
- C28 pad 2: GNDA -> +5V
- C29 pad 1: Net-(U13-ToBUFF) -> +2V5
- C29 pad 2: GNDA -> GND
- C3 pad 1: /DACCH1 -> GND
- C3 pad 2: GNDA -> Net-(U5-OUTVC12)
- C31 pad 1: Net-(U15-Rb) -> GND
- C31 pad 2: GNDA -> +5V
- C33 pad 1: Net-(U15-ToBUFF) -> +3V3_MIDI
- C33 pad 2: GNDA -> GND
- C4 pad 1: /DACCH0 -> GND
- C4 pad 2: GNDA -> Net-(U5-OUTVC12)
- C5 pad 1: Net-(U5-VCM) -> GND
- C5 pad 2: GNDA -> Net-(U5-X2)
- C6 pad 1: Net-(U5-VCM) -> GND
- C6 pad 2: GNDA -> Net-(U5-X1)
- C7 pad 1: Net-(U5-OUTVC12) -> GND
- C7 pad 2: GNDA -> /MA_XTALI
- C8 pad 1: Net-(U5-OUTVC12) -> GND
- C8 pad 2: GNDA -> /MA_XTALO
- J1 pad 5: GNDA -> /TAPE_IN
- J1 pad 6: GNDA -> /MIXER_R
- J2 pad 1: unconnected-(J2-Pin_1-Pad1) -> /ESP_RX
- J2 pad 2: GND -> +5V
- J2 pad 3: /ESP_RX -> unconnected-(J2-Pin_3-Pad3)
- J2 pad 4: +5V -> /ESP_TX
- J2 pad 6: unconnected-(J2-Pin_6-Pad6) -> GND
- J6 pad 1: /A14 -> /ZXA14
- J6 pad 12: /D0 -> /ZXD0
- J6 pad 14: /D1 -> /ZXD1
- J6 pad 16: /D2 -> /ZXD2
- J6 pad 17: /A0 -> /ZXA0
- J6 pad 18: /D6 -> /ZXD6
- J6 pad 19: /A1 -> /ZXA1
- J6 pad 2: /A15 -> /ZXA15
- J6 pad 20: /D5 -> /ZXD5
- J6 pad 21: /A2 -> /ZXA2
- J6 pad 22: /D3 -> /ZXD3
- J6 pad 23: /A3 -> /ZXA3
- J6 pad 24: /D4 -> /ZXD4
- J6 pad 25: /~{IORQGE1} -> /ZXIORQGE
- J6 pad 26: /~{INT} -> unconnected-(J6-Pin_26-Pad26)
- J6 pad 28: /~{NMI} -> unconnected-(J6-Pin_28-Pad28)
- J6 pad 29: /~{RDROM} -> /~{ZXRDROM}
- J6 pad 3: /A12 -> /ZXA12
- J6 pad 30: /~{HALT} -> unconnected-(J6-Pin_30-Pad30)
- J6 pad 32: /~{MREQ} -> /~{ZXMREQ}
- J6 pad 34: /~{IORQ1} -> /~{ZXIORQ}
- J6 pad 36: /~{RD} -> /~{ZXRD}
- J6 pad 37: /~{BUSR} -> unconnected-(J6-Pin_37-Pad37)
- J6 pad 38: /~{WR} -> /~{ZXWR}
- J6 pad 39: /~{RES} -> /~{ZXRES}
- J6 pad 4: /A13 -> /ZXA13
- J6 pad 41: /A7 -> /ZXA7
- J6 pad 42: /~{WAIT} -> /~{ZXWAIT}
- J6 pad 43: /A6 -> /ZXA6
- J6 pad 45: /A5 -> /ZXA5
- J6 pad 47: /A4 -> /ZXA4
- J6 pad 48: /~{M1} -> /~{ZXM1}
- J6 pad 49: /~{CSROM} -> /~{ZXCSROM}
- J6 pad 51: /~{BUSA} -> unconnected-(J6-Pin_51-Pad51)
- J6 pad 52: /A8 -> /ZXA8
- J6 pad 53: /A9 -> /ZXA9
- J6 pad 54: /A10 -> /ZXA10
- J6 pad 55: /A11 -> /ZXA11
- J6 pad 6: /D7 -> /ZXD7
- J6 pad 7: /~{DOS} -> unconnected-(J6-Pin_7-Pad7)
- Q1 pad 1: +3V3_2 -> +3V3
- R1 pad 2: +3V3_2 -> +3V3
- R11 pad 2: +3V3_2 -> +3V3
- R3 pad 1: /DACCH3 -> /~{NMI}
- R3 pad 2: Net-(U7-B0) -> +3V3
- R33 pad 1: GNDA -> /~{RD}
- R33 pad 2: /AY_B1 -> +5V
- R36 pad 1: GNDA -> /~{BUSRQ}
- R36 pad 2: /AY_A1 -> +3V3
- R37 pad 1: Net-(U16A--) -> /CONF_DONE
- R37 pad 2: Net-(U13-Mp) -> +3V3
- R38 pad 1: Net-(U12-OP-O) -> Net-(D1-A)
- R38 pad 2: /FM1_ENA -> +3V3
- R39 pad 1: GNDA -> /INIT_DONE
- R39 pad 2: /AY_C2 -> +3V3
- R4 pad 1: /DACCH2 -> /~{INT}
- R4 pad 2: Net-(U7-B2) -> +3V3
- R40 pad 1: GNDA -> /~{STATUS}
- R40 pad 2: /AY_B2 -> +3V3
- R41 pad 1: GNDA -> GND
- R41 pad 2: /AY_A2 -> /MEMA21
- R42 pad 1: Net-(U17A--) -> /MEMA18
- R42 pad 2: Net-(U15-Mp) -> +3V3
- R43 pad 1: Net-(U14-OP-O) -> /MEMA17
- R43 pad 2: /FM2_ENA -> +3V3
- R5 pad 1: /DACCH1 -> /~{MREQ}
- R5 pad 2: Net-(U7-B4) -> +5V
- R6 pad 1: /DACCH0 -> /~{IORQ}
- R6 pad 2: Net-(U7-B6) -> +5V
- R9 pad 1: GNDA -> /~{WR}
- R9 pad 2: /AY_C1 -> +5V
- U1 pad 3: +3V3_2 -> +3V3
- U1 pad 8: +3V3_2 -> +3V3
- U12 pad 1: GNDA -> /~{ZXBLKROM}
- U12 pad 2: /AD1 -> +5V
- U12 pad 3: /AD2 -> GND
- U12 pad 4: /AD3 -> /~{ZXRDROM}
- U12 pad 5: /AD4 -> +5V
- U13 pad 1: +5VA_1 -> /~{ZXGENWAIT}
- U13 pad 2: Net-(U13-ToBUFF) -> GND
- U13 pad 3: Net-(U12-SH) -> GND
- U13 pad 4: /FM1_ENA -> /~{ZXWAIT}
- U13 pad 5: Net-(U12-S) -> +5V
- U14 pad 1: GNDA -> /~{WARMRES}
- U14 pad 2: /AD1 -> GND
- U14 pad 3: /AD2 -> GND
- U14 pad 4: /AD3 -> /~{Z80RES}
- U14 pad 5: /AD4 -> +5V
- U15 pad 1: +5VA_2 -> GND
- U15 pad 2: Net-(U15-ToBUFF) -> /YMD0
- U15 pad 3: Net-(U14-SH) -> /YMD1
- U15 pad 4: /FM2_ENA -> /YMD2
- U15 pad 5: Net-(U14-S) -> /YMD3
- U15 pad 6: GNDA -> /YMD4
- U15 pad 7: Net-(U15-Rb) -> /YMD5
- U15 pad 8: Net-(U15-Mp) -> /YMD6
- U16 pad 1: Net-(U16A--) -> GND
- U16 pad 2: Net-(U16A--) -> /YMD0
- U16 pad 3: Net-(U13-Rb) -> /YMD1
- U16 pad 4: GNDA -> /YMD2
- U16 pad 5: Net-(U13-ToBUFF) -> /YMD3
- U16 pad 6: /FM1 -> /YMD4
- U16 pad 7: /FM1 -> /YMD5
- U16 pad 8: +5VA -> /YMD6
- U17 pad 1: Net-(U17A--) -> /DAC_BITCK
- U17 pad 2: Net-(U17A--) -> /DAC_LRCK
- U17 pad 3: Net-(U15-Rb) -> /DAC_DAT
- U17 pad 5: Net-(U15-ToBUFF) -> unconnected-(U17-VDD-Pad5)
- U17 pad 6: /FM2 -> /DAC_AOL
- U17 pad 7: /FM2 -> /DAC_VREF
- U17 pad 8: +5VA -> /DAC_AOR
- U2 pad 1: /GMA15 -> /MEMA15
- U2 pad 11: /~{GWR} -> /~{MEMWE}
- U2 pad 12: +5V -> +3V3
- U2 pad 16: /GMA17 -> /MEMA18
- U2 pad 17: /GMA18 -> /MEMA17
- U2 pad 18: /GA0 -> /RA7
- U2 pad 19: /GA1 -> /RA6
- U2 pad 2: /GA7 -> /MEMA14
- U2 pad 20: /GA2 -> /RA5
- U2 pad 21: /GA3 -> /RA4
- U2 pad 22: /GA4 -> /RA3
- U2 pad 23: /GA5 -> /RA2
- U2 pad 24: /GA6 -> /RA1
- U2 pad 25: /GA13 -> /RA0
- U2 pad 26: /~{GRAM2} -> /~{OUT_RAMCS0}
- U2 pad 28: /~{GRD} -> /~{MEMOE}
- U2 pad 29: /GD5 -> /RD0
- U2 pad 3: /GA14 -> /RA13
- U2 pad 31: /GD3 -> /RD1
- U2 pad 33: /GD1 -> /RD2
- U2 pad 35: /GD0 -> /RD3
- U2 pad 37: +5V -> +3V3
- U2 pad 38: /GD2 -> /RD4
- U2 pad 4: /GA12 -> /RA12
- U2 pad 40: /GD4 -> /RD5
- U2 pad 42: /GD6 -> /RD6
- U2 pad 44: /GD7 -> /RD7
- U2 pad 45: unconnected-(U2-A20/D15-Pad45) -> /MEMA21
- U2 pad 48: /GMA16 -> /MEMA16
- U2 pad 5: /GA11 -> /RA11
- U2 pad 6: /GA10 -> /RA10
- U2 pad 7: /GA9 -> /RA9
- U2 pad 8: /GA8 -> /RA8
- U2 pad 9: unconnected-(U2-A19-Pad9) -> /MEMA19
- U3 pad 1: unconnected-(U3-IO-Pad1) -> /MEMA15
- U3 pad 10: /~{GRST} -> unconnected-(U3-NC-Pad10)
- U3 pad 11: /GA0 -> /~{MEMWE}
- U3 pad 12: /GA1 -> +3V3
- U3 pad 13: GND -> unconnected-(U3-NC-Pad13)
- U3 pad 14: /GA2 -> unconnected-(U3-~{BHE}-Pad14)
- U3 pad 15: /GA3 -> unconnected-(U3-~{BLE}-Pad15)
- U3 pad 16: /GA4 -> /MEMA18
- U3 pad 17: GND -> /MEMA17
- U3 pad 18: /GA5 -> /RA7
- U3 pad 19: /GA6 -> /RA6
- U3 pad 2: /~{GRAM2} -> /MEMA14
- U3 pad 20: /TMS -> /RA5
- U3 pad 21: /GA7 -> /RA4
- U3 pad 22: /GA8 -> /RA3
- U3 pad 23: /GA9 -> /RA2
- U3 pad 24: +3V3 -> /RA1
- U3 pad 25: /GA10 -> /RA0
- U3 pad 26: GND -> /~{OUT_RAMCS1}
- U3 pad 27: /~{GWR} -> GND
- U3 pad 28: /~{GRD} -> /~{MEMOE}
- U3 pad 29: /~{GIORQ} -> /RD0
- U3 pad 3: GND -> /RA13
- U3 pad 30: /~{GMREQ} -> unconnected-(U3-D8-Pad30)
- U3 pad 31: /GA11 -> /RD1
- U3 pad 32: /GA12 -> unconnected-(U3-D9-Pad32)
- U3 pad 33: GND -> /RD2
- U3 pad 34: /GA13 -> unconnected-(U3-D10-Pad34)
- U3 pad 35: /GA14 -> /RD3
- U3 pad 36: /GA15 -> unconnected-(U3-D11-Pad36)
- U3 pad 37: /GD3 -> +3V3
- U3 pad 38: /GD5 -> /RD4
- U3 pad 39: /GD6 -> unconnected-(U3-D12-Pad39)
- U3 pad 4: /TDI -> /RA12
- U3 pad 40: /GD2 -> /RD5
- U3 pad 41: /GD7 -> unconnected-(U3-D13-Pad41)
- U3 pad 42: /GD4 -> /RD6
- U3 pad 43: /GCLK -> unconnected-(U3-D14-Pad43)
- U3 pad 44: /~{GINT} -> /RD7
- U3 pad 45: /GD0 -> /MEMA21
- U3 pad 46: /GD1 -> GND
- U3 pad 47: /~{GROM} -> GND
- U3 pad 48: /GMA15 -> /MEMA16
- U3 pad 5: /GMA17 -> /RA11
- U3 pad 6: /GMA16 -> /RA10
- U3 pad 7: /GMA18 -> /RA9
- U3 pad 8: /~{GRAM1} -> /RA8
- U3 pad 9: /~{GM1} -> /MEMA19
- U4 pad 1: /GCLK_BUF -> /CLK_Z80
- U4 pad 10: /GD1 -> /D1
- U4 pad 12: /~{GINT} -> /~{INT}
- U4 pad 13: +5V -> /~{NMI}
- U4 pad 15: /~{GMREQ} -> /~{MREQ}
- U4 pad 16: /~{GIORQ} -> /~{IORQ}
- U4 pad 18: /~{GRD} -> /~{RD}
- U4 pad 19: /~{GWR} -> /~{WR}
- U4 pad 2: /GD4 -> /D4
- U4 pad 20: unconnected-(U4-~{BUSACK}-Pad20) -> /~{BUSAK}
- U4 pad 22: +5V -> /~{BUSRQ}
- U4 pad 23: /~{GRST} -> /~{Z80RES}
- U4 pad 24: /~{GM1} -> /~{M1}
- U4 pad 27: /GA0 -> /A0
- U4 pad 28: /GA1 -> /A1
- U4 pad 29: /GA2 -> /A2
- U4 pad 3: /GD3 -> /D3
- U4 pad 30: /GA3 -> /A3
- U4 pad 31: /GA4 -> /A4
- U4 pad 32: /GA5 -> /A5
- U4 pad 34: /GA6 -> /A6
- U4 pad 35: /GA7 -> /A7
- U4 pad 36: /GA8 -> /A8
- U4 pad 37: /GA9 -> /A9
- U4 pad 38: /GA10 -> /A10
- U4 pad 4: /GD5 -> /D5
- U4 pad 40: /GA11 -> /A11
- U4 pad 41: /GA12 -> /A12
- U4 pad 42: /GA13 -> /A13
- U4 pad 43: /GA14 -> /A14
- U4 pad 44: /GA15 -> /A15
- U4 pad 5: /GD6 -> /D6
- U4 pad 7: /GD2 -> /D2
- U4 pad 8: /GD7 -> /D7
- U4 pad 9: /GD0 -> /D0
- U5 pad 10: GNDA -> GND
- U5 pad 11: +3V3_2 -> +3V3_MIDI
- U5 pad 12: +3V3_2 -> +3V3_MIDI
- U5 pad 14: GNDA -> GND
- U5 pad 15: GNDA -> GND
- U5 pad 16: /MIDI_IN -> /MIDI_DATA
- U5 pad 20: +3V3_2 -> +3V3_MIDI
- U5 pad 31: +3V3_2 -> +3V3_MIDI
- U5 pad 35: +3V3_2 -> +3V3_MIDI
- U5 pad 38: /~{RSTOUT} -> /~{RESET}
- U5 pad 39: /MIDI_CLK -> Net-(U5-X1)
- U5 pad 40: unconnected-(U5-X2-Pad40) -> Net-(U5-X2)
- U5 pad 41: +3V3_2 -> +3V3_MIDI
- U5 pad 46: +3V3_2 -> +3V3_MIDI
- U5 pad 47: +3V3_2 -> +3V3_MIDI
- U5 pad 6: +3V3_2 -> +3V3_MIDI
- U5 pad 7: GNDA -> GND
- U5 pad 8: +3V3_2 -> +3V3_MIDI
- U6 pad 1: unconnected-(U6-NC-Pad1) -> /MEMA18
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Other:
- board size 100 x 80.8 mm -> 100 x 100 mm

Commit message: wip pcb rev.A
Parts:
- U4: footprint my:TQFP-44_14x14mm_P0.8mm -> my:Z80_FEC_VEC

Commit message: wip pcb rev.A. Main board almost done
Parts:
- removed U24: EPM3064ATC100, Package_QFP:TQFP-100_14x14mm_P0.5mm
- added U29: EPM3128ATC100, Package_QFP:TQFP-100_14x14mm_P0.5mm, F.Cu at (176.7, 77.5)
- added X3: 14 MHz, my:Oscillator_SMD_7050_7.0x5.0mm, F.Cu at (174.3, 63.8)
- U2: moved to B.Cu
- moved U28 82.2 mm to (132.2, 92.9), turned to 180 degrees
- moved C15 78.8 mm to (133.9, 92.9), turned to 180 degrees
- moved C10 78.2 mm to (134.4, 90.6), turned to 0 degrees
- moved U26 74.3 mm to (141.5, 92.9), turned to 180 degrees
- moved C29 70.9 mm to (143.2, 92.9), turned to 180 degrees
- moved C28 69.4 mm to (143.6, 90.6), turned to 0 degrees
- moved U25 67.6 mm to (150.7, 92.9), turned to 180 degrees
- moved C21 64.4 mm to (152.4, 92.9), turned to 180 degrees
- moved C14 62.2 mm to (152.8, 90.6), turned to 0 degrees
- moved R42 16.7 mm to (152.9, 141.6)
- moved R43 16.7 mm to (151.3, 141.6)
- moved U16 10.8 mm to (159.2, 63.1)
- moved U15 10.7 mm to (145.2, 63.1)
- moved R14 9.30 mm to (141.0, 130.2)
- moved R19 9.30 mm to (141.0, 125.7)
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Connections:
- U15 pad 11: unconnected-(U15-~{IC}-Pad11) -> /~{YMRST}
- U16 pad 11: unconnected-(U16-~{IC}-Pad11) -> /~{YMRST}
Routing:
- net /TAPE_IN: track 0.00 -> 35.7 mm
- net /TAPE_OUT: track 0.00 -> 32.6 mm
- net /ESP_RX: track 0.00 -> 30.5 mm
- net /ESP_TX: track 0.00 -> 28.7 mm, vias 0 -> 1
- net /RA3: track 0.00 -> 21.3 mm, vias 0 -> 1
- net /RA2: track 0.00 -> 21.3 mm, vias 0 -> 1
- net /RA0: track 0.00 -> 17.8 mm, vias 0 -> 1
- net /RD7: track 0.00 -> 17.7 mm, vias 0 -> 1
- net /~{MEMOE}: track 0.00 -> 17.6 mm, vias 0 -> 1
- net /RD6: track 0.00 -> 17.6 mm, vias 0 -> 1
- net /RD5: track 0.00 -> 17.6 mm, vias 0 -> 1
- net /RD4: track 0.00 -> 17.6 mm, vias 0 -> 1
- net /RD3: track 0.00 -> 17.6 mm, vias 0 -> 1
- net /RD2: track 0.00 -> 17.6 mm, vias 0 -> 1
- net /RD1: track 0.00 -> 17.6 mm, vias 0 -> 1
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Other:
- outline, holes or cut-outs redrawn

Commit message: wip pcb rev.A
Parts:
- removed JP2: SolderJumper_2_Bridged, Jumper:SolderJumper-2_P1.3mm_Bridged_RoundedPad1.0x1.5mm
- removed LOGO1: graphic, mygraphic:black-mage-6.7x9.5
- removed R23, R25, R34: 10k, Resistor_SMD:R_0603_1608Metric_Pad0.98x0.95mm_HandSolder
- removed R27, R28: 47k, Resistor_SMD:R_0603_1608Metric_Pad0.98x0.95mm_HandSolder
- removed R63: 3.3k, Resistor_SMD:R_0805_2012Metric_Pad1.20x1.40mm_HandSolder
- removed U19: TDA1543T, Package_SO:SOIC-16W_7.5x10.3mm_P1.27mm
- removed U21: 74ACT245, Package_SO:TSSOP-20_4.4x6.5mm_P0.65mm
- removed Y1: 12 MHz, Crystal:Crystal_SMD_SeikoEpson_TSX3225-4Pin_3.2x2.5mm_HandSoldering
- added C30: 10u, Capacitor_SMD:C_0805_2012Metric_Pad1.18x1.45mm_HandSolder, B.Cu at (152.7, 57.2)
- added C32: 100n, Capacitor_SMD:C_0603_1608Metric_Pad1.08x0.95mm_HandSolder, B.Cu at (150.9, 57.2)
- added C34: 22u, Capacitor_Tantalum_SMD:CP_EIA-3216-18_Kemet-A_Pad1.58x1.35mm_HandSolder, B.Cu at (149.0, 57.2)
- added C35: 22u, Capacitor_Tantalum_SMD:CP_EIA-3216-18_Kemet-A_Pad1.58x1.35mm_HandSolder, B.Cu at (143.6, 84.2)
- added C36: 2.2u, Capacitor_SMD:C_0603_1608Metric_Pad1.08x0.95mm_HandSolder, B.Cu at (130.8, 83.4)
- added C37: 2.2n, Capacitor_SMD:C_0603_1608Metric_Pad1.08x0.95mm_HandSolder, B.Cu at (130.1, 78.6)
- added C38: 2.2n, Capacitor_SMD:C_0603_1608Metric_Pad1.08x0.95mm_HandSolder, B.Cu at (131.7, 78.6)
- added C39: 100n, Capacitor_SMD:C_0603_1608Metric_Pad1.08x0.95mm_HandSolder, B.Cu at (127.4, 83.4)
- added C40: 100n, Capacitor_SMD:C_0603_1608Metric_Pad1.08x0.95mm_HandSolder, B.Cu at (130.8, 86.6)
- added C41: 10u, Capacitor_SMD:C_0805_2012Metric_Pad1.18x1.45mm_HandSolder, B.Cu at (129.0, 86.6)
- added C42: 100n, Capacitor_SMD:C_0603_1608Metric_Pad1.08x0.95mm_HandSolder, B.Cu at (123.1, 65.9)
- added C43: 100n, Capacitor_SMD:C_0603_1608Metric_Pad1.08x0.95mm_HandSolder, B.Cu at (142.3, 65.9)
- added C44: 100n, Capacitor_SMD:C_0603_1608Metric_Pad1.08x0.95mm_HandSolder, B.Cu at (159.0, 55.1)
- added C45: 100n, Capacitor_SMD:C_0603_1608Metric_Pad1.08x0.95mm_HandSolder, B.Cu at (120.7, 119.3)
- added C46: 100n, Capacitor_SMD:C_0603_1608Metric_Pad1.08x0.95mm_HandSolder, B.Cu at (113.2, 119.3)
- added C47: 100n, Capacitor_SMD:C_0603_1608Metric_Pad1.08x0.95mm_HandSolder, B.Cu at (186.0, 135.4)
- added C48: 100n, Capacitor_SMD:C_0603_1608Metric_Pad1.08x0.95mm_HandSolder, B.Cu at (161.8, 139.7)
- added C49: 100n, Capacitor_SMD:C_0603_1608Metric_Pad1.08x0.95mm_HandSolder, B.Cu at (147.2, 128.0)
- added C50: 100n, Capacitor_SMD:C_0603_1608Metric_Pad1.08x0.95mm_HandSolder, B.Cu at (128.0, 140.1)
- added C51: 100n, Capacitor_SMD:C_0603_1608Metric_Pad1.08x0.95mm_HandSolder, B.Cu at (137.9, 110.6)
- added C52: 100n, Capacitor_SMD:C_0603_1608Metric_Pad1.08x0.95mm_HandSolder, B.Cu at (144.1, 116.7)
- added C53: 100n, Capacitor_SMD:C_0603_1608Metric_Pad1.08x0.95mm_HandSolder, B.Cu at (131.7, 116.8)
- added C54: 100n, Capacitor_SMD:C_0603_1608Metric_Pad1.08x0.95mm_HandSolder, B.Cu at (137.9, 123.0)
- added C55: 100n, Capacitor_SMD:C_0603_1608Metric_Pad1.08x0.95mm_HandSolder, B.Cu at (168.9, 63.6)
- added C56: 100n, Capacitor_SMD:C_0603_1608Metric_Pad1.08x0.95mm_HandSolder, B.Cu at (162.7, 69.8)
- added C57: 100n, Capacitor_SMD:C_0603_1608Metric_Pad1.08x0.95mm_HandSolder, B.Cu at (175.0, 69.8)
- added C58: 100n, Capacitor_SMD:C_0603_1608Metric_Pad1.08x0.95mm_HandSolder, B.Cu at (168.9, 76.0)
- added C59: 100n, Capacitor_SMD:C_0603_1608Metric_Pad1.08x0.95mm_HandSolder, B.Cu at (128.5, 126.8)
- added C60: 100n, Capacitor_SMD:C_0603_1608Metric_Pad1.08x0.95mm_HandSolder, B.Cu at (108.8, 112.2)
- added C61: 100n, Capacitor_SMD:C_0603_1608Metric_Pad1.08x0.95mm_HandSolder, B.Cu at (189.8, 91.6)
- added C62: 100n, Capacitor_SMD:C_0603_1608Metric_Pad1.08x0.95mm_HandSolder, B.Cu at (151.9, 103.3)
- added C63: 100n, Capacitor_SMD:C_0603_1608Metric_Pad1.08x0.95mm_HandSolder, B.Cu at (189.8, 96.7)
- added C64: 100n, Capacitor_SMD:C_0603_1608Metric_Pad1.08x0.95mm_HandSolder, B.Cu at (163.7, 97.5)
- added C65: 100n, Capacitor_SMD:C_0603_1608Metric_Pad1.08x0.95mm_HandSolder, B.Cu at (169.6, 97.6)
- added C66: 100n, Capacitor_SMD:C_0603_1608Metric_Pad1.08x0.95mm_HandSolder, B.Cu at (161.3, 102.9)
- added C67: 100n, Capacitor_SMD:C_0603_1608Metric_Pad1.08x0.95mm_HandSolder, B.Cu at (161.3, 108.8)
- added C68: 100n, Capacitor_SMD:C_0603_1608Metric_Pad1.08x0.95mm_HandSolder, B.Cu at (169.6, 111.3)
- added C69: 100n, Capacitor_SMD:C_0603_1608Metric_Pad1.08x0.95mm_HandSolder, B.Cu at (172.6, 111.3)
- added C70: 100n, Capacitor_SMD:C_0603_1608Metric_Pad1.08x0.95mm_HandSolder, B.Cu at (166.7, 97.6)
- added C71: 100n, Capacitor_SMD:C_0603_1608Metric_Pad1.08x0.95mm_HandSolder, B.Cu at (172.6, 97.6)
- added C72: 100n, Capacitor_SMD:C_0603_1608Metric_Pad1.08x0.95mm_HandSolder, B.Cu at (161.3, 100.0)
- added C73: 100n, Capacitor_SMD:C_0603_1608Metric_Pad1.08x0.95mm_HandSolder, B.Cu at (161.3, 105.9)
- added C74: 100n, Capacitor_SMD:C_0603_1608Metric_Pad1.08x0.95mm_HandSolder, B.Cu at (163.7, 111.3)
- added C75: 100n, Capacitor_SMD:C_0603_1608Metric_Pad1.08x0.95mm_HandSolder, B.Cu at (166.7, 111.3)
- added C76: 100n, Capacitor_SMD:C_0603_1608Metric_Pad1.08x0.95mm_HandSolder, B.Cu at (145.3, 55.4)
- added C77: 100n, Capacitor_SMD:C_0603_1608Metric_Pad1.08x0.95mm_HandSolder, B.Cu at (139.7, 61.4)
- added C78: 100n, Capacitor_SMD:C_0603_1608Metric_Pad1.08x0.95mm_HandSolder, B.Cu at (135.0, 59.0)
- added C79: 100n, Capacitor_SMD:C_0603_1608Metric_Pad1.08x0.95mm_HandSolder, B.Cu at (140.0, 54.2)
- added C80: 100n, Capacitor_SMD:C_0603_1608Metric_Pad1.08x0.95mm_HandSolder, B.Cu at (175.0, 105.9)
- added C81: 100n, Capacitor_SMD:C_0603_1608Metric_Pad1.08x0.95mm_HandSolder, B.Cu at (175.0, 102.9)
- added C82: 100n, Capacitor_SMD:C_0603_1608Metric_Pad1.08x0.95mm_HandSolder, B.Cu at (122.7, 124.8)
- added C83: 100n, Capacitor_SMD:C_0603_1608Metric_Pad1.08x0.95mm_HandSolder, B.Cu at (114.7, 92.5)
- added C84: 47u, Capacitor_Tantalum_SMD:CP_EIA-3528-21_Kemet-B_Pad1.50x2.35mm_HandSolder, B.Cu at (121.7, 122.3)
- added C85: 100n, Capacitor_SMD:C_0603_1608Metric_Pad1.08x0.95mm_HandSolder, B.Cu at (119.0, 95.8)
- added C86: 100n, Capacitor_SMD:C_0603_1608Metric_Pad1.08x0.95mm_HandSolder, B.Cu at (111.2, 93.0)
- added C87: 100n, Capacitor_SMD:C_0603_1608Metric_Pad1.08x0.95mm_HandSolder, B.Cu at (114.8, 100.2)
- added C88: 100n, Capacitor_SMD:C_0603_1608Metric_Pad1.08x0.95mm_HandSolder, B.Cu at (119.5, 100.2)
- added C89: 100n, Capacitor_SMD:C_0603_1608Metric_Pad1.08x0.95mm_HandSolder, B.Cu at (132.2, 86.6)
- added C90: 100n, Capacitor_SMD:C_0603_1608Metric_Pad1.08x0.95mm_HandSolder, B.Cu at (141.0, 86.6)
- added C91: 100n, Capacitor_SMD:C_0603_1608Metric_Pad1.08x0.95mm_HandSolder, B.Cu at (131.4, 81.6)
- added C92: 100n, Capacitor_SMD:C_0603_1608Metric_Pad1.08x0.95mm_HandSolder, B.Cu at (126.8, 81.6)
- added C93: 100n, Capacitor_SMD:C_0603_1608Metric_Pad1.08x0.95mm_HandSolder, B.Cu at (135.6, 81.6)
- added C94: 100n, Capacitor_SMD:C_0603_1608Metric_Pad1.08x0.95mm_HandSolder, B.Cu at (140.1, 81.6)
- added C95: 100n, Capacitor_SMD:C_0603_1608Metric_Pad1.08x0.95mm_HandSolder, B.Cu at (114.5, 87.2)
- added C96: 100n, Capacitor_SMD:C_0603_1608Metric_Pad1.08x0.95mm_HandSolder, B.Cu at (120.3, 87.2)
- added C97: 100n, Capacitor_SMD:C_0603_1608Metric_Pad1.08x0.95mm_HandSolder, B.Cu at (189.8, 110.7)
- added C98: 100n, Capacitor_SMD:C_0603_1608Metric_Pad1.08x0.95mm_HandSolder, B.Cu at (189.8, 122.9)
- added G***: LOGO, mygraphic:black-mage-12.5x8.6, F.Cu at (168.1, 104.5)
- added JP3: Jumper, Connector_PinHeader_2.54mm:PinHeader_1x02_P2.54mm_Vertical, F.Cu at (194.8, 140.5)
- added Q2: BC847, Package_TO_SOT_SMD:SOT-23, B.Cu at (189.8, 125.6)
- added R60: 51, Resistor_SMD:R_0603_1608Metric_Pad0.98x0.95mm_HandSolder, B.Cu at (179.7, 104.0)
- added U30: LP2985-3.3, Package_TO_SOT_SMD:SOT-23-5_HandSoldering, F.Cu at (151.3, 57.1)
- added U31: LP2985-3.3, Package_TO_SOT_SMD:SOT-23-5_HandSoldering, F.Cu at (145.6, 84.2)
- added U32: PCM5102A, Package_SO:TSSOP-20_4.4x6.5mm_P0.65mm, F.Cu at (129.1, 84.2)
- C11, C27: value 10u -> 2.2n; footprint Capacitor_Tantalum_SMD:CP_EIA-3216-18_Kemet-A_Pad1.58x1.35mm_HandSolder -> Capacitor_SMD:C_0603_1608Metric_Pad1.08x0.95mm_HandSolder; moved to B.Cu
- C12, C13: value 10u -> 100n; footprint Capacitor_Tantalum_SMD:CP_EIA-3216-18_Kemet-A_Pad1.58x1.35mm_HandSolder -> Capacitor_SMD:C_0603_1608Metric_Pad1.08x0.95mm_HandSolder; moved to B.Cu
- C16: footprint Capacitor_Tantalum_SMD:CP_EIA-3216-18_Kemet-A_Pad1.58x1.35mm_HandSolder -> Capacitor_SMD:C_0805_2012Metric_Pad1.18x1.45mm_HandSolder; moved to B.Cu
- C33: value 22u -> 100n; footprint Capacitor_Tantalum_SMD:CP_EIA-3216-18_Kemet-A_Pad1.58x1.35mm_HandSolder -> Capacitor_SMD:C_0603_1608Metric_Pad1.08x0.95mm_HandSolder
- C5, C6: value 22p -> 100n
- C9: value 10u -> 2.2u; footprint Capacitor_Tantalum_SMD:CP_EIA-3216-18_Kemet-A_Pad1.58x1.35mm_HandSolder -> Capacitor_SMD:C_0603_1608Metric_Pad1.08x0.95mm_HandSolder; moved to B.Cu
- R10, R12: value 47k -> 470
- R13: value 24k -> 470
- R15: value 24k -> 6.8k
- R47: value 6.8k -> 1k
- R8: value 10k -> 470
- U17: value TDA1543 -> 74LVC2G04DB; footprint Package_DIP:DIP-8_W7.62mm -> Package_TO_SOT_SMD:SOT-23-6_Handsoldering
- U2: moved to F.Cu
- U27: value 1117-3.3 -> PCM5102A; footprint Package_TO_SOT_SMD:SOT-223-3_TabPin2 -> Package_SO:TSSOP-20_4.4x6.5mm_P0.65mm
- U3: moved to B.Cu
- X3: value 14 MHz -> 24 MHz
- Y2: footprint Crystal:Crystal_SMD_SeikoEpson_TSX3225-4Pin_3.2x2.5mm_HandSoldering -> my:Crystal_SMD_3225-4Pin_3.2x2.5mm_HandSoldering
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Connections:
- C11 pad 1: /DACCH0 -> GND
- C11 pad 2: Net-(C11-Pad2) -> /PSG_L
- C12 pad 1: /DACCH1 -> GND
- C12 pad 2: Net-(C12-Pad2) -> Net-(U27-VNEG)
- C13 pad 1: /AY_A1 -> GND
- C13 pad 2: Net-(C13-Pad2) -> Net-(U27-LDOO)
- C16 pad 1: /AY_A2 -> GND
- C16 pad 2: Net-(C16-Pad2) -> Net-(U27-LDOO)
- C17 pad 1: /AY_B1 -> /MIDI_L
- C18 pad 1: /AY_B2 -> /MA_LEFT
- C19 pad 1: /FM1 -> /NGS_AOL
- C20 pad 1: /FM2 -> /PSG_L
- C22 pad 1: /AY_C1 -> /PSG_R
- C23 pad 1: /AY_C2 -> /NGS_AOR
- C24 pad 1: /DACCH2 -> /MA_RIGHT
- C25 pad 1: /DACCH3 -> /MIDI_R
- C26 pad 2: GNDA -> GND
- C27 pad 1: /MIDI_R -> GND
- C27 pad 2: Net-(C27-Pad2) -> /PSG_R
- C33 pad 1: +3V3_MIDI -> GND
- C33 pad 2: GND -> Net-(U31-BP)
- C5 pad 2: Net-(U5-X2) -> +2V5
- C6 pad 2: Net-(U5-X1) -> +2V5
- C7 pad 2: /MA_XTALI -> /MA_XTALO
- C8 pad 2: /MA_XTALO -> /MA_XTALI
- C9 pad 1: /MIDI_L -> Net-(U27-CAPM)
- C9 pad 2: Net-(C9-Pad2) -> Net-(U27-CAPP)
- J1 pad 3: GNDA -> GND
- J1 pad 4: GNDA -> GND
- J4 pad R2: GNDA -> GND
- J4 pad S: GNDA -> GND
- R10 pad 1: /MIXER_L -> Net-(U27-OUTR)
- R10 pad 2: Net-(C11-Pad2) -> /PSG_R
- R12 pad 1: /MIXER_L -> Net-(U32-OUTL)
- R12 pad 2: Net-(C12-Pad2) -> /NGS_AOL
- R13 pad 1: /MIXER_L -> Net-(U32-OUTR)
- R13 pad 2: Net-(C13-Pad2) -> /NGS_AOR
- R15 pad 1: /MIXER_L -> Net-(Q2-B)
- R15 pad 2: Net-(C16-Pad2) -> Net-(R15-Pad2)
- R59 pad 1: /MA_XTALO -> /MA_XTALI
- R59 pad 2: /MA_XTALI -> /MA_XTALO
- R8 pad 1: /MIXER_L -> Net-(U27-OUTL)
- R8 pad 2: Net-(C9-Pad2) -> /PSG_L
- U11 pad 128: /MA_CLK -> Net-(U11-IO/DEV_OE)
- U11 pad 32: /ZXID4 -> /ZXD4
- U11 pad 33: /ZXID3 -> /ZXD3
- U11 pad 36: /ZXID5 -> /ZXD5
- U11 pad 37: /ZXID6 -> /ZXD6
- U11 pad 38: /ZXID2 -> /ZXD2
- U11 pad 39: /ZXID1 -> /ZXD1
- U11 pad 41: /ZXID0 -> /ZXD0
- U11 pad 42: /ZXID7 -> /ZXD7
- U11 pad 43: /ZXBUSIN -> unconnected-(U11-IO-Pad43)
- U11 pad 44: /~{ZXBUSENA} -> unconnected-(U11-IO-Pad44)
- U15 pad 12: unconnected-(U15-5V/~{3V}-Pad12) -> +5V
- U15 pad 23: unconnected-(U15-BCO-Pad23) -> /YMBCO0
- U15 pad 24: unconnected-(U15-DO-Pad24) -> /YMDO0
- U15 pad 25: unconnected-(U15-WCO-Pad25) -> /YMWCO0
- U15 pad 26: unconnected-(U15-LRO-Pad26) -> /YMLRO0
- U15 pad 27: unconnected-(U15-VDD-Pad27) -> +5V
- U16 pad 12: unconnected-(U16-5V/~{3V}-Pad12) -> +5V
- U16 pad 23: unconnected-(U16-BCO-Pad23) -> /YMBCO1
- U16 pad 24: unconnected-(U16-DO-Pad24) -> /YMDO1
- U16 pad 25: unconnected-(U16-WCO-Pad25) -> /YMWCO1
- U16 pad 26: unconnected-(U16-LRO-Pad26) -> /YMLRO1
- U16 pad 27: unconnected-(U16-VDD-Pad27) -> +5V
- U17 pad 1: /DAC_BITCK -> /~{ZXRES}
- U17 pad 2: /DAC_LRCK -> GND
- U17 pad 3: /DAC_DAT -> GND
- U17 pad 4: GNDA -> unconnected-(U17-Pad4)
- U17 pad 5: unconnected-(U17-VDD-Pad5) -> +5V
- U17 pad 6: /DAC_AOL -> Net-(R15-Pad2)
- U23 pad 16: /MA_XTALI -> /MA_XTALO
- U23 pad 17: /MA_XTALO -> /MA_XTALI
- U23 pad 34: GNDA -> GND
- U23 pad 37: GNDA -> GND
- U23 pad 44: GNDA -> GND
- U27 pad 1: GND -> +3V3A
- U27 pad 2: +3V3_MIDI -> Net-(U27-CAPP)
- U27 pad 3: +5V -> GND
- U29 pad 10: unconnected-(U29-I/O-Pad10) -> /YMDO1
- U29 pad 100: unconnected-(U29-I/O-Pad100) -> /YMBCO0
- U29 pad 12: unconnected-(U29-I/O-Pad12) -> /YMWCO1
- U29 pad 13: unconnected-(U29-I/O-Pad13) -> /YMLRO1
- U29 pad 14: unconnected-(U29-I/O-Pad14) -> /YMCK
- U29 pad 15: unconnected-(U29-TMS-Pad15) -> /TMS
- U29 pad 16: unconnected-(U29-I/O-Pad16) -> /YMD0
- U29 pad 17: unconnected-(U29-I/O-Pad17) -> /YMD1
- U29 pad 19: unconnected-(U29-I/O-Pad19) -> /YMD2
- U29 pad 2: unconnected-(U29-I/O-Pad2) -> /~{YMWR}
- U29 pad 20: unconnected-(U29-I/O-Pad20) -> /YMD3
- U29 pad 21: unconnected-(U29-I/O-Pad21) -> /YMD4
- U29 pad 22: unconnected-(U29-I/O-Pad22) -> /YMD5
- U29 pad 23: unconnected-(U29-I/O-Pad23) -> /YMD6
- U29 pad 24: unconnected-(U29-I/O-Pad24) -> /YMD7
- U29 pad 25: unconnected-(U29-I/O-Pad25) -> /~{YMRST}
- U29 pad 27: unconnected-(U29-I/O-Pad27) -> /PSG_LRCK
- U29 pad 28: unconnected-(U29-I/O-Pad28) -> /PSG_DIN
- U29 pad 29: unconnected-(U29-I/O-Pad29) -> /PSG_BCK
- U29 pad 44: unconnected-(U29-I/O-Pad44) -> /~{ZXM1}
- U29 pad 45: unconnected-(U29-I/O-Pad45) -> /ZXA4
- U29 pad 46: unconnected-(U29-I/O-Pad46) -> /ZXA5
- U29 pad 47: unconnected-(U29-I/O-Pad47) -> /ZXA6
- U29 pad 48: unconnected-(U29-I/O-Pad48) -> /ZXA7
- U29 pad 49: unconnected-(U29-I/O-Pad49) -> /~{ZXWR}
- U29 pad 5: unconnected-(U29-I/O-Pad5) -> /~{YMRD}
- U29 pad 52: unconnected-(U29-I/O-Pad52) -> /~{ZXIORQ}
- U29 pad 54: unconnected-(U29-I/O-Pad54) -> /ZXD4
- U29 pad 55: unconnected-(U29-I/O-Pad55) -> /ZXD3
- U29 pad 56: unconnected-(U29-I/O-Pad56) -> /ZXA3
- U29 pad 57: unconnected-(U29-I/O-Pad57) -> /ZXD5
- U29 pad 58: unconnected-(U29-I/O-Pad58) -> /ZXA2
- U29 pad 6: unconnected-(U29-I/O-Pad6) -> /YMA0
- U29 pad 60: unconnected-(U29-I/O-Pad60) -> /ZXD6
- U29 pad 61: unconnected-(U29-I/O-Pad61) -> /ZXA1
- U29 pad 62: unconnected-(U29-TCK-Pad62) -> /TCK
- U29 pad 63: unconnected-(U29-I/O-Pad63) -> /ZXD2
- U29 pad 64: unconnected-(U29-I/O-Pad64) -> /ZXA0
- U29 pad 67: unconnected-(U29-I/O-Pad67) -> /ZXD1
- U29 pad 68: unconnected-(U29-I/O-Pad68) -> /ZXD0
- U29 pad 69: unconnected-(U29-I/O-Pad69) -> /ZXD7
- U29 pad 7: unconnected-(U29-I/O-Pad7) -> /YMA1
- U29 pad 70: unconnected-(U29-I/O-Pad70) -> /ZXA13
- U29 pad 71: unconnected-(U29-I/O-Pad71) -> /ZXA14
- U29 pad 72: unconnected-(U29-I/O-Pad72) -> /ZXA15
- U29 pad 8: unconnected-(U29-I/O-Pad8) -> /~{YMCS1}
- U29 pad 87: Net-(U29-GCLK1) -> unconnected-(U29-GCLK1-Pad87)
- U29 pad 88: unconnected-(U29-OE1-Pad88) -> /~{ZXRD}
- U29 pad 89: unconnected-(U29-GCLRn-Pad89) -> /~{ZXRES}
- U29 pad 9: unconnected-(U29-I/O-Pad9) -> /YMBCO1
- U29 pad 90: unconnected-(U29-OE2/GCLK2-Pad90) -> Net-(U29-OE2/GCLK2)
- U29 pad 92: unconnected-(U29-I/O-Pad92) -> /MIDI_CLK
- U29 pad 93: unconnected-(U29-I/O-Pad93) -> /~{MIDI_RST}
- U29 pad 96: unconnected-(U29-I/O-Pad96) -> /YMLRO0
- U29 pad 97: unconnected-(U29-I/O-Pad97) -> /YMWCO0
- U29 pad 98: unconnected-(U29-I/O-Pad98) -> /~{YMCS0}
- U29 pad 99: unconnected-(U29-I/O-Pad99) -> /YMDO0
- U3 pad 1: /MEMA15 -> /RA1
- U3 pad 16: /MEMA18 -> /MEMA19
- U3 pad 17: /MEMA17 -> /RA8
- U3 pad 18: /RA7 -> /RA9
- U3 pad 19: /RA6 -> /RA10
- U3 pad 2: /MEMA14 -> /RA2
- U3 pad 20: /RA5 -> /RA11
- U3 pad 21: /RA4 -> /RA12
- U3 pad 22: /RA3 -> /RA13
- U3 pad 23: /RA2 -> /MEMA14
- U3 pad 24: /RA1 -> /MEMA15
- U3 pad 25: /RA0 -> /MEMA16
- U3 pad 29: /RD0 -> /RD7
- U3 pad 3: /RA13 -> /RA3
- U3 pad 31: /RD1 -> /RD6
- U3 pad 33: /RD2 -> /RD5
- U3 pad 35: /RD3 -> /RD4
- U3 pad 38: /RD4 -> /RD3
- U3 pad 4: /RA12 -> /RA4
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Routing:
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- added copper zone on B.Cu, net +2V5
- added copper zone on F.Cu, net +3V3
Other:
- outline, holes or cut-outs redrawn
- board text added: "NeoGS design by NedoPC"
- board text added: "TOP PCB Rev.${REVISION} Eugene Lozovoy 2024"
- board text added: "ZXEVO.1010"
- board text removed: "1010"
- board text removed: "PCB Rev.${REVISION} Eugene Lozovoy 2024"
- board text removed: "ZXEVO"

Commit message: wip pcb rev.A
Parts:
- removed U20: ESP32-WROOM-32, RF_Module:ESP32-WROOM-32
- added C99: 100u, Capacitor_SMD:CP_Elec_5x5.9, F.Cu at (133.1, 104.2)
- R1, R2, R7: value 10k -> 6.8k
- R11: value 4.7k -> 6.8k
- U11: footprint Package_QFP:TQFP-144_20x20mm_P0.5mm -> PCM_Package_QFP_AKL:TQFP-144_20x20mm_P0.5mm
- moved C61 39.6 mm to (151.2, 100.5), turned to 180 degrees
- moved U8 38.8 mm to (151.2, 96.0), turned to 180 degrees
- moved R53 38.7 mm to (151.2, 95.3), turned to 180 degrees
- moved U12 38.7 mm to (151.2, 99.6), turned to 180 degrees
- moved R54 38.6 mm to (151.2, 99.0), turned to 180 degrees
- moved C63 38.6 mm to (151.2, 96.8), turned to 180 degrees
- moved R14 7.85 mm to (133.9, 126.6), turned to 180 degrees
- moved R51 5.40 mm to (133.9, 129.7), turned to 180 degrees
- moved R52 4.39 mm to (133.9, 128.1), turned to 180 degrees
- moved C21 3.85 mm to (132.3, 97.7), turned to 0 degrees
- moved C15 3.42 mm to (118.0, 106.2), turned to 0 degrees
- moved U7 3.33 mm to (131.6, 128.1), turned to 0 degrees
- moved C59 3.09 mm to (131.3, 128.1), turned to 90 degrees
- moved C14 2.98 mm to (135.2, 95.4)
- moved C28 2.98 mm to (144.6, 95.4)
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Connections:
- U29 pad 31: unconnected-(U29-I/O-Pad31) -> /ZXD7
- U29 pad 32: unconnected-(U29-I/O-Pad32) -> /ZXD0
- U29 pad 35: unconnected-(U29-I/O-Pad35) -> /ZXD1
- U29 pad 36: unconnected-(U29-I/O-Pad36) -> /ZXD2
- U29 pad 37: unconnected-(U29-I/O-Pad37) -> /ZXD6
- U29 pad 40: unconnected-(U29-I/O-Pad40) -> /ZXD5
- U29 pad 41: unconnected-(U29-I/O-Pad41) -> /ZXD3
- U29 pad 42: unconnected-(U29-I/O-Pad42) -> /ZXD4
- U29 pad 50: unconnected-(U29-I/O-Pad50) -> /~{ZXRD}
- U29 pad 52: /~{ZXIORQ} -> /~{ZXMREQ}
- U29 pad 54: /ZXD4 -> /ZXA3
- U29 pad 55: /ZXD3 -> /ZXA2
- U29 pad 56: /ZXA3 -> /ZXA1
- U29 pad 57: /ZXD5 -> /ZXA0
- U29 pad 58: /ZXA2 -> /ZXA13
- U29 pad 60: /ZXD6 -> /ZXA14
- U29 pad 61: /ZXA1 -> /ZXA15
- U29 pad 63: /ZXD2 -> unconnected-(U29-I/O-Pad63)
- U29 pad 64: /ZXA0 -> unconnected-(U29-I/O-Pad64)
- U29 pad 67: /ZXD1 -> unconnected-(U29-I/O-Pad67)
- U29 pad 68: /ZXD0 -> unconnected-(U29-I/O-Pad68)
- U29 pad 69: /ZXD7 -> unconnected-(U29-I/O-Pad69)
- U29 pad 70: /ZXA13 -> unconnected-(U29-I/O-Pad70)
- U29 pad 71: /ZXA14 -> unconnected-(U29-I/O-Pad71)
- U29 pad 72: /ZXA15 -> unconnected-(U29-I/O-Pad72)
- U29 pad 88: /~{ZXRD} -> unconnected-(U29-OE1-Pad88)
Routing:
- net +3V3: track 25.0 -> 170.5 mm, vias 5 -> 32
- net /MP3_XRESET: track 2.59 -> 122.8 mm, vias 0 -> 2
- net /MP3_REQ: track 2.68 -> 119.3 mm, vias 0 -> 2
- net /MP3_CLK: track 2.93 -> 119.5 mm, vias 0 -> 2
- net /MP3_DAT: track 3.34 -> 119.7 mm, vias 0 -> 2
- net /MP3_SYNC: track 2.84 -> 118.6 mm, vias 0 -> 2
- net +5V: track 13.9 -> 100.4 mm, vias 3 -> 14
- net /MA_CS: track 3.53 -> 89.3 mm, vias 0 -> 2
- net /MA_DI: track 2.43 -> 87.7 mm, vias 0 -> 2
- net /MA_DO: track 2.35 -> 86.5 mm, vias 0 -> 2
- net /MA_CLK: track 2.47 -> 82.0 mm, vias 0 -> 3
- net /ZXA4: track 0.00 -> 78.2 mm, vias 0 -> 3
- net /ZXA5: track 0.00 -> 76.8 mm, vias 0 -> 3
- net /ZXA6: track 0.00 -> 71.8 mm, vias 0 -> 3
- net /ZXA7: track 0.00 -> 70.1 mm, vias 0 -> 3
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