File: pcb_top/rev.A/zxevo1010_top.kicad_pcb (KiCad board)
At the start: 2 copper layers, 100 x 100 mm, 197 parts, among them J1 Conn_02x05_Odd_Even, J2 Conn_02x05_Odd_Even, J3 Conn_02x05_Odd_Even, J4 PJ-320, J6 Conn_02x30_Row_Letter_First, Q1 BSS138, Q2 BC847, U1 ESP-12E, U10 EPM3064ATC100, U11 EP1K30TC144, U12 74AHCT1G125DB, U13 74AHCT1G125DB, U14 74AHCT1G125DB, U15 YMF288-M, U16 YMF288-M, U17 74LVC2G04DB, U18 MAX809LEUR, U2 CY62167EV30LL-45ZXI, U22 74LXC245, U23 MA8201, U25 1117-3.3, U26 1117-2.5, U27 PCM5102A, U28 1117-1.8, U29 EPM3128ATC100, U3 CY62167EV30LL-45ZXI, U30 LP2985-3.3, U31 LP2985-3.3, U32 PCM5102A, U4 Z84C0020FEC, U5 SAM2695, U6 29F040, U7 74LVC1G04DB, U8 74AHCT1G125DB, U9 VS1053b, X1 20 MHz, X2 24 MHz, X3 24 MHz, Y2 14 MHz

Commit message: wip pcb rev.A
Parts:
- added TP1: TestPoint, TestPoint:TestPoint_Pad_D1.0mm, F.Cu at (164.1, 80.0)
- added TP2: TestPoint, TestPoint:TestPoint_Pad_D1.0mm, F.Cu at (159.2, 63.6)
- added TP3: TestPoint, TestPoint:TestPoint_Pad_D1.0mm, F.Cu at (176.9, 62.5)
- C5, C6, C64, C65, C66, C67, C68, C69, C70, C71, C72, C73, C74, C75, C80, C81: footprint Capacitor_SMD:C_0603_1608Metric_Pad1.08x0.95mm_HandSolder -> Capacitor_SMD:C_0805_2012Metric_Pad1.18x1.45mm_HandSolder
- moved R46 56.7 mm to (123.0, 100.2)
- moved R41 31.5 mm to (160.3, 114.0), turned to 180 degrees
- moved R45 18.6 mm to (175.6, 114.0), turned to 0 degrees
- moved R44 13.8 mm to (164.8, 139.7), turned to 90 degrees
- moved R42 9.76 mm to (163.3, 139.7), turned to 90 degrees
- moved R43 7.82 mm to (159.3, 139.8), turned to 90 degrees
- moved R57 4.49 mm to (178.5, 129.2)
- moved R3 3.38 mm to (185.2, 131.8)
- moved R33 3.38 mm to (180.8, 131.8)
- moved R36 3.38 mm to (177.8, 131.8)
- moved R4 3.38 mm to (186.8, 131.8)
- moved R5 3.38 mm to (183.8, 131.8)
- moved R6 3.38 mm to (182.2, 131.8)
- moved R9 3.38 mm to (179.2, 131.8)
- moved C98 2.45 mm to (189.8, 120.5)
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Connections:
- J6 pad 58: +12V -> unconnected-(J6-Pin_58-Pad58)
- U2 pad 1: /MEMA15 -> /MEMA16
- U2 pad 48: /MEMA16 -> /MEMA15
- U22 pad 14: /A0 -> /A4
- U22 pad 15: /A1 -> /A3
- U22 pad 17: /A3 -> /A1
- U22 pad 18: /A4 -> /A0
- U22 pad 2: /RA4 -> /RA0
- U22 pad 3: /RA3 -> /RA1
- U22 pad 5: /RA1 -> /RA3
- U22 pad 6: /RA0 -> /RA4
- U29 pad 1: unconnected-(U29-I/O-Pad1) -> Net-(TP2-Pad1)
- U29 pad 30: unconnected-(U29-I/O-Pad30) -> Net-(TP1-Pad1)
- U29 pad 75: unconnected-(U29-I/O-Pad75) -> Net-(TP3-Pad1)
- U3 pad 24: /MEMA15 -> /MEMA16
- U3 pad 25: /MEMA16 -> /MEMA15
Routing:
- net /D6: track 2.62 -> 99.5 mm, vias 0 -> 6
- net /D4: track 3.46 -> 99.9 mm, vias 0 -> 4
- net /~{ZXRES}: track 0.00 -> 94.4 mm, vias 0 -> 4
- net /A11: track 2.76 -> 95.6 mm, vias 0 -> 3
- net /A13: track 2.48 -> 94.5 mm, vias 0 -> 4
- net /A14: track 2.68 -> 94.3 mm, vias 0 -> 2
- net /D0: track 4.45 -> 95.8 mm, vias 0 -> 8
- net /D3: track 3.01 -> 93.3 mm, vias 0 -> 4
- net /D5: track 2.81 -> 91.1 mm, vias 0 -> 4
- net /D7: track 3.74 -> 91.8 mm, vias 0 -> 6
- net /A15: track 2.87 -> 88.7 mm
- net /A12: track 2.56 -> 85.2 mm, vias 0 -> 6
- net /D2: track 3.37 -> 83.0 mm, vias 0 -> 4
- net /D1: track 4.77 -> 81.2 mm, vias 0 -> 6
- net /A7: track 3.74 -> 78.4 mm, vias 0 -> 5
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- added copper zone on B.Cu, net +5V

Commit message: wip pcb rev.A
Parts:
- moved R14 7.82 mm to (127.6, 131.3), turned to 90 degrees
- moved C51 6.51 mm to (144.1, 112.6), turned to 90 degrees
- moved C54 6.20 mm to (131.7, 123.2), turned to -90 degrees
- moved R51 4.97 mm to (129.2, 131.3), turned to 90 degrees
- moved R9 4.47 mm to (182.2, 128.5), turned to 90 degrees
- moved R52 4.46 mm to (130.7, 131.3), turned to 90 degrees
- moved R6 3.68 mm to (183.8, 128.5), turned to 90 degrees
- moved R4 3.66 mm to (185.3, 128.5), turned to 90 degrees
- moved C20 3.06 mm to (115.3, 70.2)
- moved C18 3.06 mm to (109.0, 70.2)
- moved R20 3.00 mm to (108.4, 70.2)
- moved R22 3.00 mm to (114.8, 70.2)
- moved R36 2.90 mm to (180.7, 131.8)
- moved U7 2.58 mm to (129.2, 129.0), turned to -90 degrees
- moved R57 2.25 mm to (180.7, 128.5), turned to 90 degrees
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Connections:
- U2 pad 1: /MEMA16 -> /MEMA19
- U2 pad 16: /MEMA18 -> /MEMA17
- U2 pad 17: /MEMA17 -> /MEMA21
- U2 pad 18: /RA7 -> /RA9
- U2 pad 19: /RA6 -> /RA8
- U2 pad 2: /MEMA14 -> /MEMA15
- U2 pad 29: /RD0 -> /RD6
- U2 pad 3: /RA13 -> /MEMA16
- U2 pad 31: /RD1 -> /RD7
- U2 pad 33: /RD2 -> /RD5
- U2 pad 35: /RD3 -> /RD4
- U2 pad 38: /RD4 -> /RD2
- U2 pad 4: /RA12 -> /MEMA18
- U2 pad 40: /RD5 -> /RD3
- U2 pad 42: /RD6 -> /RD0
- U2 pad 44: /RD7 -> /RD1
- U2 pad 45: /MEMA21 -> /RA6
- U2 pad 48: /MEMA15 -> /RA7
- U2 pad 5: /RA11 -> /RA10
- U2 pad 6: /RA10 -> /RA11
- U2 pad 7: /RA9 -> /RA12
- U2 pad 8: /RA8 -> /RA13
- U2 pad 9: /MEMA19 -> /MEMA14
- U3 pad 16: /MEMA19 -> /MEMA14
- U3 pad 17: /RA8 -> /RA13
- U3 pad 18: /RA9 -> /RA12
- U3 pad 19: /RA10 -> /RA11
- U3 pad 20: /RA11 -> /RA10
- U3 pad 21: /RA12 -> /MEMA18
- U3 pad 22: /RA13 -> /MEMA16
- U3 pad 23: /MEMA14 -> /MEMA15
- U3 pad 24: /MEMA16 -> /MEMA19
- U3 pad 25: /MEMA15 -> /RA7
- U3 pad 29: /RD7 -> /RD1
- U3 pad 31: /RD6 -> /RD0
- U3 pad 33: /RD5 -> /RD3
- U3 pad 35: /RD4 -> /RD2
- U3 pad 38: /RD3 -> /RD4
- U3 pad 40: /RD2 -> /RD5
- U3 pad 42: /RD1 -> /RD7
- U3 pad 44: /RD0 -> /RD6
- U3 pad 45: /MEMA21 -> /RA6
- U3 pad 6: /RA6 -> /RA8
- U3 pad 7: /RA7 -> /RA9
- U3 pad 8: /MEMA17 -> /MEMA21
- U3 pad 9: /MEMA18 -> /MEMA17
Routing:
- net /~{MEMOE}: track 0.94 -> 75.5 mm, vias 1 -> 5
- net +5V: track 123.5 -> 191.3 mm, vias 18 -> 25
- net /~{ROMCS}: track 0.00 -> 55.8 mm, vias 0 -> 4
- net /CS_CFG: track 1.11 -> 51.9 mm, vias 1 -> 4
- net +3V3: track 190.7 -> 235.9 mm, vias 33 -> 42
- net /MEMA19: track 5.28 -> 48.8 mm, vias 1 -> 2
- net /~{MEMWE}: track 37.3 -> 80.6 mm, vias 4 -> 6
- net /~{STATUS}: track 2.23 -> 45.2 mm, vias 1 -> 4
- net /RD2: track 4.97 -> 46.8 mm, vias 1 -> 3
- net /RD1: track 4.97 -> 46.8 mm, vias 1 -> 3
- net /RD3: track 4.97 -> 46.8 mm, vias 1 -> 3
- net /INIT_DONE: track 2.92 -> 44.7 mm, vias 1 -> 4
- net /CONF_DONE: track 2.29 -> 42.9 mm, vias 1 -> 4
- net /~{OUT_RAMCS1}: track 0.00 -> 40.5 mm, vias 0 -> 1
- net /RD0: track 4.97 -> 45.4 mm, vias 1 -> 3
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
Commit message: wip pcb rev.A
Parts:
- added R23: 0, Resistor_SMD:R_1206_3216Metric, B.Cu at (185.4, 74.2)
- moved C63 41.0 mm to (190.8, 94.5)
- moved C61 41.0 mm to (190.8, 99.7)
- moved U8 38.7 mm to (189.9, 94.5), turned to -90 degrees
- moved U12 38.7 mm to (189.9, 99.7), turned to -90 degrees
- moved R53 36.4 mm to (188.9, 94.5), turned to 90 degrees
- moved R54 36.4 mm to (188.9, 99.7), turned to 90 degrees
- moved C21 2.44 mm to (134.8, 97.7), turned to 180 degrees
- moved R45 2.01 mm to (177.4, 113.0), turned to -90 degrees
- moved C62 1.90 mm to (149.9, 101.4)
- moved R56 1.90 mm to (152.6, 101.4)
- moved U14 1.90 mm to (151.2, 101.3)
- moved R55 1.66 mm to (188.9, 110.8), turned to 90 degrees
- moved R15 1.16 mm to (190.7, 119.7), turned to -90 degrees
- moved C97 1.00 mm to (190.8, 110.8), turned to -90 degrees
- moved C98 0.96 mm to (189.2, 119.7), turned to -90 degrees
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Connections:
- C89 pad 2: +3V3 -> +3V3A
- C90 pad 2: +3V3 -> +3V3A
- U27 pad 17: +3V3 -> +3V3A
- U27 pad 20: +3V3 -> +3V3A
- U32 pad 17: +3V3 -> +3V3A
- U32 pad 20: +3V3 -> +3V3A
Routing:
- net +5V: track 191.3 -> 441.9 mm, vias 25 -> 40
- net /TCK: track 61.6 -> 148.0 mm, vias 5 -> 7
- net /~{RD}: track 41.7 -> 122.8 mm, vias 6 -> 7
- net /~{IORQ}: track 47.7 -> 128.6 mm, vias 6 -> 7
- net /~{WR}: track 50.0 -> 126.7 mm, vias 6 -> 7
- net +3V3: track 235.9 -> 304.9 mm, vias 42 -> 47
- net GND: track 164.1 -> 225.7 mm, vias 202 -> 241
- net +2V5: track 0.00 -> 54.1 mm, vias 0 -> 11
- net /~{ZXBLKROM}: track 4.92 -> 57.6 mm, vias 1 -> 3
- net /~{ZXRDROM}: track 57.6 -> 10.9 mm, vias 2 -> 0
- net /~{ZXBLKIORQ}: track 7.58 -> 51.4 mm, vias 1 -> 3
- net /ZXIORQGE: track 51.1 -> 8.64 mm, vias 2 -> 0
- net /~{WARMRES}: track 29.6 -> 61.4 mm, vias 3 -> 7
- net /~{CONFIG}: track 13.4 -> 41.2 mm, vias 1 -> 4
- net /CLK_Z80: track 63.8 -> 88.8 mm, vias 0 -> 1
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
Commit message: wip pcb rev.A
Parts:
- C42, C43: footprint Capacitor_SMD:C_0603_1608Metric_Pad1.08x0.95mm_HandSolder -> Capacitor_SMD:C_0805_2012Metric_Pad1.18x1.45mm_HandSolder
- moved U14 57.3 mm to (194.8, 138.5)
- moved R56 57.2 mm to (196.2, 138.5)
- moved C62 57.2 mm to (193.4, 138.5)
- moved R40 9.55 mm to (151.2, 94.9), turned to 180 degrees
- moved R49 2.68 mm to (121.6, 115.8), turned to 180 degrees
- moved C60 1.73 mm to (107.0, 112.2), turned to 0 degrees
- moved JP3 1.65 mm to (194.8, 142.1)
- moved R39 1.44 mm to (168.4, 92.8), turned to 0 degrees
- moved R37 1.31 mm to (176.3, 92.8)
- moved R50 1.29 mm to (121.6, 114.2), turned to 180 degrees
- moved R38 1.01 mm to (173.0, 92.8)
- moved D1 0.18 mm to (173.0, 91.7)
- moved C53 0.10 mm to (131.7, 117.9)
Connections:
- J3 pad 3: /TDO_3032 -> /TDO
- J3 pad 9: /TDI_FPGA -> /TDI
- R26 pad 2: /TDI_FPGA -> /TDI
- R3 pad 2: +3V3 -> +5V
- R36 pad 2: +3V3 -> +5V
- R4 pad 2: +3V3 -> +5V
- R42 pad 2: +3V3 -> +5V
- R43 pad 2: +3V3 -> +5V
- R44 pad 2: +3V3 -> +5V
- R53 pad 1: +3V3 -> +5V
- R54 pad 1: +3V3 -> +5V
- R55 pad 1: +3V3 -> +5V
- R56 pad 1: +3V3 -> +5V
- U10 pad 4: /TDOFPGA_TDI3032 -> /TDI
- U10 pad 73: /TDO_3032 -> /TDI_FPGA
- U11 pad 4: /TDOFPGA_TDI3032 -> /TDI_PSG
- U2 pad 14: unconnected-(U2-~{BHE}-Pad14) -> /~{RD}
- U2 pad 15: unconnected-(U2-~{BLE}-Pad15) -> /~{WR}
- U29 pad 4: unconnected-(U29-TDI-Pad4) -> /TDI_PSG
- U29 pad 73: unconnected-(U29-TDO-Pad73) -> /TDO
Routing:
- net +3V3: track 304.9 -> 455.0 mm, vias 47 -> 53
- net /TDO: track 0.00 -> 87.3 mm, vias 0 -> 3
- net /TDI: track 0.00 -> 74.3 mm, vias 0 -> 2
- net /~{WARMRES}: track 61.4 -> 125.9 mm, vias 7 -> 10
- net /TDI_PSG: track 0.00 -> 58.0 mm, vias 0 -> 6
- net /TMS: track 95.3 -> 148.7 mm, vias 5 -> 11
- net /CLK_FPGA: track 0.00 -> 47.2 mm, vias 0 -> 1
- net /TDI_FPGA: track 5.15 -> 52.0 mm, vias 0 -> 2
- net /CS_CFG: track 50.5 -> 96.8 mm, vias 4 -> 6
- net /TCK: track 148.0 -> 191.0 mm, vias 7 -> 9
- net +5V: track 441.9 -> 484.1 mm, vias 40 -> 41
- net /CONF_DONE: track 41.6 -> 82.4 mm, vias 4 -> 7
- net /INIT_DONE: track 43.3 -> 75.8 mm, vias 4 -> 6
- net /~{STATUS}: track 42.9 -> 64.2 mm, vias 4 -> 6
- net GND: track 225.7 -> 235.8 mm, vias 241 -> 242
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Other:
- board text added: "JTAG chain: 1 NEOGS CPLD 2 NEOGS FPGA 3 PSG CPLD"
