File: pcb_top/rev.A/zxevo1010_top.kicad_pcb (KiCad board)
At the start: 2 copper layers, 100 x 100 mm, 201 parts, among them J1 Conn_02x05_Odd_Even, J2 Conn_02x05_Odd_Even, J3 Conn_02x05_Odd_Even, J4 PJ-320, J6 Conn_02x30_Row_Letter_First, Q1 BSS138, Q2 BC847, U1 ESP-12E, U10 EPM3064ATC100, U11 EP1K30TC144, U12 74AHCT1G125DB, U13 74AHCT1G125DB, U14 74AHCT1G125DB, U15 YMF288-M, U16 YMF288-M, U17 74LVC2G04DB, U18 MAX809LEUR, U2 CY62167EV30LL-45ZXI, U22 74LXC245, U23 MA8201, U25 1117-3.3, U26 1117-2.5, U27 PCM5102A, U28 1117-1.8, U29 EPM3128ATC100, U3 CY62167EV30LL-45ZXI, U30 LP2985-3.3, U31 LP2985-3.3, U32 PCM5102A, U4 Z84C0020FEC, U5 SAM2695, U6 29F040, U7 74LVC1G04DB, U8 74AHCT1G125DB, U9 VS1053b, X1 20 MHz, X2 24 MHz, X3 24 MHz, Y2 14 MHz

Commit message: wip pcb rev.A (almost done)
Parts:
- removed the R23 at (185.4, 74.2)
- removed the U7 at (129.2, 129.0)
- removed Y2: 14 MHz, my:Crystal_SMD_3225-4Pin_3.2x2.5mm_HandSoldering
- added U17: SN74LVC2G04DBVR, Package_TO_SOT_SMD:SOT-23-6_Handsoldering, F.Cu at (129.2, 129.1)
- added Y1: 14 MHz, Crystal:Crystal_HC49-4H_Vertical, F.Cu at (114.7, 105.6)
- C4: renamed from C26; footprint Capacitor_SMD:C_0805_2012Metric_Pad1.18x1.45mm_HandSolder -> Capacitor_SMD:C_0603_1608Metric_Pad1.08x0.95mm_HandSolder
- U10: renamed from U17; value 74LVC2G04DB -> SN74LVC2G04DBVR
- U11: renamed from U13; value 74AHCT1G125DB -> SN74AHCT1G125DBVR
- U12: renamed from U14; value 74AHCT1G125DB -> SN74AHCT1G125DBVR
- U3: renamed from U10; value EPM3064ATC100 -> EPM3128ATC100
- U7: renamed from U8; value 74AHCT1G125DB -> SN74AHCT1G125DBVR
- U8: renamed from U12; value 74AHCT1G125DB -> SN74AHCT1G125DBVR
- U9: renamed from U22; value 74LXC245 -> SN74LXC8T245PWR
- moved R11 29.6 mm to (129.7, 115.2), turned to 90 degrees
- moved U26 15.0 mm to (132.7, 98.6), turned to -90 degrees
- moved C47 14.0 mm to (131.3, 101.8), turned to 180 degrees
- moved C46 11.3 mm to (130.4, 96.5), turned to 90 degrees
- moved C8 7.20 mm to (119.6, 107.3), turned to 180 degrees
- moved U24 7.11 mm to (140.1, 98.6), turned to -90 degrees
- moved C43 5.62 mm to (138.7, 101.8)
- moved R9 5.12 mm to (117.2, 104.3)
- moved U25 5.04 mm to (147.4, 98.6), turned to -90 degrees
- moved C42 4.59 mm to (129.1, 106.7), turned to -135 degrees
- moved C45 4.44 mm to (146.0, 101.8)
- moved R39 4.12 mm to (180.9, 127.9), turned to 90 degrees
- moved R34 4.12 mm to (184.2, 127.9), turned to 90 degrees
- moved R43 4.12 mm to (179.3, 127.9), turned to 90 degrees
- moved C69 4.11 mm to (140.6, 110.5), turned to 180 degrees
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- renumbered C36 to C1, C17 to C10, C18 to C11, C19 to C12, C20 to C13, C22 to C14, C23 to C15, C24 to C16, C25 to C17, C1 to C18, C2 to C19, C37 to C2, C3 to C20, C4 to C21, C9 to C22, C27 to C23, C11 to C24, C12 to C25, C13 to C26, C16 to C27, C84 to C28, C76 to C29, C38 to C3, C77 to C30, C78 to C31, C79 to C32, C91 to C33, C92 to C34, C93 to C35, C94 to C36, C95 to C37, C96 to C38, C90 to C39, C89 to C40, C14 to C41, C99 to C42, C21 to C43, C28 to C44, C29 to C45, C10 to C46, C15 to C47, C31 to C48, C33 to C49, C39 to C5, C35 to C50, C30 to C51, C32 to C52, C34 to C53, C42 to C54, C43 to C55, C44 to C56, C45 to C57, C46 to C58, C47 to C59, C40 to C6, C48 to C60, C59 to C61, C60 to C62, C61 to C63, C62 to C64, C63 to C65, C97 to C66, C98 to C67, C50 to C68, C51 to C69, C41 to C7, C52 to C70, C53 to C71, C54 to C72, C55 to C73, C56 to C74, C57 to C75, C58 to C76, C64 to C77, C65 to C78, C66 to C79, C67 to C80, C68 to C81, C69 to C82, C80 to C83, C81 to C84, C82 to C85, C49 to C89, C7 to C9, C70 to C90, C71 to C91, C72 to C92, C73 to C93, C74 to C94, C75 to C95, C5 to C96, C6 to C97, C83 to C98, C85 to C99, J6 to J1, J1 to J2, J2 to J3, J3 to J5, JP3 to JP1, JP1 to JP2, Q2 to Q1, Q1 to Q2, R12 to R1, R45 to R10, R40 to R11, R16 to R12, R18 to R13, R19 to R14, R53 to R15, R46 to R16, R60 to R17, R58 to R18, R47 to R19, R37 to R2, R54 to R20, R41 to R21, R15 to R22, R17 to R23, R55 to R24, R20 to R25, R21 to R26, R22 to R27, R29 to R28, R30 to R29, R13 to R3, R31 to R30, R32 to R31, R56 to R32, R57 to R33, R3 to R34, R4 to R35, R48 to R36, R24 to R37, R26 to R38, R33 to R39, R42 to R4, R9 to R40, R5 to R41, R6 to R42, R36 to R43, R51 to R44, R49 to R45, R14 to R46, R50 to R47, R52 to R48, R35 to R49, R43 to R5, R8 to R50, R10 to R51, R11 to R52, R1 to R53, R7 to R54, R2 to R55, R44 to R6, R38 to R7, R39 to R8, R59 to R9, TP2 to TP1, TP3 to TP2, TP1 to TP3, U32 to U1, U6 to U13, U4 to U14, U2 to U15, U3 to U16, U15 to U18, U16 to U19, U23 to U2, U5 to U20, U29 to U21, U27 to U22, U1 to U23, U25 to U24, U26 to U25, U28 to U26, U31 to U27, U30 to U28, U18 to U4, U11 to U5, U9 to U6
Connections:
- U16 pad 15: unconnected-(U3-~{BLE}-Pad15) -> /~{MEMOE}
Routing:
- net /CLK_FPGA: track 47.2 -> 131.8 mm, vias 1 -> 5
- net /CLKSEL0: track 2.24 -> 78.6 mm, vias 1 -> 5
- net /CLKSEL1: track 2.28 -> 77.8 mm, vias 1 -> 5
- net Net-(JP1-A): track 0.00 -> 22.2 mm, vias 0 -> 1
- net +5V: track 484.1 -> 505.3 mm, vias 41 -> 54
- net /~{MEMOE}: track 89.1 -> 107.9 mm, vias 5 -> 8
- net /~{Z80RES}: track 56.7 -> 73.2 mm, vias 5 -> 7
- net +1V8: track 43.2 -> 33.5 mm, vias 7 -> 10
- net +3V3: track 455.0 -> 446.1 mm, vias 53 -> 58
- net /D4: track 98.0 -> 89.6 mm, vias 4 -> 6
- net /A8: track 75.3 -> 67.8 mm, vias 5 -> 6
- net /TDI_FPGA: track 52.0 -> 59.6 mm
- net /A11: track 87.2 -> 80.4 mm, vias 4 -> 8
- net /D6: track 97.9 -> 91.6 mm
- net +2V5: track 54.1 -> 48.0 mm
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- added copper zone on F.Cu, net +5V
Other:
- board text added: "16x 100n"
- board text added: "TSFM + MIDI + SounDrive + NeoGS + WiFi"
- board text added: "↑ 8x 10u ↑"

Commit message: wip pcb rev.A
Parts:
- added G***: LOGO, mygraphic:jack35, F.Cu at (132.9, 55.7)
- added Q3: BSS138, Package_TO_SOT_SMD:SOT-23, B.Cu at (122.8, 134.8)
- added R56: 6.8k, Resistor_SMD:R_0603_1608Metric_Pad0.98x0.95mm_HandSolder, B.Cu at (122.8, 137.5)
- added R57: 6.8k, Resistor_SMD:R_0603_1608Metric_Pad0.98x0.95mm_HandSolder, B.Cu at (147.5, 65.6)
- added R58: 6.8k, Resistor_SMD:R_0603_1608Metric_Pad0.98x0.95mm_HandSolder, B.Cu at (128.4, 65.6)
- C25, C33, C34, C35, C36, C5: value 100n -> 2.2u
- C28: value 47u -> 22u; footprint Capacitor_Tantalum_SMD:CP_EIA-3528-21_Kemet-B_Pad1.50x2.35mm_HandSolder -> Capacitor_Tantalum_SMD:CP_EIA-3216-18_Kemet-A_Pad1.58x1.35mm_HandSolder
- C42: footprint Capacitor_SMD:CP_Elec_5x5.9 -> Capacitor_Tantalum_SMD:CP_EIA-6032-28_Kemet-C_Pad2.25x2.35mm_HandSolder
- Q1: value BC847 -> BSS138
- R23, R31: value 47k -> 22k
- R25, R30: value 47k -> 18k
- R26, R27: value 10k -> 47k
- R28, R29: value 24k -> 47k
- R32: value 6.8k -> 1k
- R49: value 10k -> 6.8k
- R7: value 100 -> 120
- X3: value 24 MHz -> 32 MHz
- moved TP1 21.7 mm to (180.3, 68.8)
- moved C42 1.27 mm to (128.2, 107.5)
- moved C28 0.26 mm to (122.5, 122.3)
Connections:
- J1 pad 3: /ZXA12 -> unconnected-(J1-Pin_3-Pad3)
- J1 pad 31: /RS -> unconnected-(J1-Pin_31-Pad31)
- J1 pad 50: /~{ZXRFSH} -> unconnected-(J1-Pin_50-Pad50)
- J1 pad 52: /ZXA8 -> unconnected-(J1-Pin_52-Pad52)
- J1 pad 53: /ZXA9 -> unconnected-(J1-Pin_53-Pad53)
- J1 pad 54: /ZXA10 -> unconnected-(J1-Pin_54-Pad54)
- J1 pad 55: /ZXA11 -> unconnected-(J1-Pin_55-Pad55)
- J3 pad 5: unconnected-(J3-Pin_5-Pad5) -> /~{ESP_RST}
- U18 pad 16: unconnected-(U18-~{COM}-Pad16) -> GND
- U18 pad 22: unconnected-(U18-~{STBY}-Pad22) -> Net-(U18-~{STBY})
- U19 pad 16: unconnected-(U19-~{COM}-Pad16) -> GND
- U19 pad 22: unconnected-(U19-~{STBY}-Pad22) -> Net-(U19-~{STBY})
- U21 pad 1: Net-(TP1-Pad1) -> /~{YMCS0}
- U21 pad 100: /YMBCO0 -> /YMWCO0
- U21 pad 63: unconnected-(U21-I/O-Pad63) -> Net-(TP1-Pad1)
- U21 pad 96: /YMLRO0 -> /YMBCO0
- U21 pad 97: /YMWCO0 -> /YMDO0
- U21 pad 98: /~{YMCS0} -> /MIDI_DATA
- U21 pad 99: /YMDO0 -> /YMLRO0
- U23 pad 1: /~{RESET} -> Net-(Q3-S)
Routing:
- net /~{ESP_RST}: track 0.00 -> 37.3 mm, vias 0 -> 3
- net /MIDI_DATA: track 0.00 -> 27.6 mm
- net +5V: track 505.3 -> 514.1 mm, vias 54 -> 56
- net +3V3: track 446.1 -> 450.3 mm
- net Net-(TP1-Pad1): track 1.79 -> 5.30 mm
- net Net-(Q3-S): track 0.00 -> 3.49 mm, vias 0 -> 1
- net /YMBCO0: track 16.0 -> 19.0 mm
- net /YMWCO0: track 21.6 -> 18.6 mm
- net /YMLRO0: track 24.6 -> 22.6 mm
- net /~{YMCS0}: track 10.1 -> 8.26 mm
- net /YMDO0: track 18.3 -> 19.8 mm
- net Net-(U19-~{STBY}): track 0.00 -> 1.35 mm, vias 0 -> 1
- net GND: track 236.2 -> 237.4 mm, vias 350 -> 353
- net Net-(U18-~{STBY}): track 0.00 -> 0.64 mm, vias 0 -> 1
Other:
- board text added: "NC"

Commit message: wip pcb rev.A
Parts:
- removed C1, C22, C25, C5: 2.2u, Capacitor_SMD:C_0603_1608Metric_Pad1.08x0.95mm_HandSolder
- removed C2, C23, C24, C3: 2.2n, Capacitor_SMD:C_0603_1608Metric_Pad1.08x0.95mm_HandSolder
- removed C39, C40: 100n, Capacitor_SMD:C_0603_1608Metric_Pad1.08x0.95mm_HandSolder
- added C100: 100n, Capacitor_SMD:C_0603_1608Metric_Pad1.08x0.95mm_HandSolder, B.Cu at (152.4, 59.0)
- added J6: PJ392, Connector_PinHeader_2.54mm:PinHeader_1x03_P2.54mm_Vertical, F.Cu at (156.0, 54.7)
- added R59: 51, Resistor_SMD:R_0603_1608Metric_Pad0.98x0.95mm_HandSolder, B.Cu at (153.1, 57.2)
- added R60: 470, Resistor_SMD:R_0603_1608Metric_Pad0.98x0.95mm_HandSolder, B.Cu at (153.1, 54.7)
- added U29: SN74AHCT1G125DBVR, Package_TO_SOT_SMD:SOT-23-5_HandSoldering, F.Cu at (152.3, 57.6)
- C33, C34, C35, C36: value 2.2u -> 1u
- C49, C52: value 100n -> 10n
- R1, R3, R50, R51: value 470 -> 6.8k
- R26, R27, R28, R29: value 47k -> 8.2k
- U1, U22: value PCM5102A -> UDA1334ATS; footprint Package_SO:TSSOP-20_4.4x6.5mm_P0.65mm -> Package_SO:SSOP-16_4.4x5.2mm_P0.65mm
- moved C34 11.8 mm to (137.7, 86.3), turned to 180 degrees
- moved C36 11.1 mm to (130.2, 86.3), turned to 180 degrees
- moved C51 6.16 mm to (147.4, 60.4), turned to 90 degrees
- moved R3 5.88 mm to (132.8, 79.7), turned to 180 degrees
- moved R51 4.65 mm to (140.3, 79.6), turned to 180 degrees
- moved C6 4.48 mm to (132.0, 82.3), turned to 180 degrees
- moved C26 4.36 mm to (139.6, 82.2), turned to 180 degrees
- moved C7 3.93 mm to (132.0, 84.3), turned to 180 degrees
- moved C56 3.79 mm to (159.3, 58.9), turned to -90 degrees
- moved C33 3.23 mm to (128.2, 82.3)
- moved C52 3.20 mm to (149.3, 54.4), turned to -90 degrees
- moved C27 3.11 mm to (139.6, 84.3), turned to 180 degrees
- moved U28 2.98 mm to (148.4, 57.6), turned to 90 degrees
- moved C12 2.62 mm to (109.0, 62.4)
- moved C15 2.62 mm to (109.0, 65.0)
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Connections:
- C26 pad 2: Net-(U22-LDOO) -> Net-(U22-Vref(DAC))
- C27 pad 2: Net-(U22-LDOO) -> Net-(U22-Vref(DAC))
- C6 pad 2: Net-(U1-LDOO) -> Net-(U1-Vref(DAC))
- C7 pad 2: Net-(U1-LDOO) -> Net-(U1-Vref(DAC))
- R1 pad 1: Net-(U1-OUTL) -> Net-(U1-DEEM/CLKOUT)
- R1 pad 2: /NGS_AOL -> +3V3A
- R3 pad 1: Net-(U1-OUTR) -> GND
- R3 pad 2: /NGS_AOR -> Net-(U1-DEEM/CLKOUT)
- R50 pad 1: Net-(U22-OUTL) -> Net-(U22-DEEM/CLKOUT)
- R50 pad 2: /PSG_L -> +3V3A
- R51 pad 1: Net-(U22-OUTR) -> GND
- R51 pad 2: /PSG_R -> Net-(U22-DEEM/CLKOUT)
- U1 pad 1: +3V3A -> /DAC_BITCK
- U1 pad 12: GND -> Net-(U1-Vref(DAC))
- U1 pad 13: /DAC_BITCK -> +3V3A
- U1 pad 14: /DAC_DAT -> /NGS_AOL
- U1 pad 15: /DAC_LRCK -> GND
- U1 pad 16: GND -> /NGS_AOR
- U1 pad 2: Net-(U1-CAPP) -> /DAC_LRCK
- U1 pad 3: GND -> /DAC_DAT
- U1 pad 4: Net-(U1-CAPM) -> +3V3A
- U1 pad 5: Net-(U1-VNEG) -> GND
- U1 pad 6: Net-(U1-OUTL) -> GND
- U1 pad 7: Net-(U1-OUTR) -> GND
- U1 pad 8: +3V3A -> GND
- U1 pad 9: GND -> Net-(U1-DEEM/CLKOUT)
- U21 pad 100: /YMWCO0 -> /YMLRO0
- U21 pad 27: /PSG_LRCK -> /PSG_DIN
- U21 pad 28: /PSG_DIN -> /PSG_LRCK
- U21 pad 94: unconnected-(U21-I/O-Pad94) -> /MIDI_SENSE
- U21 pad 98: /MIDI_DATA -> /YMWCO0
- U21 pad 99: /YMLRO0 -> /MIDI_DATA
- U22 pad 1: +3V3A -> /PSG_BCK
- U22 pad 12: GND -> Net-(U22-Vref(DAC))
- U22 pad 13: /PSG_BCK -> +3V3A
- U22 pad 14: /PSG_DIN -> /PSG_L
- U22 pad 15: /PSG_LRCK -> GND
- U22 pad 16: GND -> /PSG_R
- U22 pad 2: Net-(U22-CAPP) -> /PSG_LRCK
- U22 pad 3: GND -> /PSG_DIN
- U22 pad 4: Net-(U22-CAPM) -> +3V3A
- U22 pad 5: Net-(U22-VNEG) -> GND
- U22 pad 6: Net-(U22-OUTL) -> GND
- U22 pad 7: Net-(U22-OUTR) -> GND
- U22 pad 8: +3V3A -> GND
- U22 pad 9: GND -> Net-(U22-DEEM/CLKOUT)
Routing:
- net GND: track 237.4 -> 214.2 mm, vias 353 -> 363
- net /MIDI_SENSE: track 0.00 -> 17.3 mm
- net +3V3A: track 74.8 -> 61.4 mm, vias 12 -> 16
- net /PSG_R: track 32.5 -> 26.3 mm, vias 1 -> 0
- net /MIXER_L: track 34.4 -> 29.1 mm
- net /MIDI_DATA: track 27.6 -> 32.4 mm
- net +5V: track 514.1 -> 518.8 mm, vias 56 -> 55
- net Net-(R60-Pad1): track 0.00 -> 4.63 mm, vias 0 -> 1
- net Net-(U22-Vref(DAC)): track 0.00 -> 4.57 mm, vias 0 -> 2
- net Net-(U1-Vref(DAC)): track 0.00 -> 4.52 mm, vias 0 -> 2
- net /NGS_AOR: track 33.2 -> 28.7 mm, vias 1 -> 0
- net +3V3_MIDI: track 54.8 -> 50.5 mm
- net Net-(U1-LDOO): track 3.79 -> 0.00 mm, vias 2 -> 0
- net Net-(U22-LDOO): track 3.79 -> 0.00 mm, vias 2 -> 0
- net Net-(U21-OE2/GCLK2): track 9.78 -> 13.3 mm
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Other:
- board text added: "2"
- board text added: "4"
- board text added: "5"
- board text added: "J6 MIDI OUT"
- board text added: "R"
- board text added: "S"
- board text added: "T"
- board text added: "shield"
- board text added: "sink"
- board text added: "source"
