File: pcb_top/rev.A/zxevo1010_top.kicad_sch (KiCad schematic)
At the start: 90 parts, among them J1 Conn_01x04, J6 Conn_02x30_Row_Letter_First, U1 ESP-12E, U12 YM2203, U13 YM3014B, U14 YM2203, U15 YM3014B, U16 LMV358IDR, U17 LMV358IDR, U2 CY62167ELL, U3 EPM3256ATC144, U4 Z84C0020FEC, U5 SAM2695, U6 27C512, U7 74HCT245D, U8 74AHCT1G125DB, U9 LMV358IDR

Commit message: wip pcbs rev.A
Parts:
- removed C14, C21: 10u, Capacitor_SMD:CP_Elec_4x5.4, symbol Device:C_Polarized
- removed C15: 100n, Capacitor_SMD:C_0603_1608Metric_Pad1.08x0.95mm_HandSolder, symbol Device:C
- removed J1: Conn_01x04, Connector_PinHeader_2.54mm:PinHeader_1x04_P2.54mm_Vertical, symbol Connector_Generic:Conn_01x04
- removed R14: 27k, Resistor_SMD:R_0603_1608Metric_Pad0.98x0.95mm_HandSolder, symbol Device:R
- removed R18, R26: 10k, Resistor_SMD:R_0603_1608Metric_Pad0.98x0.95mm_HandSolder, symbol Device:R
- removed R19: 10K, Resistor_SMD:R_0603_1608Metric_Pad0.98x0.95mm_HandSolder, symbol Device:R
- removed U9: LMV358IDR, Package_SO:SOIC-8_3.9x4.9mm_P1.27mm, symbol Amplifier_Operational:LMV358
- added J1: Conn_02x05_Odd_Even, Connector_PinHeader_2.54mm:PinHeader_2x04_P2.54mm_Vertical, symbol Connector_Generic:Conn_02x04_Odd_Even
- added J2: Conn_02x05_Odd_Even, Connector_PinHeader_2.54mm:PinHeader_2x05_P2.54mm_Vertical, symbol Connector_Generic:Conn_02x05_Odd_Even
- added Q1: BSS138, Package_TO_SOT_SMD:SOT-23, symbol Transistor_FET:BSS138
- added R7: 10k, Resistor_SMD:R_0603_1608Metric_Pad0.98x0.95mm_HandSolder, symbol Device:R
- R11: value 47k -> 4.7k
Connections:
- net +3V3_2: now also R11.2, Q1.1 (G)
- net +5V: now also J2.4 (Pin_4)
- net ESP_RX: now also J2.3 (Pin_3), Q1.3 (D); no longer U1.21 (GPIO3/RXD)
- net ESP_TX: now also J2.9 (Pin_9)
- net GND: now also J2.10 (Pin_10), J2.2 (Pin_2), R7.2
- net GNDA: now also J1.3 (Pin_3), J1.4 (Pin_4), J1.5 (Pin_5), J1.6 (Pin_6)
- net MIXER_L: now reaches R10.1, R12.1, R13.1, R15.1, R17.1, R20.1, R21.1, R22.1, R8.1
- net MIXER_L: now also J1.2 (Pin_2)
- net at R11.1: now also U1.21 (GPIO3/RXD), Q1.2 (S)
- net MIXER_R: now reaches R23.1, R25.1, R27.1, R28.1, R29.1, R30.1, R31.1, R32.1, R34.1
- net MIXER_R: now also J1.8 (Pin_8)
- net ESP_CTS: no longer names the net of U1.7 (GPIO13)
- net ESP_CTS: now also R7.1
- new net TAPE_IN: J1.7 (Pin_7)
- new net TAPE_OUT: J1.1 (Pin_1)
- no-connect marks 84 -> 89

Commit message: wip pcb rev.A
Parts:
- removed C10, C26, C30, C31: 10u, Capacitor_SMD:CP_Elec_4x5.4, symbol Device:C_Polarized
- removed C29, C33: 2.2n, Capacitor_SMD:C_0603_1608Metric_Pad1.08x0.95mm_HandSolder, symbol Device:C
- removed C32: 100n, Capacitor_SMD:C_0603_1608Metric_Pad1.08x0.95mm_HandSolder, symbol Device:C
- removed U12, U14: YM2203, Package_DIP:DIP-40_W15.24mm_Socket, symbol my:YM2203
- removed U13, U15: YM3014B, Package_DIP:DIP-8_W7.62mm_Socket, symbol my:YM3014B
- removed U16, U17: LMV358IDR, Package_SO:SOIC-8_3.9x4.9mm_P1.27mm, symbol Amplifier_Operational:LMV358
- removed U3: EPM3256ATC144, PCM_Package_QFP_AKL:TQFP-144_20x20mm_P0.5mm, symbol my:EPM3256ATC144
- removed U6: 27C512, my:PLCC-32_11.4x14.0mm_P1.27mm-longpads, symbol Memory_EPROM:27C512PLCC
- removed U7: 74HCT245D, Package_SO:SOIC-20W_7.5x12.8mm_P1.27mm, symbol 74xx:74HC245
- added C10, C14, C31: 10u, Capacitor_SMD:C_0805_2012Metric_Pad1.18x1.45mm_HandSolder, symbol Device:C
- added C15, C21, C29, C33: 22u, Capacitor_Tantalum_SMD:CP_EIA-3216-18_Kemet-A_Pad1.58x1.35mm_HandSolder, symbol Device:C_Polarized
- added C26: 100n, Capacitor_SMD:C_0805_2012Metric_Pad1.18x1.45mm_HandSolder, symbol Device:C
- added D1: LED, LED_SMD:LED_0603_1608Metric_Pad1.05x0.95mm_HandSolder, symbol Device:LED
- added J3: Conn_02x05_Odd_Even, Connector_PinHeader_2.54mm:PinHeader_2x05_P2.54mm_Vertical, symbol Connector_Generic:Conn_02x05_Odd_Even
- added J4: PJ-320, my:PJ-320A_D, symbol Connector_Audio:AudioJack4
- added JP2: SolderJumper_2_Bridged, Jumper:SolderJumper-2_P1.3mm_Bridged_RoundedPad1.0x1.5mm, symbol Jumper:SolderJumper_2_Bridged
- added R14, R19, R48, R49, R50, R51, R52: 51, Resistor_SMD:R_0603_1608Metric_Pad0.98x0.95mm_HandSolder, symbol Device:R
- added R16, R18, R24, R26, R44, R46, R47, R53, R54, R55, R56, R58: 6.8k, Resistor_SMD:R_0603_1608Metric_Pad0.98x0.95mm_HandSolder, symbol Device:R
- added R35: 10k, Resistor_SMD:R_0603_1608Metric_Pad0.98x0.95mm_HandSolder, symbol Device:R
- added R45: 1K, Resistor_SMD:R_0603_1608Metric_Pad0.98x0.95mm_HandSolder, symbol Device:R
- added R57: 1k, Resistor_SMD:R_0603_1608Metric_Pad0.98x0.95mm_HandSolder, symbol Device:R
- added R59: 1M, Resistor_SMD:R_0603_1608Metric_Pad0.98x0.95mm_HandSolder, symbol Device:R
- added R63: 3.3k, Resistor_SMD:R_0805_2012Metric_Pad1.20x1.40mm_HandSolder, symbol Device:R
- added U10, U24: EPM3064ATC100, Package_QFP:TQFP-100_14x14mm_P0.5mm, symbol my:EPM3064ATC100
- added U11: EP1K30TC144, Package_QFP:TQFP-144_20x20mm_P0.5mm, symbol my:EP1K30TC144
- added U12, U13, U14: 74AHCT1G125DB, Package_TO_SOT_SMD:SOT-23-5_HandSoldering, symbol 74xGxx:74LVC1G125
- added U15, U16: YMF288-M, Package_SO:SOP-28_8.4x18.16mm_P1.27mm, symbol my:YMF288-M
- added U17: TDA1543, Package_DIP:DIP-8_W7.62mm, symbol my:TDA1543
- added U18: MAX809LEUR, Package_TO_SOT_SMD:SOT-23, symbol my:MAX809
- added U19: TDA1543T, Package_SO:SOIC-16W_7.5x10.3mm_P1.27mm, symbol my:TDA1543T
- added U20: ESP32-WROOM-32, RF_Module:ESP32-WROOM-32, symbol RF_Module:ESP32-WROOM-32
- added U21: 74ACT245, Package_SO:TSSOP-20_4.4x6.5mm_P0.65mm, symbol 74xx:74LS245
- added U22: 74LXC245, Package_SO:TSSOP-20_4.4x6.5mm_P0.65mm, symbol 74xx:74LS245
- added U23: MA8201, Package_QFP:MQFP-44_10x10mm_P0.8mm, symbol my:MA8201
- added U25, U27: 1117-3.3, Package_TO_SOT_SMD:SOT-223-3_TabPin2, symbol Regulator_Linear:AZ1117-3.3
- added U26: 1117-2.5, Package_TO_SOT_SMD:SOT-223-3_TabPin2, symbol Regulator_Linear:AZ1117-2.5
- added U28: 1117-1.8, Package_TO_SOT_SMD:SOT-223-3_TabPin2, symbol Regulator_Linear:AZ1117-1.8
- added U3: CY62167EV30LL-45ZXI, Package_SO:TSOP-I-48_18.4x12mm_P0.5mm, symbol my:CY62167E
- added U6: 29F040, my:PLCC-32_11.4x14.0mm_P1.27mm-longpads, symbol my:29C040
- added U7: 74LVC1G04DB, Package_TO_SOT_SMD:SOT-23-5_HandSoldering, symbol 74xGxx:74LVC1G04
- added U9: VS1053b, Package_QFP:LQFP-48_7x7mm_P0.5mm, symbol my:VS1053
- added X1: 20 MHz, my:Oscillator_SMD_7050_7.0x5.0mm, symbol Oscillator:XO91
- added X2: 24 MHz, my:Oscillator_SMD_7050_7.0x5.0mm, symbol Oscillator:XO91
- added Y1: 12 MHz, Crystal:Crystal_SMD_SeikoEpson_TSX3225-4Pin_3.2x2.5mm_HandSoldering, symbol Device:Crystal_GND24
- added Y2: 14 MHz, Crystal:Crystal_SMD_SeikoEpson_TSX3225-4Pin_3.2x2.5mm_HandSoldering, symbol Device:Crystal_GND24
- C1, C3: value 10n -> 100n
- C11, C12, C13, C16, C17, C18, C19, C20, C22, C23, C24, C25, C27, C9: footprint Capacitor_SMD:CP_Elec_4x5.4 -> Capacitor_Tantalum_SMD:CP_EIA-3216-18_Kemet-A_Pad1.58x1.35mm_HandSolder
- C2, C4: value 10n -> 10u; footprint Capacitor_SMD:C_0603_1608Metric_Pad1.08x0.95mm_HandSolder -> Capacitor_SMD:C_0805_2012Metric_Pad1.18x1.45mm_HandSolder
- C28: value 100n -> 10u; footprint Capacitor_SMD:C_0603_1608Metric_Pad1.08x0.95mm_HandSolder -> Capacitor_SMD:C_0805_2012Metric_Pad1.18x1.45mm_HandSolder
- C5: value 100n -> 22p
- C6: value 10u -> 22p; footprint Capacitor_SMD:C_0805_2012Metric_Pad1.18x1.45mm_HandSolder -> Capacitor_SMD:C_0603_1608Metric_Pad1.08x0.95mm_HandSolder
- C7: value 100n -> 33p
- C8: value 10u -> 33p; footprint Capacitor_SMD:C_0805_2012Metric_Pad1.18x1.45mm_HandSolder -> Capacitor_SMD:C_0603_1608Metric_Pad1.08x0.95mm_HandSolder
- J1: footprint Connector_PinHeader_2.54mm:PinHeader_2x04_P2.54mm_Vertical -> Connector_PinSocket_2.54mm:PinSocket_2x03_P2.54mm_Vertical; symbol Connector_Generic:Conn_02x04_Odd_Even -> Connector_Generic:Conn_02x03_Odd_Even
- J2: footprint Connector_PinHeader_2.54mm:PinHeader_2x05_P2.54mm_Vertical -> Connector_PinSocket_2.54mm:PinSocket_2x03_P2.54mm_Vertical; symbol Connector_Generic:Conn_02x05_Odd_Even -> Connector_Generic:Conn_02x03_Odd_Even
- R3, R4, R43, R5, R6: value 1k -> 6.8k
- R33, R36, R9: value 3.3k -> 6.8k
- R37: value 470 -> 1k
- R38: value 1k -> 100
- R39, R40, R41: value 3.3k -> 1k
- R42: value 470 -> 6.8k
- U2: value CY62167ELL -> CY62167EV30LL-45ZXI
Connections:
- net FM1_ENA is gone; now on net +3V3: R38.2
- net FM2_ENA is gone; now on net +3V3: R43.2
- net GA15 is gone; now on net A15: U4.44 (A15)
- net GCLK is gone; now on net +5V: U8.2
- net GMA17 is gone; now on net MEMA18: U2.16 (A18)
- net GMA18 is gone; now on net MEMA17: U2.17 (A17)
- net ~{GINT} is gone; now on net ~{INT}: U4.12 (~{INT})
- net ~{GIORQ} is gone; now on net ~{IORQ}: U4.16 (~{IORQ})
- net ~{GM1} is gone; now on net ~{M1}: U4.24 (~{M1})
- net ~{GMREQ} is gone; now on net ~{MREQ}: U4.15 (~{MREQ})
- net ~{RSTOUT} is gone; now on net ~{RESET}: U5.38 (~{RST}/~{PD})
- net +3V3: now also Q1.1 (G), R1.2, R11.2, R3.2, R36.2, R37.2, R39.2, R4.2, R40.2, R42.2, U1.3 (EN), U1.8 (VCC), U2.12 (CE2), U2.37 (VCC), C21.1, J3.4 (Pin_4), R16.2, R18.2, R24.1, R26.1, R44.2, R45.1, R46.2, R53.1, R54.1, R55.1, R56.1, U10.18 (VCCIO), U10.3 (VCCIO), U10.34 (VCCIO), U10.39 (VCCINT), U10.51 (VCCIO), U10.66 (VCCIO), U10.82 (VCCIO), U10.91 (VCCINT), U11.10 (IO), U11.115 (VCCIO), U11.120 (IO), U11.124 (Dedicated_Input), U11.134 (VCCIO), U11.24 (VCCIO), U11.45 (VCCIO), U11.5 (VCCIO), U11.61 (VCCIO), U11.71 (VCCIO), U11.76 (MSEL1), U11.77 (MSEL0), U11.94 (VCCIO), U22.20 (VCC), U23.13 (DVDD1), U23.19 (DVDD2), U23.30 (TEST0), U23.6 (DVDD3), U25.2 (VO), U3.12 (CE2), U3.37 (VCC), U9.14 (IOVDD), U9.19 (IOVDD), U9.26 (RX), U9.32 (XTEST), U9.6 (IOVDD)
- net +5V: now also C28.2, J2.2 (Pin_2), R33.2, R5.2, R6.2, R9.2, C10.2, C14.2, C31.2, R57.2, U12.2, U12.5 (VCC), U13.5 (VCC), U14.5 (VCC), U18.3 (VCC), U21.20 (VCC), U25.3 (VI), U26.3 (VI), U27.3 (VI), U28.3 (VI), U6.32 (VCC), U7.5 (VCC), X1.1 (EN), X1.4 (V+), X2.1 (EN), X2.4 (V+); no longer J2.4 (Pin_4), U2.12 (CE2), U2.37 (VCC), U4.13 (~{NMI}), U4.22 (~{BUSRQ})
- net A0: now also U4.27 (A0), U11.102 (IO), U22.14 (B4), U6.12 (A0); no longer J6.17 (Pin_17)
- net A1: now also U4.28 (A1), U11.101 (IO), U22.15 (B3), U6.11 (A1); no longer J6.19 (Pin_19)
- net A10: now also U4.38 (A10), U10.35 (I/O), U11.90 (IO), U6.23 (A10); no longer J6.54 (Pin_54)
- net A11: now also U4.40 (A11), U10.32 (I/O), U11.89 (IO), U6.25 (A11); no longer J6.55 (Pin_55)
- net A12: now also U4.41 (A12), U10.31 (I/O), U11.88 (IO), U6.4 (A12); no longer J6.3 (Pin_3)
- net A13: now also U4.42 (A13), U10.30 (I/O), U11.87 (IO), U6.28 (A13); no longer J6.4 (Pin_4)
- net A14: now also U4.43 (A14), U10.29 (I/O), U11.86 (IO); no longer J6.1 (Pin_1)
- net A15: now also U10.25 (I/O), U11.83 (IO); no longer J6.2 (Pin_2)
- net A2: now also U4.29 (A2), U11.100 (IO), U22.16 (B2), U6.10 (A2); no longer J6.21 (Pin_21)
- net A3: now also U4.30 (A3), U11.99 (IO), U22.17 (B1), U6.9 (A3); no longer J6.23 (Pin_23)
- net A4: now also U4.31 (A4), U11.98 (IO), U22.18 (B0), U6.8 (A4); no longer J6.47 (Pin_47)
- net A5: now also U4.32 (A5), U11.97 (IO), U22.13 (B5), U6.7 (A5); no longer J6.45 (Pin_45)
- net A6: now also U4.34 (A6), U10.37 (I/O), U11.96 (IO), U6.6 (A6); no longer J6.43 (Pin_43)
- net A7: now also U4.35 (A7), U10.36 (I/O), U11.95 (IO), U6.5 (A7); no longer J6.41 (Pin_41)
- net A8: now also U4.36 (A8), U11.92 (IO), U22.12 (B6), U6.27 (A8); no longer J6.52 (Pin_52)
- net A9: now also U4.37 (A9), U11.91 (IO), U22.11 (B7), U6.26 (A9); no longer J6.53 (Pin_53)
- net AY_A1: no longer R36.2
- net AY_A2: no longer R41.2
- net AY_B1: no longer R33.2
- net AY_B2: no longer R40.2
- net AY_C1: no longer R9.2
- net AY_C2: no longer R39.2
- net D0: now also U4.9 (D0), U10.48 (I/O), U11.108 (DATA0), U11.117 (IO), U6.13 (D0); no longer J6.12 (Pin_12)
- net D1: now also U4.10 (D1), U10.45 (I/O), U11.112 (IO/DATA4), U6.14 (D1); no longer J6.14 (Pin_14)
- net D2: now also U4.7 (D2), U10.47 (I/O), U11.109 (IO/DATA1), U6.15 (D2); no longer J6.16 (Pin_16)
- net D3: now also U4.3 (D3), U10.46 (I/O), U11.111 (IO/DATA3), U6.17 (D3); no longer J6.22 (Pin_22)
- net D4: now also U4.2 (D4), U10.42 (I/O), U11.116 (IO/DATA7), U6.18 (D4); no longer J6.24 (Pin_24)
- net D5: now also U4.4 (D5), U10.44 (I/O), U11.110 (IO/DATA2), U6.19 (D5); no longer J6.20 (Pin_20)
- net D6: now also U4.5 (D6), U10.40 (I/O), U11.114 (IO/DATA6), U6.20 (D6); no longer J6.18 (Pin_18)
- net D7: now also U4.8 (D7), U10.41 (I/O), U11.113 (IO/DATA5), U6.21 (D7); no longer J6.6 (Pin_6)
- net DACCH0: no longer C4.1, R6.1
- net DACCH1: no longer C3.1, R5.1
- net DACCH2: no longer C2.1, R4.1
- net DACCH3: no longer C1.1, R3.1
- net ESP_RX: now also J2.1 (Pin_1); no longer J2.3 (Pin_3)
- net ESP_TX: now also J2.4 (Pin_4); no longer J2.9 (Pin_9)
- net GND: now also C1.1, C2.1, C28.1, C3.1, C4.1, C5.1, C6.1, C7.1, C8.1, J2.6 (Pin_6), R41.1, U5.10 (A0), U5.14 (~{CS}), U5.15 (~{RD}), U5.7 (MICIN), C10.1, C14.1, C15.2, C21.2, C29.2, C31.1, C33.2, J3.10 (Pin_10), J3.2 (Pin_2), R35.2, R47.1, R58.1, U10.11 (GNDIO), U10.26 (GNDIO), U10.33 (GNDIO), U10.38 (GNDINT), U10.43 (GNDIO), U10.53 (GNDIO), U10.59 (GNDIO), U10.65 (GNDIO), U10.74 (GNDIO), U10.78 (GNDIO), U10.86 (GNDINT), U10.95 (GNDIO), U11.104 (GND), U11.106 (nCE), U11.123 (GND), U11.129 (GND), U11.139 (GND), U11.15 (GND), U11.25 (GND), U11.40 (GND), U11.52 (GND), U11.57 (GND_CKLK), U11.58 (GND), U11.6 (GND), U11.66 (GND), U11.84 (GND), U11.93 (GND), U12.3 (GND), U13.2, U13.3 (GND), U14.2, U14.3 (GND), U15.1 (VSS), U15.14 (VSS), U16.1 (VSS), U16.14 (VSS), U18.1 (GND), U21.10 (GND), U22.1 (A->B), U22.10 (GND), U22.19 (CE), U23.15 (DGND1), U23.21 (DGND2), U23.4 (DGND3), U24.11 (GNDIO), U24.26 (GNDIO), U24.33 (GNDIO), U24.38 (GNDINT), U24.43 (GNDIO), U24.53 (GNDIO), U24.59 (GNDIO), U24.65 (GNDIO), U24.74 (GNDIO), U24.78 (GNDIO), U24.86 (GNDINT), U24.95 (GNDIO), U25.1 (GND), U26.1 (GND), U27.1 (GND), U28.1 (GND), U3.27 (GND), U3.46 (GND), U3.47 (~{BYTE}), U6.16 (GND), U7.3 (GND), U9.16 (DGND), U9.20 (DGND), U9.21 (DGND), U9.22 (DGND), U9.35 (DGND), U9.4 (DGND), X1.2 (GND), X2.2 (GND), Y1.2, Y1.4, Y2.2, Y2.4; no longer J2.10 (Pin_10), J2.2 (Pin_2), U8.1
- net GNDA: now also C26.2, J4.R2, J4.S, R63.2, U17.4 (GND), U19.6 (GND), U23.34 (AGND1), U23.37 (AGND34), U23.44 (AGND56), U9.37 (AGND), U9.40 (AGND), U9.41 (AGND), U9.47 (AGND); no longer C1.2, C2.2, C28.2, C3.2, C4.2, C5.2, C6.2, C7.2, C8.2, J1.5 (Pin_5), J1.6 (Pin_6), R33.1, R36.1, R39.1, R40.1, R41.1, R9.1, U5.10 (A0), U5.14 (~{CS}), U5.15 (~{RD}), U5.7 (MICIN)
- net MIXER_R: now also J1.6 (Pin_6); no longer J1.8 (Pin_8)
- net TAPE_IN: now also J1.5 (Pin_5), J4.T; no longer J1.7 (Pin_7)
- net TAPE_OUT: now also J4.R1
- net TCK: now also J3.1 (Pin_1), R35.1, U10.62 (TCK), U11.1 (TCK)
- net TMS: now also J3.5 (Pin_5), R24.2, U10.15 (TMS), U11.34 (TMS)
- net ~{INT}: now also R4.1, U11.59 (IO); no longer J6.26 (Pin_26)
- net ~{IORQ}: now also R6.1, U10.23 (I/O), U11.144 (IO/nCS)
- net ~{M1}: now also U11.51 (IO); no longer J6.48 (Pin_48)
- net ~{MREQ}: now also R5.1, U10.19 (I/O), U11.56 (Dedicated_Input); no longer J6.32 (Pin_32)
- net ~{NMI}: now also R3.1, U4.13 (~{NMI}), U11.60 (IO); no longer J6.28 (Pin_28)
- net ~{RD}: now also R33.1, U4.18 (~{RD}), U10.20 (I/O), U11.141 (IO/nRS); no longer J6.36 (Pin_36)
- net ~{WR}: now also R9.1, U4.19 (~{WR}), U10.21 (I/O), U11.142 (IO/nWS); no longer J6.38 (Pin_38)
- net CONF_DONE: now reaches R37.1
- net CONF_DONE: now also U10.98 (I/O), U11.2 (CONF_DONE)
- net at R38.1: now also D1.2 (A)
- net at U5.40 (X2): now also C5.2, Y1.1
- net MEMA17: now reaches R43.1
- net MEMA17: now also U11.79 (IO), U3.17 (A17), U6.30 (A17)
- net ~{BUSAK}: now reaches U4.20 (~{BUSACK})
- net ~{BUSAK}: now also U11.63 (IO)
- net MEMA21: now reaches U2.45 (A20/D15)
- net MEMA21: now also R41.2, U11.73 (IO), U3.45 (A20/D15)
- net MEMA19: now reaches U2.9 (A19)
- net MEMA19: now also U10.68 (I/O), U3.9 (A19)
- net MEMA18: now reaches R42.1
- net MEMA18: now also U11.78 (IO), U3.16 (A18), U6.1 (A18)
- net +3V3_2 renamed +3V3_MIDI
- net +3V3_MIDI: now also C33.1, U27.2 (VO); no longer Q1.1 (G), R1.2, R11.2, U1.3 (EN), U1.8 (VCC)
- net GA0 renamed RA7
- net RA7: now also U10.76 (I/O), U3.18 (A7); no longer U4.27 (A0)
- net GA1 renamed RA6
- net RA6: now also U10.79 (I/O), U3.19 (A6); no longer U4.28 (A1)
- net GA10 renamed RA10
- net RA10: now also U10.61 (I/O), U3.6 (A10); no longer U4.38 (A10)
- net GA11 renamed RA11
- net RA11: now also U10.60 (I/O), U3.5 (A11); no longer U4.40 (A11)
- net GA12 renamed RA12
- net RA12: now also U10.58 (I/O), U3.4 (A12); no longer U4.41 (A12)
- net GA13 renamed RA0
- net RA0: now also U22.6 (A4), U3.25 (A0); no longer U4.42 (A13)
- net GA14 renamed RA13
- net RA13: now also U10.57 (I/O), U3.3 (A13); no longer U4.43 (A14)
- net GA2 renamed RA5
- net RA5: now also U22.7 (A5), U3.20 (A5); no longer U4.29 (A2)
- net GA3 renamed RA4
- net RA4: now also U22.2 (A0), U3.21 (A4); no longer U4.30 (A3)
- net GA4 renamed RA3
- net RA3: now also U22.3 (A1), U3.22 (A3); no longer U4.31 (A4)
- net GA5 renamed RA2
- net RA2: now also U22.4 (A2), U3.23 (A2); no longer U4.32 (A5)
- net GA6 renamed RA1
- net RA1: now also U22.5 (A3), U3.24 (A1); no longer U4.34 (A6)
- net GA7 renamed MEMA14
- net MEMA14: now also U10.56 (I/O), U11.82 (IO), U3.2 (A14), U6.29 (A14); no longer U4.35 (A7)
- net GA8 renamed RA8
- net RA8: now also U22.8 (A6), U3.8 (A8); no longer U4.36 (A8)
- net GA9 renamed RA9
- net RA9: now also U22.9 (A7), U3.7 (A9); no longer U4.37 (A9)
- net GCLK_BUF renamed CLK_Z80
- net CLK_Z80: now also R51.1; no longer U8.4
- net GD0 renamed RD3
- net RD3: now also U10.54 (I/O), U3.35 (D3); no longer U4.9 (D0)
- net GD1 renamed RD2
- net RD2: now also U10.52 (I/O), U3.33 (D2); no longer U4.10 (D1)
- net GD2 renamed RD4
- net RD4: now also U10.80 (I/O), U3.38 (D4); no longer U4.7 (D2)
- net GD3 renamed RD1
- net RD1: now also U10.63 (I/O), U3.31 (D1); no longer U4.3 (D3)
- net GD4 renamed RD5
- net RD5: now also U10.81 (I/O), U3.40 (D5); no longer U4.2 (D4)
- net GD5 renamed RD0
- net RD0: now also U10.64 (I/O), U3.29 (D0); no longer U4.4 (D5)
- net GD6 renamed RD6
- net RD6: now also U10.85 (I/O), U3.42 (D6); no longer U4.5 (D6)
- net GD7 renamed RD7
- net RD7: now also U10.84 (I/O), U3.44 (D7); no longer U4.8 (D7)
- net GMA15 renamed MEMA15
- net MEMA15: now also U10.67 (I/O), U11.81 (IO), U3.1 (A15), U6.3 (A15)
- net GMA16 renamed MEMA16
- net MEMA16: now also R44.1, U11.80 (IO), U3.48 (A16), U6.2 (A16)
- net MIDI_CLK: no longer names the net of U5.39 (X1)
- net MIDI_CLK: now also C6.2, Y1.3
- net MIDI_IN renamed MIDI_DATA
- net ~{BUSA}: no longer names the net of J6.51 (Pin_51)
- net ~{BUSR}: no longer names the net of J6.37 (Pin_37)
- net ~{CSROM} renamed ~{ZXCSROM}
- net ~{ZXCSROM}: now also U11.31 (IO)
- net ~{DOS}: no longer names the net of J6.7 (Pin_7)
- net ~{GRAM2} renamed ~{OUT_RAMCS0}
- net ~{OUT_RAMCS0}: now also U10.83 (I/O)
- net ~{GRD} renamed ~{MEMOE}
- net ~{MEMOE}: now also U10.75 (I/O), U11.65 (IO), U3.28 (~{OE}), U6.24 (~{OE}); no longer U4.18 (~{RD})
- net ~{GRST} renamed ~{Z80RES}
- net ~{Z80RES}: now also R57.1, U11.49 (IO), U14.4
- net ~{GWR} renamed ~{MEMWE}
- net ~{MEMWE}: now also U10.69 (I/O), U11.64 (IO), U3.11 (~{WE}), U6.31 (~{WE}); no longer U4.19 (~{WR})
- net ~{HALT}: no longer names the net of J6.30 (Pin_30)
- net ~{IORQ1} renamed ~{ZXIORQ}
- net ~{ZXIORQ}: now also U11.28 (IO)
- net ~{IORQGE1} renamed ZXIORQGE
- net ZXIORQGE: now also U8.4
- net ~{RDROM} renamed ~{ZXRDROM}
- net ~{ZXRDROM}: now also U12.4
- net ~{RES} renamed ~{ZXRES}
- net ~{ZXRES}: now also JP2.1 (A)
- net ~{RFSH} renamed ~{ZXRFSH}
- net ~{WAIT} renamed ~{ZXWAIT}
- net ~{ZXWAIT}: now also U13.4
- new net: R49.2, R50.2, X2.3 (OUT)
- new net: R19.1, U10.96 (I/O)
- new net: R48.2, X1.3 (OUT)
- new net: R14.2, R51.2, R52.2, U7.4
- new net: R45.2, U11.107 (DCLK)
- new net: U20.1 (GND), U20.15 (GND), U20.38 (GND), U20.39 (GND)
- new net: C3.2, C4.2, U5.34 (OUTVC12)
- new net: C1.2, C2.2, U5.5 (VCM)
- new net: R58.2, U9.11 (GPIO6/I2S_SCLK), U9.12 (GPIO7/I2S_SDATA), U9.25 (GPIO5/I2S_MCLK), U9.33 (GPIO0), U9.34 (GPIO1), U9.36 (GPIO4/I2S_LROUT)
- new net +1V8: C15.1, U28.2 (VO), U9.24 (CVDD), U9.31 (CVDD), U9.5 (CVDD), U9.7 (CVDD)
- new net +2V5: C29.1, U11.103 (VCCINT), U11.126 (Dedicated_Input), U11.127 (VCCINT), U11.16 (VCCINT), U11.50 (VCCINT), U11.53 (VCC_CKLK), U11.75 (VCCINT), U11.85 (VCCINT), U26.2 (VO)
- new net +3V3A: U23.35 (AVDD1), U23.42 (AVDD45), U9.38 (AVDD), U9.43 (AVDD), U9.45 (AVDD)
- new net CLK20IN: R48.1, U10.90 (OE2/GCLK2)
- new net CLK24IN: R49.1, U10.88 (OE1)
- new net CLKOUT: R19.2, U7.2
- new net CLKSEL0: R16.1, U10.92 (I/O), U11.119 (IO)
- new net CLKSEL1: R18.1, U10.93 (I/O), U11.118 (IO)
- new net CLK_24MHZ: R50.1, U11.55 (Dedicated_Clock)
- new net CLK_3032: R14.1, U10.87 (GCLK1)
- new net CLK_FPGA: R52.1, U11.125 (Dedicated_Clock)
- new net CS_CFG: U10.9 (I/O), U11.143 (IO/CS)
- new net DAC_AOL: U17.6 (AOL), U19.12 (AOL)
- new net DAC_AOR: U17.8 (AOR), U19.14 (AOR)
- new net DAC_BITCK: U11.140 (IO), U17.1 (BCK), U19.3 (BCK)
- new net DAC_DAT: U11.137 (IO), U17.3 (DATA), U19.5 (DATA)
- new net DAC_LRCK: U11.138 (IO), U17.2 (WS), U19.4 (WS)
- new net DAC_VREF: R63.1, U17.7 (VREF), U19.13 (VREF)
- new net INIT_DONE: R39.1, U10.99 (I/O), U11.14 (IO/INIT_DONE)
- new net LED_DIAG: D1.1 (K), U11.11 (IO/RDYnBUSY)
- new net MA_CLK: U11.128 (IO/DEV_OE), U23.26 (SCLK), U9.28 (SCLK)
- new net MA_CS: R46.1, U11.130 (IO), U23.22 (XCS), U9.23 (xCS)
- new net MA_DI: U11.121 (IO), U23.28 (SO), U9.30 (SO)
- new net MA_DO: U11.122 (IO/DEV_CLRn), U23.27 (SI), U9.29 (SI)
- new net MA_LEFT: U23.43 (LEFT), U9.46 (LEFT)
- new net MA_RCAP: C26.1, U23.41 (RCAP), U9.44 (RCAP)
- new net MA_RIGHT: U23.36 (RIGHT), U9.39 (RIGHT)
- new net MA_XTALI: C7.2, R59.2, U23.16 (XTALO), U9.18 (XTALI), Y2.3
- new net MA_XTALO: C8.2, R59.1, U23.17 (XTALI), U9.17 (XTALO), Y2.1
- new net MP3_CLK: U11.133 (IO), U23.9 (DCLK), U9.9 (GPIO2/DCLK)
- new net MP3_DAT: U11.132 (IO), U23.10 (SDATA), U9.10 (GPIO3/SDATA)
- new net MP3_REQ: U11.135 (IO), U23.8 (DREQ), U9.8 (DREQ)
- new net MP3_SYNC: U11.131 (IO), U23.12 (BSYNC), U9.13 (xDCS/BSYNC)
- new net MP3_XRESET: R47.2, U11.136 (IO), U23.3 (XRESET), U9.3 (xRESET)
- new net TDI_FPGA: J3.9 (Pin_9), R26.2, U11.105 (TDI)
- new net TDOFPGA_TDI3032: U10.4 (TDI), U11.4 (TDO)
- new net TDO_3032: J3.3 (Pin_3), U10.73 (TDO)
- new net YMA0: U15.20 (A0), U16.20 (A0)
- new net YMA1: U15.21 (A1), U16.21 (A1)
- new net YMCK: U15.28 (MCLK), U16.28 (MCLK)
- new net YMD0: U15.2 (D0), U16.2 (D0)
- new net YMD1: U15.3 (D1), U16.3 (D1)
- new net YMD2: U15.4 (D2), U16.4 (D2)
- new net YMD3: U15.5 (D3), U16.5 (D3)
- new net YMD4: U15.6 (D4), U16.6 (D4)
- new net YMD5: U15.7 (D5), U16.7 (D5)
- new net YMD6: U15.8 (D6), U16.8 (D6)
- new net YMD7: U15.9 (D7), U16.9 (D7)
- new net ZXA0: J6.17 (Pin_17), U11.17 (IO)
- new net ZXA1: J6.19 (Pin_19), U11.18 (IO)
- new net ZXA10: J6.54 (Pin_54)
- new net ZXA11: J6.55 (Pin_55)
- new net ZXA12: J6.3 (Pin_3)
- new net ZXA13: J6.4 (Pin_4)
- new net ZXA14: J6.1 (Pin_1), U11.12 (IO)
- new net ZXA15: J6.2 (Pin_2), U11.13 (IO)
- new net ZXA2: J6.21 (Pin_21), U11.19 (IO)
- new net ZXA3: J6.23 (Pin_23), U11.20 (IO)
- new net ZXA4: J6.47 (Pin_47), U11.26 (IO)
- new net ZXA5: J6.45 (Pin_45), U11.23 (IO)
- new net ZXA6: J6.43 (Pin_43), U11.22 (IO)
- new net ZXA7: J6.41 (Pin_41), U11.21 (IO)
- new net ZXA8: J6.52 (Pin_52)
- new net ZXA9: J6.53 (Pin_53)
- new net ZXBUSIN: U11.43 (IO), U21.1 (A->B)
- new net ZXD0: J6.12 (Pin_12), U21.8 (A6)
- new net ZXD1: J6.14 (Pin_14), U21.7 (A5)
- new net ZXD2: J6.16 (Pin_16), U21.6 (A4)
- new net ZXD3: J6.22 (Pin_22), U21.3 (A1)
- new net ZXD4: J6.24 (Pin_24), U21.2 (A0)
- new net ZXD5: J6.20 (Pin_20), U21.4 (A2)
- new net ZXD6: J6.18 (Pin_18), U21.5 (A3)
- new net ZXD7: J6.6 (Pin_6), U21.9 (A7)
- new net ZXID0: U11.41 (IO), U21.12 (B6)
- new net ZXID1: U11.39 (IO), U21.13 (B5)
- new net ZXID2: U11.38 (IO), U21.14 (B4)
- new net ZXID3: U11.33 (IO), U21.17 (B1)
- new net ZXID4: U11.32 (IO), U21.18 (B0)
- new net ZXID5: U11.36 (IO), U21.16 (B2)
- new net ZXID6: U11.37 (IO), U21.15 (B3)
- new net ZXID7: U11.42 (IO/LOCK), U21.11 (B7)
- new net ~{BUSRQ}: R36.1, U11.62 (IO), U4.22 (~{BUSRQ})
- new net ~{COLDRES}: U10.89 (GCLRn), U18.2 (~{RST})
- new net ~{CONFIG}: U10.6 (I/O), U11.74 (nCONFIG)
- new net ~{IN_RAMCS0}: U10.13 (I/O), U11.72 (IO)
- new net ~{IN_RAMCS1}: U10.14 (I/O), U11.70 (IO)
- new net ~{IN_RAMCS2}: U10.16 (I/O), U11.69 (IO)
- new net ~{IN_RAMCS3}: U10.17 (I/O), U11.68 (IO)
- new net ~{OUT_RAMCS1}: U10.71 (I/O), U3.26 (~{CE1})
- new net ~{ROMCS}: U10.8 (I/O), U11.67 (IO), U6.22 (~{CE})
- new net ~{STATUS}: R40.1, U10.100 (I/O), U11.35 (nSTATUS)
- new net ~{WARMRES}: JP2.2 (B), R56.2, U10.10 (I/O), U11.54 (Dedicated_Input), U14.1
- new net ~{YMCS0}: U15.17 (~{CS})
- new net ~{YMCS1}: U16.17 (~{CS})
- new net ~{YMRD}: U15.19 (~{RD}), U16.19 (~{RD})
- new net ~{YMWR}: U15.18 (~{WR}), U16.18 (~{WR})
- new net ~{ZXBLKIORQ}: R53.2, U11.46 (IO), U8.1
- new net ~{ZXBLKROM}: R54.2, U11.47 (IO), U12.1
- new net ~{ZXBUSENA}: U11.44 (IO), U21.19 (CE)
- new net ~{ZXGENWAIT}: R55.2, U11.48 (IO), U13.1
- new net ~{ZXM1}: J6.48 (Pin_48)
- new net ~{ZXMREQ}: J6.32 (Pin_32), U11.27 (IO)
- new net ~{ZXRD}: J6.36 (Pin_36), U11.29 (IO)
- new net ~{ZXWR}: J6.38 (Pin_38), U11.30 (IO)
- no-connect marks 89 -> 95
Other:
- note added: "Power"
- note removed: "CPLD"
- note removed: "GENERAL SOUND"
- note removed: "TURBO SOUND FM"
- note removed: "open-drain"
- title: ZXEVO.1010 -> ZXEVO.1010 (TOP board)
- moved on the sheet: C11, C12, C13, C16, C17, C18, C19, C20, C22, C23, C24, C25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

Commit message: wip pcb rev.A
Parts:
- U4: footprint my:TQFP-44_14x14mm_P0.8mm -> my:Z80_FEC_VEC; ValueAlt (none) -> Z84C0020VEC
Changed lines of the file:
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@@
 		)
 		(property "Value" "Z84C0020FEC"
-			(at 95.885 243.205 0)
+			(at 96.266 241.808 0)
 			(effects
 				(font
@@
 			)
 		)
-		(property "Footprint" "my:TQFP-44_14x14mm_P0.8mm"
+		(property "Footprint" "my:Z80_FEC_VEC"
 			(at 85.09 269.24 0)
 			(effects
@@
 			)
 		)
+		(property "ValueAlt" "Z84C0020VEC"
+			(at 96.266 243.84 0)
+			(effects
+				(font
+					(size 1 1)
+				)
+			)
+		)

Commit message: wip pcb rev.A. Main board almost done
Parts:
- removed U24: EPM3064ATC100, Package_QFP:TQFP-100_14x14mm_P0.5mm, symbol my:EPM3064ATC100
- added U29: EPM3128ATC100, Package_QFP:TQFP-100_14x14mm_P0.5mm, symbol my:EPM3128ATC100
- added X3: 14 MHz, my:Oscillator_SMD_7050_7.0x5.0mm, symbol Oscillator:XO91
Connections:
- net +3V3: now also U29.18 (VCCIO), U29.3 (VCCIO), U29.34 (VCCIO), U29.39 (VCCINT), U29.51 (VCCIO), U29.66 (VCCIO), U29.82 (VCCIO), U29.91 (VCCINT)
- net +5V: now also X3.1 (EN), X3.4 (V+)
- net GND: now also U29.11 (GNDIO), U29.26 (GNDIO), U29.33 (GNDIO), U29.38 (GNDINT), U29.43 (GNDIO), U29.53 (GNDIO), U29.59 (GNDIO), U29.65 (GNDIO), U29.74 (GNDIO), U29.78 (GNDIO), U29.86 (GNDINT), U29.95 (GNDIO), X3.2 (GND)
- net ~{YMRST}: now reaches U16.11 (~{IC})
- net ~{YMRST}: now also U15.11 (~{IC})
- new net: U29.87 (GCLK1), X3.3 (OUT)
Other:
- note added: "NemoBus"
- note added: "NeoGS"
- moved on the sheet: C1, C11, C12, C13, C16, C17, C18, C19, C2, C20, C22, C23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

Commit message: wip pcb rev.A
Parts:
- removed C11, C12, C13, C16, C27, C9: 10u, Capacitor_Tantalum_SMD:CP_EIA-3216-18_Kemet-A_Pad1.58x1.35mm_HandSolder, symbol Device:C_Polarized
- removed C33: 22u, Capacitor_Tantalum_SMD:CP_EIA-3216-18_Kemet-A_Pad1.58x1.35mm_HandSolder, symbol Device:C_Polarized
- removed JP2: SolderJumper_2_Bridged, Jumper:SolderJumper-2_P1.3mm_Bridged_RoundedPad1.0x1.5mm, symbol Jumper:SolderJumper_2_Bridged
- removed R23, R25, R34: 10k, Resistor_SMD:R_0603_1608Metric_Pad0.98x0.95mm_HandSolder, symbol Device:R
- removed R27, R28: 47k, Resistor_SMD:R_0603_1608Metric_Pad0.98x0.95mm_HandSolder, symbol Device:R
- removed R63: 3.3k, Resistor_SMD:R_0805_2012Metric_Pad1.20x1.40mm_HandSolder, symbol Device:R
- removed U17: TDA1543, Package_DIP:DIP-8_W7.62mm, symbol my:TDA1543
- removed U19: TDA1543T, Package_SO:SOIC-16W_7.5x10.3mm_P1.27mm, symbol my:TDA1543T
- removed U21: 74ACT245, Package_SO:TSSOP-20_4.4x6.5mm_P0.65mm, symbol 74xx:74LS245
- removed U27: 1117-3.3, Package_TO_SOT_SMD:SOT-223-3_TabPin2, symbol Regulator_Linear:AZ1117-3.3
- removed Y1: 12 MHz, Crystal:Crystal_SMD_SeikoEpson_TSX3225-4Pin_3.2x2.5mm_HandSoldering, symbol Device:Crystal_GND24
- added C11, C27, C37, C38: 2.2n, Capacitor_SMD:C_0603_1608Metric_Pad1.08x0.95mm_HandSolder, symbol Device:C
- added C12, C13, C32, C33, C39, C40, C42, C43, C44, C45, C46, C47, C48, C49, C50, C51, C52, C53, C54, C55, C56, C57, C58, C59, C60, C61, C62, C63, C64, C65, C66, C67, C68, C69, C70, C71, C72, C73, C74, C75, C76, C77, C78, C79, C80, C81, C82, C83, C85, C86, C87, C88, C89, C90, C91, C92, C93, C94, C95, C96, C97, C98: 100n, Capacitor_SMD:C_0603_1608Metric_Pad1.08x0.95mm_HandSolder, symbol Device:C
- added C16, C30, C41: 10u, Capacitor_SMD:C_0805_2012Metric_Pad1.18x1.45mm_HandSolder, symbol Device:C
- added C34, C35: 22u, Capacitor_Tantalum_SMD:CP_EIA-3216-18_Kemet-A_Pad1.58x1.35mm_HandSolder, symbol Device:C_Polarized
- added C36, C9: 2.2u, Capacitor_SMD:C_0603_1608Metric_Pad1.08x0.95mm_HandSolder, symbol Device:C
- added C84: 47u, Capacitor_Tantalum_SMD:CP_EIA-3528-21_Kemet-B_Pad1.50x2.35mm_HandSolder, symbol Device:C_Polarized
- added JP3: Jumper, Connector_PinHeader_2.54mm:PinHeader_1x02_P2.54mm_Vertical, symbol Jumper:Jumper_2_Open
- added Q2: BC847, Package_TO_SOT_SMD:SOT-23, symbol Transistor_BJT:BC847
- added R60: 51, Resistor_SMD:R_0603_1608Metric_Pad0.98x0.95mm_HandSolder, symbol Device:R
- added U17: 74LVC2G04DB, Package_TO_SOT_SMD:SOT-23-6_Handsoldering, symbol 74xGxx:74LVC2G04
- added U27, U32: PCM5102A, Package_SO:TSSOP-20_4.4x6.5mm_P0.65mm, symbol Audio:PCM5102A
- added U30, U31: LP2985-3.3, Package_TO_SOT_SMD:SOT-23-5_HandSoldering, symbol Regulator_Linear:LP2985-3.3
- C5, C6: value 22p -> 100n
- R1, R2, R7: value 10k -> 6.8k
- R10, R12: value 47k -> 470
- R11: value 4.7k -> 6.8k
- R13: value 24k -> 470
- R15: value 24k -> 6.8k
- R47: value 6.8k -> 1k
- R8: value 10k -> 470
- X3: value 14 MHz -> 24 MHz
- Y2: footprint Crystal:Crystal_SMD_SeikoEpson_TSX3225-4Pin_3.2x2.5mm_HandSoldering -> my:Crystal_SMD_3225-4Pin_3.2x2.5mm_HandSoldering
Connections:
- net AY_B1 is gone; now on net MIDI_L: C17.1
- net AY_B2 is gone; now on net MA_LEFT: C18.1
- net AY_C1 is gone; now on net PSG_R: C22.1
- net AY_C2 is gone; now on net NGS_AOR: C23.1
- net DACCH2 is gone; now on net MA_RIGHT: C24.1
- net DACCH3 is gone; now on net MIDI_R: C25.1
- net FM1 is gone; now on net NGS_AOL: C19.1
- net FM2 is gone; now on net PSG_L: C20.1
- net GNDA is gone; now on net GND: C26.2, J1.3 (Pin_3), J1.4 (Pin_4), J4.R2, J4.S, U23.34 (AGND1), U23.37 (AGND34), U23.44 (AGND56), U5.13 (GND), U5.18 (GND), U5.25 (GND), U5.36 (GND), U5.4 (AGND), U5.45 (GND), U5.48 (GND), U5.49 (GND), U5.9 (GND), U9.37 (AGND), U9.40 (AGND), U9.41 (AGND), U9.47 (AGND)
- net ZXID0 is gone; now on net ZXD0: U11.41 (IO)
- net ZXID1 is gone; now on net ZXD1: U11.39 (IO)
- net ZXID2 is gone; now on net ZXD2: U11.38 (IO)
- net ZXID3 is gone; now on net ZXD3: U11.33 (IO)
- net ZXID4 is gone; now on net ZXD4: U11.32 (IO)
- net ZXID5 is gone; now on net ZXD5: U11.36 (IO)
- net ZXID6 is gone; now on net ZXD6: U11.37 (IO)
- net ZXID7 is gone; now on net ZXD7: U11.42 (IO/LOCK)
- net +1V8: now also C83.2, C85.2
- net +2V5: now also C5.2, C6.2, C70.2, C71.2, C72.2, C73.2, C74.2, C75.2
- net +3V3: now also C49.2, C50.2, C51.2, C52.2, C53.2, C54.2, C55.2, C56.2, C57.2, C58.2, C64.2, C65.2, C66.2, C67.2, C68.2, C69.2, C80.2, C81.2, C82.2, C84.1, C86.2, C87.2, C88.2, C89.2, C90.2, U27.17 (XSMT), U27.20 (DVDD), U32.17 (XSMT), U32.20 (DVDD)
- net +3V3A: now also C35.1, C91.2, C92.2, C93.2, C94.2, C95.2, C96.2, U27.1 (CPVDD), U27.8 (AVDD), U31.5 (VOUT), U32.1 (CPVDD), U32.8 (AVDD)
- net +3V3_MIDI: now also C34.1, C76.2, C77.2, C78.2, C79.2, U30.5 (VOUT)
- net +5V: now also U15.12 (5V/~{3V}), U15.27 (VDD), U16.12 (5V/~{3V}), U16.27 (VDD), C30.2, C42.2, C43.2, C44.2, C45.2, C46.2, C47.2, C48.2, C59.2, C60.2, C61.2, C62.2, C63.2, C97.2, C98.2, U17.5 (VCC), U30.1 (VIN), U30.3 (ON/~{OFF}), U31.1 (VIN), U31.3 (ON/~{OFF})
- net DAC_BITCK: now also U32.13 (BCK)
- net DAC_DAT: now also U32.14 (DIN)
- net DAC_LRCK: now also U32.15 (LRCK)
- net GND: now also C11.1, C12.1, C13.1, C16.1, C27.1, C30.1, C32.1, C33.1, C34.2, C35.2, C37.1, C38.1, C39.1, C40.1, C41.1, C42.1, C43.1, C44.1, C45.1, C46.1, C47.1, C48.1, C49.1, C50.1, C51.1, C52.1, C53.1, C54.1, C55.1, C56.1, C57.1, C58.1, C59.1, C60.1, C61.1, C62.1, C63.1, C64.1, C65.1, C66.1, C67.1, C68.1, C69.1, C70.1, C71.1, C72.1, C73.1, C74.1, C75.1, C76.1, C77.1, C78.1, C79.1, C80.1, C81.1, C82.1, C83.1, C84.2, C85.1, C86.1, C87.1, C88.1, C89.1, C90.1, C91.1, C92.1, C93.1, C94.1, C95.1, C96.1, C97.1, C98.1, Q2.2 (E), U17.2 (GND), U17.3, U27.10 (DEMP), U27.11 (FLT), U27.12 (SCK), U27.16 (FMT), U27.19 (DGND), U27.3 (CPGND), U27.9 (AGND), U30.2 (GND), U31.2 (GND), U32.10 (DEMP), U32.11 (FLT), U32.12 (SCK), U32.16 (FMT), U32.19 (DGND), U32.3 (CPGND), U32.9 (AGND)
- net MA_CLK: now also R60.1; no longer U11.128 (IO/DEV_OE)
- net MA_XTALI: now also C8.2, R59.1, U23.17 (XTALI), Y2.1; no longer C7.2, R59.2, U23.16 (XTALO), Y2.3
- net MA_XTALO: now also C7.2, R59.2, U23.16 (XTALO), Y2.3; no longer C8.2, R59.1, U23.17 (XTALI), Y2.1
- net MEMA14: now also U3.23 (A2); no longer U3.2 (A14)
- net MEMA15: now also U3.24 (A1); no longer U3.1 (A15)
- net MEMA16: now also U3.25 (A0); no longer U3.48 (A16)
- net MEMA17: now also U3.8 (A8); no longer U3.17 (A17)
- net MEMA18: now also U3.9 (A19); no longer U3.16 (A18)
- net MEMA19: now also U3.16 (A18); no longer U3.9 (A19)
- net MIXER_L: no longer R10.1, R12.1, R13.1, R15.1, R8.1
- net RA0: now also U3.48 (A16); no longer U3.25 (A0)
- net RA1: now also U3.1 (A15); no longer U3.24 (A1)
- net RA10: now also U3.19 (A6); no longer U3.6 (A10)
- net RA11: now also U3.20 (A5); no longer U3.5 (A11)
- net RA12: now also U3.21 (A4); no longer U3.4 (A12)
- net RA13: now also U3.22 (A3); no longer U3.3 (A13)
- net RA2: now also U3.2 (A14); no longer U3.23 (A2)
- net RA3: now also U3.3 (A13); no longer U3.22 (A3)
- net RA4: now also U3.4 (A12); no longer U3.21 (A4)
- net RA5: now also U3.5 (A11); no longer U3.20 (A5)
- net RA6: now also U3.6 (A10); no longer U3.19 (A6)
- net RA7: now also U3.7 (A9); no longer U3.18 (A7)
- net RA8: now also U3.17 (A17); no longer U3.8 (A8)
- net RA9: now also U3.18 (A7); no longer U3.7 (A9)
- net RD0: now also U3.44 (D7); no longer U3.29 (D0)
- net RD1: now also U3.42 (D6); no longer U3.31 (D1)
- net RD2: now also U3.40 (D5); no longer U3.33 (D2)
- net RD3: now also U3.38 (D4); no longer U3.35 (D3)
- net RD4: now also U3.35 (D3); no longer U3.38 (D4)
- net RD5: now also U3.33 (D2); no longer U3.40 (D5)
- net RD6: now also U3.31 (D1); no longer U3.42 (D6)
- net RD7: now also U3.29 (D0); no longer U3.44 (D7)
- net TCK: now also U29.62 (TCK)
- net TMS: now also U29.15 (TMS)
- net YMA0: now also U29.6 (I/O)
- net YMA1: now also U29.7 (I/O)
- net YMCK: now also U29.14 (I/O)
- net YMD0: now also U29.16 (I/O)
- net YMD1: now also U29.17 (I/O)
- net YMD2: now also U29.19 (I/O)
- net YMD3: now also U29.20 (I/O)
- net YMD4: now also U29.21 (I/O)
- net YMD5: now also U29.22 (I/O)
- net YMD6: now also U29.23 (I/O)
- net YMD7: now also U29.24 (I/O)
- net ZXA0: now also U29.64 (I/O)
- net ZXA1: now also U29.61 (I/O)
- net ZXA13: now also U29.70 (I/O)
- net ZXA14: now also U29.71 (I/O)
- net ZXA15: now also U29.72 (I/O)
- net ZXA2: now also U29.58 (I/O)
- net ZXA3: now also U29.56 (I/O)
- net ZXA4: now also U29.45 (I/O)
- net ZXA5: now also U29.46 (I/O)
- net ZXA6: now also U29.47 (I/O)
- net ZXA7: now also U29.48 (I/O)
- net ZXD0: now also U29.68 (I/O)
- net ZXD1: now also U29.67 (I/O)
- net ZXD2: now also U29.63 (I/O)
- net ZXD3: now also U29.55 (I/O)
- net ZXD4: now also U29.54 (I/O)
- net ZXD5: now also U29.57 (I/O)
- net ZXD6: now also U29.60 (I/O)
- net ZXD7: now also U29.69 (I/O)
- net ~{RESET}: no longer U5.38 (~{RST}/~{PD})
- net ~{WARMRES}: now also JP3.2 (B)
- net ~{YMCS0}: now also U29.98 (I/O)
- net ~{YMCS1}: now also U29.8 (I/O)
- net ~{YMRD}: now also U29.5 (I/O)
- net ~{YMRST}: now also U29.25 (I/O)
- net ~{YMWR}: now also U29.2 (I/O)
- net ~{ZXIORQ}: now also U29.52 (I/O)
- net ~{ZXM1}: now also U29.44 (I/O)
- net ~{ZXRD}: now also U29.88 (OE1)
- net ~{ZXRES}: now also U29.89 (GCLRn), U17.1
- net ~{ZXWR}: now also U29.49 (I/O)
- net at R15.2: now also U17.6
- net NGS_AOL: now reaches R12.2
- net NGS_AOL: now also C38.2
- net YMDO1: now reaches U29.10 (I/O)
- net YMDO1: now also U16.24 (DO)
- net YMBCO0: now reaches U29.100 (I/O)
- net YMBCO0: now also U15.23 (BCO)
- net YMWCO1: now reaches U29.12 (I/O)
- net YMWCO1: now also U16.25 (WCO)
- net YMLRO1: now reaches U29.13 (I/O)
- net YMLRO1: now also U16.26 (LRO)
- net PSG_LRCK: now reaches U29.27 (I/O)
- net PSG_LRCK: now also U27.15 (LRCK)
- net PSG_DIN: now reaches U29.28 (I/O)
- net PSG_DIN: now also U27.14 (DIN)
- net PSG_BCK: now reaches U29.29 (I/O)
- net PSG_BCK: now also U27.13 (BCK)
- net at U29.87 (GCLK1): no longer X3.3 (OUT)
- net YMBCO1: now reaches U29.9 (I/O)
- net YMBCO1: now also U16.23 (BCO)
- net at U29.90 (OE2/GCLK2): now also X3.3 (OUT)
- net MIDI_CLK: now reaches U29.92 (I/O)
- net MIDI_CLK: now also U5.39 (X1)
- net ~{MIDI_RST}: now reaches U29.93 (I/O)
- net ~{MIDI_RST}: now also U5.38 (~{RST}/~{PD})
- net YMLRO0: now reaches U29.96 (I/O)
- net YMLRO0: now also U15.26 (LRO)
- net YMWCO0: now reaches U29.97 (I/O)
- net YMWCO0: now also U15.25 (WCO)
- net YMDO0: now reaches U29.99 (I/O)
- net YMDO0: now also U15.24 (DO)
- net PSG_L: now reaches R8.2
- net PSG_L: now also C11.2
- net PSG_R: now reaches R10.2
- net PSG_R: now also C27.2
- net NGS_AOR: now reaches R13.2
- net NGS_AOR: now also C37.2
- net at U5.40 (X2): no longer C5.2
- net ZXBUSIN: no longer names the net of U11.43 (IO)
- net ~{ZXBUSENA}: no longer names the net of U11.44 (IO)
- new net: R13.1, U32.7 (OUTR)
- new net: JP3.1 (A), Q2.3 (C)
- new net: C13.2, C16.2, U27.18 (LDOO)
- new net: C40.2, C41.2, U32.18 (LDOO)
- new net: C36.1, U32.4 (CAPM)
- new net: C36.2, U32.2 (CAPP)
- new net: C39.2, U32.5 (VNEG)
- new net: R60.2, U11.128 (IO/DEV_OE)
- new net: C33.2, U31.4 (BP)
- new net: R8.1, U27.6 (OUTL)
- new net: C9.2, U27.2 (CAPP)
- new net: C9.1, U27.4 (CAPM)
- new net: C12.2, U27.5 (VNEG)
- new net: R10.1, U27.7 (OUTR)
- new net: C32.2, U30.4 (BP)
- new net: Q2.1 (B), R15.1
- new net: R12.1, U32.6 (OUTL)
- no-connect marks 95 -> 107
Other:
- note added: "PSG + FM + SounDrive"
- moved on the sheet: C1, C10, C15, C17, C18, C19, C2, C20, C22, C23, C24, C25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

Commit message: wip pcb rev.A
Parts:
- removed U20: ESP32-WROOM-32, RF_Module:ESP32-WROOM-32, symbol RF_Module:ESP32-WROOM-32
- added C99: 100u, Capacitor_SMD:CP_Elec_5x5.9, symbol Device:C_Polarized
- U11: footprint Package_QFP:TQFP-144_20x20mm_P0.5mm -> PCM_Package_QFP_AKL:TQFP-144_20x20mm_P0.5mm
Connections:
- net +3V3: now also C99.1
- net GND: now also C99.2
- net ZXA0: now also U29.57 (I/O); no longer U29.64 (I/O)
- net ZXA1: now also U29.56 (I/O); no longer U29.61 (I/O)
- net ZXA13: now also U29.58 (I/O); no longer U29.70 (I/O)
- net ZXA14: now also U29.60 (I/O); no longer U29.71 (I/O)
- net ZXA15: now also U29.61 (I/O); no longer U29.72 (I/O)
- net ZXA2: now also U29.55 (I/O); no longer U29.58 (I/O)
- net ZXA3: now also U29.54 (I/O); no longer U29.56 (I/O)
- net ZXD0: now also U29.32 (I/O); no longer U29.68 (I/O)
- net ZXD1: now also U29.35 (I/O); no longer U29.67 (I/O)
- net ZXD2: now also U29.36 (I/O); no longer U29.63 (I/O)
- net ZXD3: now also U29.41 (I/O); no longer U29.55 (I/O)
- net ZXD4: now also U29.42 (I/O); no longer U29.54 (I/O)
- net ZXD5: now also U29.40 (I/O); no longer U29.57 (I/O)
- net ZXD6: now also U29.37 (I/O); no longer U29.60 (I/O)
- net ZXD7: now also U29.31 (I/O); no longer U29.69 (I/O)
- net ~{ZXIORQ}: no longer U29.52 (I/O)
- net ~{ZXMREQ}: now also U29.52 (I/O)
- net ~{ZXRD}: now also U29.50 (I/O); no longer U29.88 (OE1)
Other:
- moved on the sheet: C10, C15, C21, C28, C29, C30, C31, C32, C33, C34, C35, U26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
