File: pcb_top/rev.A/zxevo1010_top.kicad_sch (KiCad schematic)
At the start: 196 parts, among them J1 Conn_02x05_Odd_Even, J2 Conn_02x05_Odd_Even, J3 Conn_02x05_Odd_Even, J4 PJ-320, J6 Conn_02x30_Row_Letter_First, Q1 BSS138, Q2 BC847, U1 ESP-12E, U10 EPM3064ATC100, U11 EP1K30TC144, U12 74AHCT1G125DB, U13 74AHCT1G125DB, U14 74AHCT1G125DB, U15 YMF288-M, U16 YMF288-M, U17 74LVC2G04DB, U18 MAX809LEUR, U2 CY62167EV30LL-45ZXI, U22 74LXC245, U23 MA8201, U25 1117-3.3, U26 1117-2.5, U27 PCM5102A, U28 1117-1.8, U29 EPM3128ATC100, U3 CY62167EV30LL-45ZXI, U30 LP2985-3.3, U31 LP2985-3.3, U32 PCM5102A, U4 Z84C0020FEC, U5 SAM2695, U6 29F040, U7 74LVC1G04DB, U8 74AHCT1G125DB, U9 VS1053b, X1 20 MHz, X2 24 MHz, X3 24 MHz, Y2 14 MHz

Commit message: wip pcb rev.A
Parts:
- added TP1, TP2, TP3: TestPoint, TestPoint:TestPoint_Pad_D1.0mm, symbol Connector:TestPoint
- C5, C6, C64, C65, C66, C67, C68, C69, C70, C71, C72, C73, C74, C75, C80, C81: footprint Capacitor_SMD:C_0603_1608Metric_Pad1.08x0.95mm_HandSolder -> Capacitor_SMD:C_0805_2012Metric_Pad1.18x1.45mm_HandSolder
Connections:
- net A0: now also U22.18 (B0); no longer U22.14 (B4)
- net A1: now also U22.17 (B1); no longer U22.15 (B3)
- net A3: now also U22.15 (B3); no longer U22.17 (B1)
- net A4: now also U22.14 (B4); no longer U22.18 (B0)
- net MEMA15: now also U2.48 (A16), U3.25 (A0); no longer U2.1 (A15), U3.24 (A1)
- net MEMA16: now also U2.1 (A15), U3.24 (A1); no longer U2.48 (A16), U3.25 (A0)
- net RA0: now also U22.2 (A0); no longer U22.6 (A4)
- net RA1: now also U22.3 (A1); no longer U22.5 (A3)
- net RA3: now also U22.5 (A3); no longer U22.3 (A1)
- net RA4: now also U22.6 (A4); no longer U22.2 (A0)
- net at U29.1 (I/O): now also TP2.1
- net at U29.30 (I/O): now also TP1.1
- net at U29.75 (I/O): now also TP3.1
- net +12V: no longer names the net of J6.58 (Pin_58)
- no-connect marks 107 -> 108
Changed lines of the file:
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@@
 	)
 	(no_connect
+		(at 486.41 96.52)
+	)
+	(no_connect
 		(at 341.63 374.65)
 	)
@@
 	)
 	(label "MEMA15"
-		(at 247.65 246.38 0)
+		(at 247.65 243.84 0)
 		(fields_autoplaced yes)
 		(effects
@@
 	)
 	(label "A3"
-		(at 172.72 193.04 0)
+		(at 172.72 198.12 0)
 		(fields_autoplaced yes)
 		(effects
@@
 	)
 	(label "RA1"
-		(at 215.9 198.12 180)
+		(at 215.9 193.04 180)
 		(fields_autoplaced yes)
 		(effects
@@
 	)
 	(label "MEMA15"
-		(at 196.85 281.94 0)
+		(at 196.85 284.48 0)
 		(fields_autoplaced yes)
 		(effects
@@
 	)
 	(label "RA3"
-		(at 215.9 193.04 180)
+		(at 215.9 198.12 180)
 		(fields_autoplaced yes)
 		(effects
@@
 	)
 	(label "A0"
-		(at 172.72 200.66 0)
+		(at 172.72 190.5 0)
 		(fields_autoplaced yes)
 		(effects
@@
 	)
 	(label "A1"
-		(at 172.72 198.12 0)
+		(at 172.72 193.04 0)
 		(fields_autoplaced yes)
 		(effects
@@
 	)
 	(label "MEMA16"
-		(at 196.85 284.48 0)
+		(at 196.85 281.94 0)
 		(fields_autoplaced yes)
 		(effects
@@
 	)
 	(label "MEMA16"
-		(at 247.65 243.84 0)
+		(at 247.65 246.38 0)
 		(fields_autoplaced yes)
 		(effects
@@
 	)
 	(label "RA4"
-		(at 215.9 190.5 180)
+		(at 215.9 200.66 180)
 		(fields_autoplaced yes)
 		(effects
@@
 	)
 	(label "A4"
-		(at 172.72 190.5 0)
+		(at 172.72 200.66 0)
 		(fields_autoplaced yes)
 		(effects
@@
 	)
 	(label "RA0"
-		(at 215.9 200.66 180)
+		(at 215.9 190.5 180)
 		(fields_autoplaced yes)
 		(effects
@@
 	)
 	(symbol
+		(lib_id "Connector:TestPoint")
+		(at 193.04 433.07 90)
+		(unit 1)
+		(exclude_from_sim no)
+		(in_bom no)
+		(on_board yes)
+		(dnp no)
+		(property "Reference" "TP1"
+			(at 186.055 433.07 90)
+			(effects
+				(font
+					(size 1 1)
+				)
+			)
+		)
+		(property "Value" "TestPoint"
+			(at 189.738 429.895 90)
+			(effects
+				(font
+					(size 1 1)
+				)
+				(hide yes)
+			)
+		)
+		(property "Footprint" "TestPoint:TestPoint_Pad_D1.0mm"
+			(at 193.04 427.99 0)
+			(effects
+				(font
+					(size 1.27 1.27)
+				)
+				(hide yes)
+			)
+		)
+		(property "Datasheet" "~"
+			(at 193.04 427.99 0)
+			(effects
+				(font
+					(size 1.27 1.27)
+				)
+				(hide yes)
+			)
+		)
+		(property "Description" ""
+			(at 193.04 433.07 0)
+			(effects
+				(font
+					(size 1.27 1.27)
+				)
+				(hide yes)
+			)
+		)
+		(pin "1"
+		)
+		(instances
+			(project "zxevo1010_top"
+				(path "/895fa090-e1df-4200-a112-cb7c4b9368aa"
+					(reference "TP1")
+					(unit 1)
+				)
+			)
+		)
+	)
+	(symbol
 		(lib_id "Device:R")
 		(at 402.59 295.91 270)
@@
 			)
 		)
-		(property "Footprint" "Capacitor_SMD:C_0603_1608Metric_Pad1.08x0.95mm_HandSolder"
+		(property "Footprint" "Capacitor_SMD:C_0805_2012Metric_Pad1.18x1.45mm_HandSolder"
 			(at 209.8548 561.34 0)
 			(effects
@@
 	)
 	(symbol
-		(lib_id "power:+12V")
-		(at 486.41 96.52 270)
-		(unit 1)
-		(exclude_from_sim no)
-		(in_bom yes)
-		(on_board yes)
-		(dnp no)
-		(property "Reference" "#PWR064"
-			(at 482.6 96.52 0)
-			(effects
-				(font
-					(size 1 1)
-				)
-				(hide yes)
-			)
-		)
-		(property "Value" "+12V"
-			(at 489.585 96.52 90)
-			(effects
-				(font
-					(size 1 1)
-				)
-				(justify left)
-			)
-		)
-		(property "Footprint" ""
-			(at 486.41 96.52 0)
-			(effects
-				(font
-					(size 1.27 1.27)
-				)
-				(hide yes)
-			)
-		)
-		(property "Datasheet" ""
-			(at 486.41 96.52 0)
-			(effects
-				(font
-					(size 1.27 1.27)
-				)
-				(hide yes)
-			)
-		)
-		(property "Description" "Power symbol creates a global label with name \"+12V\""
-			(at 486.41 96.52 0)
-			(effects
-				(font
-					(size 1.27 1.27)
-				)
-				(hide yes)
-			)
-		)
-		(pin "1"
-		)
-		(instances
-			(project "zxevo1010"
-				(path "/895fa090-e1df-4200-a112-cb7c4b9368aa"
-					(reference "#PWR064")
-					(unit 1)
-				)
-			)
-		)
-	)
-	(symbol
 		(lib_id "74xGxx:74LVC2G04")
 		(at 290.83 207.01 0)
@@
 			)
 		)
-		(property "Footprint" "Capacitor_SMD:C_0603_1608Metric_Pad1.08x0.95mm_HandSolder"
+		(property "Footprint" "Capacitor_SMD:C_0805_2012Metric_Pad1.18x1.45mm_HandSolder"
 			(at 197.1548 561.34 0)
 			(effects
@@
 			)
 		)
-		(property "Footprint" "Capacitor_SMD:C_0603_1608Metric_Pad1.08x0.95mm_HandSolder"
+		(property "Footprint" "Capacitor_SMD:C_0805_2012Metric_Pad1.18x1.45mm_HandSolder"
 			(at 184.4548 561.34 0)
 			(effects
@@
 			)
 		)
-		(property "Footprint" "Capacitor_SMD:C_0603_1608Metric_Pad1.08x0.95mm_HandSolder"
+		(property "Footprint" "Capacitor_SMD:C_0805_2012Metric_Pad1.18x1.45mm_HandSolder"
 			(at 171.7548 561.34 0)
 			(effects
@@
 			)
 		)
-		(property "Footprint" "Capacitor_SMD:C_0603_1608Metric_Pad1.08x0.95mm_HandSolder"
+		(property "Footprint" "Capacitor_SMD:C_0805_2012Metric_Pad1.18x1.45mm_HandSolder"
 			(at 216.2048 561.34 0)
 			(effects
@@
 			)
 		)
-		(property "Footprint" "Capacitor_SMD:C_0603_1608Metric_Pad1.08x0.95mm_HandSolder"
+		(property "Footprint" "Capacitor_SMD:C_0805_2012Metric_Pad1.18x1.45mm_HandSolder"
 			(at 277.1648 561.34 0)
 			(effects
@@
 			)
 		)
-		(property "Footprint" "Capacitor_SMD:C_0603_1608Metric_Pad1.08x0.95mm_HandSolder"
+		(property "Footprint" "Capacitor_SMD:C_0805_2012Metric_Pad1.18x1.45mm_HandSolder"
 			(at 296.2148 561.34 0)
 			(effects
@@
 			)
 		)
-		(property "Footprint" "Capacitor_SMD:C_0603_1608Metric_Pad1.08x0.95mm_HandSolder"
+		(property "Footprint" "Capacitor_SMD:C_0805_2012Metric_Pad1.18x1.45mm_HandSolder"
 			(at 315.2648 561.34 0)
 			(effects
@@
 			)
 		)
-		(property "Footprint" "Capacitor_SMD:C_0603_1608Metric_Pad1.08x0.95mm_HandSolder"
+		(property "Footprint" "Capacitor_SMD:C_0805_2012Metric_Pad1.18x1.45mm_HandSolder"
 			(at 190.8048 561.34 0)
 			(effects
@@
 			)
 		)
-		(property "Footprint" "Capacitor_SMD:C_0603_1608Metric_Pad1.08x0.95mm_HandSolder"
+		(property "Footprint" "Capacitor_SMD:C_0805_2012Metric_Pad1.18x1.45mm_HandSolder"
 			(at 308.9148 561.34 0)
 			(effects
@@
 			)
 		)
-		(property "Footprint" "Capacitor_SMD:C_0603_1608Metric_Pad1.08x0.95mm_HandSolder"
+		(property "Footprint" "Capacitor_SMD:C_0805_2012Metric_Pad1.18x1.45mm_HandSolder"
 			(at 270.8148 561.34 0)
 			(effects
@@
 			)
 		)
-		(property "Footprint" "Capacitor_SMD:C_0603_1608Metric_Pad1.08x0.95mm_HandSolder"
+		(property "Footprint" "Capacitor_SMD:C_0805_2012Metric_Pad1.18x1.45mm_HandSolder"
 			(at 203.5048 561.34 0)
 			(effects
@@
 			)
 		)
-		(property "Footprint" "Capacitor_SMD:C_0603_1608Metric_Pad1.08x0.95mm_HandSolder"
+		(property "Footprint" "Capacitor_SMD:C_0805_2012Metric_Pad1.18x1.45mm_HandSolder"
 			(at 283.5148 561.34 0)
 			(effects
@@
 			)
 		)
-		(property "Footprint" "Capacitor_SMD:C_0603_1608Metric_Pad1.08x0.95mm_HandSolder"
+		(property "Footprint" "Capacitor_SMD:C_0805_2012Metric_Pad1.18x1.45mm_HandSolder"
 			(at 289.8648 561.34 0)
 			(effects
@@
 	)
 	(symbol
+		(lib_id "Connector:TestPoint")
+		(at 193.04 369.57 90)
+		(unit 1)
+		(exclude_from_sim no)
+		(in_bom no)
+		(on_board yes)
+		(dnp no)
+		(property "Reference" "TP2"
+			(at 186.055 369.57 90)
+			(effects
+				(font
+					(size 1 1)
+				)
+			)
+		)
+		(property "Value" "TestPoint"
+			(at 189.738 366.395 90)
+			(effects
+				(font
+					(size 1 1)
+				)
+				(hide yes)
+			)
+		)
+		(property "Footprint" "TestPoint:TestPoint_Pad_D1.0mm"
+			(at 193.04 364.49 0)
+			(effects
+				(font
+					(size 1.27 1.27)
+				)
+				(hide yes)
+			)
+		)
+		(property "Datasheet" "~"
+			(at 193.04 364.49 0)
+			(effects
+				(font
+					(size 1.27 1.27)
+				)
+				(hide yes)
+			)
+		)
+		(property "Description" ""
+			(at 193.04 369.57 0)
+			(effects
+				(font
+					(size 1.27 1.27)
+				)
+				(hide yes)
+			)
+		)
+		(pin "1"
+		)
+		(instances
+			(project "zxevo1010_top"
+				(path "/895fa090-e1df-4200-a112-cb7c4b9368aa"
+					(reference "TP2")
+					(unit 1)
+				)
+			)
+		)
+	)
+	(symbol
 		(lib_id "Device:C_Polarized")
 		(at 466.09 243.84 90)
@@
 			)
 		)
-		(property "Footprint" "Capacitor_SMD:C_0603_1608Metric_Pad1.08x0.95mm_HandSolder"
+		(property "Footprint" "Capacitor_SMD:C_0805_2012Metric_Pad1.18x1.45mm_HandSolder"
 			(at 178.1048 561.34 0)
 			(effects
@@
 			)
 		)
-		(property "Footprint" "Capacitor_SMD:C_0603_1608Metric_Pad1.08x0.95mm_HandSolder"
+		(property "Footprint" "Capacitor_SMD:C_0805_2012Metric_Pad1.18x1.45mm_HandSolder"
 			(at 302.5648 561.34 0)
 			(effects
@@
 					(unit 1)
 				)
+			)
+		)
+	)
+	(symbol
+		(lib_id "Connector:TestPoint")
+		(at 243.84 417.83 270)
+		(unit 1)
+		(exclude_from_sim no)
+		(in_bom no)
+		(on_board yes)
+		(dnp no)
+		(property "Reference" "TP3"
+			(at 250.825 417.83 90)
+			(effects
+				(font
+					(size 1 1)
+				)
+			)
+		)
+		(property "Value" "TestPoint"
+			(at 247.142 421.005 90)
+			(effects
+				(font
+					(size 1 1)
+				)
+				(hide yes)
+			)
+		)
+		(property "Footprint" "TestPoint:TestPoint_Pad_D1.0mm"
+			(at 243.84 422.91 0)
+			(effects
+				(font
+					(size 1.27 1.27)
+				)
+				(hide yes)
+			)
+		)
+		(property "Datasheet" "~"
+			(at 243.84 422.91 0)
+			(effects
+				(font
+					(size 1.27 1.27)
+				)
+				(hide yes)
+			)
+		)
+		(property "Description" ""
+			(at 243.84 417.83 0)
+			(effects
+				(font
+					(size 1.27 1.27)
+				)
+				(hide yes)
+			)
+		)
+		(pin "1"
+		)
+		(instances
+			(project "zxevo1010_top"
+				(path "/895fa090-e1df-4200-a112-cb7c4b9368aa"
+					(reference "TP3")
+					(unit 1)
+				)

Commit message: wip pcb rev.A
Connections:
- net MEMA14: now also U2.9 (A19), U3.16 (A18); no longer U2.2 (A14), U3.23 (A2)
- net MEMA15: now also U2.2 (A14), U3.23 (A2); no longer U2.48 (A16), U3.25 (A0)
- net MEMA16: now also U2.3 (A13), U3.22 (A3); no longer U2.1 (A15), U3.24 (A1)
- net MEMA17: now also U2.16 (A18), U3.9 (A19); no longer U2.17 (A17), U3.8 (A8)
- net MEMA18: now also U2.4 (A12), U3.21 (A4); no longer U2.16 (A18), U3.9 (A19)
- net MEMA19: now also U2.1 (A15), U3.24 (A1); no longer U2.9 (A19), U3.16 (A18)
- net MEMA21: now also U2.17 (A17), U3.8 (A8); no longer U2.45 (A20/D15), U3.45 (A20/D15)
- net RA10: now also U2.5 (A11), U3.20 (A5); no longer U2.6 (A10), U3.19 (A6)
- net RA11: now also U2.6 (A10), U3.19 (A6); no longer U2.5 (A11), U3.20 (A5)
- net RA12: now also U2.7 (A9), U3.18 (A7); no longer U2.4 (A12), U3.21 (A4)
- net RA13: now also U2.8 (A8), U3.17 (A17); no longer U2.3 (A13), U3.22 (A3)
- net RA6: now also U2.45 (A20/D15), U3.45 (A20/D15); no longer U2.19 (A6), U3.6 (A10)
- net RA7: now also U2.48 (A16), U3.25 (A0); no longer U2.18 (A7), U3.7 (A9)
- net RA8: now also U2.19 (A6), U3.6 (A10); no longer U2.8 (A8), U3.17 (A17)
- net RA9: now also U2.18 (A7), U3.7 (A9); no longer U2.7 (A9), U3.18 (A7)
- net RD0: now also U2.42 (D6), U3.31 (D1); no longer U2.29 (D0), U3.44 (D7)
- net RD1: now also U2.44 (D7), U3.29 (D0); no longer U2.31 (D1), U3.42 (D6)
- net RD2: now also U2.38 (D4), U3.35 (D3); no longer U2.33 (D2), U3.40 (D5)
- net RD3: now also U2.40 (D5), U3.33 (D2); no longer U2.35 (D3), U3.38 (D4)
- net RD4: now also U2.35 (D3), U3.38 (D4); no longer U2.38 (D4), U3.35 (D3)
- net RD5: now also U2.33 (D2), U3.40 (D5); no longer U2.40 (D5), U3.33 (D2)
- net RD6: now also U2.29 (D0), U3.44 (D7); no longer U2.42 (D6), U3.31 (D1)
- net RD7: now also U2.31 (D1), U3.42 (D6); no longer U2.44 (D7), U3.29 (D0)
Changed lines of the file:
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@@
 	)
 	(label "RA11"
-		(at 196.85 271.78 0)
+		(at 196.85 269.24 0)
 		(fields_autoplaced yes)
 		(effects
@@
 	)
 	(label "RD2"
-		(at 294.64 256.54 180)
+		(at 294.64 251.46 180)
 		(fields_autoplaced yes)
 		(effects
@@
 	)
 	(label "RD5"
-		(at 294.64 248.92 180)
+		(at 294.64 256.54 180)
 		(fields_autoplaced yes)
 		(effects
@@
 	)
 	(label "RA8"
-		(at 247.65 287.02 0)
+		(at 247.65 269.24 0)
 		(fields_autoplaced yes)
 		(effects
@@
 	)
 	(label "RA9"
-		(at 196.85 266.7 0)
+		(at 196.85 261.62 0)
 		(fields_autoplaced yes)
 		(effects
@@
 	)
 	(label "MEMA15"
-		(at 247.65 243.84 0)
+		(at 247.65 248.92 0)
 		(fields_autoplaced yes)
 		(effects
@@
 	)
 	(label "RD3"
-		(at 243.84 251.46 180)
+		(at 243.84 256.54 180)
 		(fields_autoplaced yes)
 		(effects
@@
 	)
 	(label "MEMA21"
-		(at 243.84 288.29 180)
+		(at 196.85 287.02 0)
 		(fields_autoplaced yes)
 		(effects
@@
 				(size 1 1)
 			)
-			(justify right bottom)
+			(justify left bottom)
 		)
 	)
@@
 	)
 	(label "RA13"
-		(at 247.65 251.46 0)
+		(at 247.65 287.02 0)
 		(fields_autoplaced yes)
 		(effects
@@
 	)
 	(label "RD3"
-		(at 294.64 254 180)
+		(at 294.64 248.92 180)
 		(fields_autoplaced yes)
 		(effects
@@
 	)
 	(label "MEMA15"
-		(at 196.85 284.48 0)
+		(at 196.85 279.4 0)
 		(fields_autoplaced yes)
 		(effects
@@
 	)
 	(label "RA13"
-		(at 196.85 276.86 0)
+		(at 196.85 264.16 0)
 		(fields_autoplaced yes)
 		(effects
@@
 	)
 	(label "RA6"
-		(at 247.65 269.24 0)
+		(at 294.64 288.29 180)
 		(fields_autoplaced yes)
 		(effects
@@
 				(size 1 1)
 			)
-			(justify left bottom)
+			(justify right bottom)
 		)
 	)
@@
 	)
 	(label "RA10"
-		(at 196.85 269.24 0)
+		(at 196.85 271.78 0)
 		(fields_autoplaced yes)
 		(effects
@@
 	)
 	(label "RA7"
-		(at 196.85 261.62 0)
+		(at 196.85 284.48 0)
 		(fields_autoplaced yes)
 		(effects
@@
 	)
 	(label "RA6"
-		(at 196.85 259.08 0)
+		(at 243.84 288.29 180)
 		(fields_autoplaced yes)
 		(effects
@@
 				(size 1 1)
 			)
-			(justify left bottom)
+			(justify right bottom)
 		)
 	)
@@
 	)
 	(label "RD4"
-		(at 243.84 254 180)
+		(at 243.84 251.46 180)
 		(fields_autoplaced yes)
 		(effects
@@
 	)
 	(label "MEMA16"
-		(at 196.85 281.94 0)
+		(at 196.85 276.86 0)
 		(fields_autoplaced yes)
 		(effects
@@
 	)
 	(label "RD7"
-		(at 294.64 243.84 180)
+		(at 294.64 259.08 180)
 		(fields_autoplaced yes)
 		(effects
@@
 	)
 	(label "MEMA17"
-		(at 247.65 264.16 0)
+		(at 247.65 292.1 0)
 		(fields_autoplaced yes)
 		(effects
@@
 	)
 	(label "RD0"
-		(at 294.64 261.62 180)
+		(at 294.64 246.38 180)
 		(fields_autoplaced yes)
 		(effects
@@
 	)
 	(label "RA7"
-		(at 247.65 266.7 0)
+		(at 247.65 243.84 0)
 		(fields_autoplaced yes)
 		(effects
@@
 	)
 	(label "RA12"
-		(at 196.85 274.32 0)
+		(at 196.85 266.7 0)
 		(fields_autoplaced yes)
 		(effects
@@
 	)
 	(label "MEMA14"
-		(at 247.65 248.92 0)
+		(at 247.65 289.56 0)
 		(fields_autoplaced yes)
 		(effects
@@
 	)
 	(label "MEMA17"
-		(at 196.85 287.02 0)
+		(at 196.85 289.56 0)
 		(fields_autoplaced yes)
 		(effects
@@
 	)
 	(label "RD1"
-		(at 294.64 259.08 180)
+		(at 294.64 243.84 180)
 		(fields_autoplaced yes)
 		(effects
@@
 	)
 	(label "MEMA21"
-		(at 294.64 288.29 180)
+		(at 247.65 264.16 0)
 		(fields_autoplaced yes)
 		(effects
@@
 				(size 1 1)
 			)
-			(justify right bottom)
+			(justify left bottom)
 		)
 	)
@@
 	)
 	(label "MEMA16"
-		(at 247.65 246.38 0)
+		(at 247.65 251.46 0)
 		(fields_autoplaced yes)
 		(effects
@@
 	)
 	(label "RD0"
-		(at 243.84 243.84 180)
+		(at 243.84 259.08 180)
 		(fields_autoplaced yes)
 		(effects
@@
 	)
 	(label "RD5"
-		(at 243.84 256.54 180)
+		(at 243.84 248.92 180)
 		(fields_autoplaced yes)
 		(effects
@@
 	)
 	(label "RA8"
-		(at 196.85 264.16 0)
+		(at 196.85 259.08 0)
 		(fields_autoplaced yes)
 		(effects
@@
 	)
 	(label "RD7"
-		(at 243.84 261.62 180)
+		(at 243.84 246.38 180)
 		(fields_autoplaced yes)
 		(effects
@@
 	)
 	(label "RA10"
-		(at 247.65 259.08 0)
+		(at 247.65 256.54 0)
 		(fields_autoplaced yes)
 		(effects
@@
 	)
 	(label "MEMA19"
-		(at 196.85 292.1 0)
+		(at 196.85 281.94 0)
 		(fields_autoplaced yes)
 		(effects
@@
 	)
 	(label "RA12"
-		(at 247.65 254 0)
+		(at 247.65 261.62 0)
 		(fields_autoplaced yes)
 		(effects
@@
 	)
 	(label "MEMA19"
-		(at 247.65 289.56 0)
+		(at 247.65 246.38 0)
 		(fields_autoplaced yes)
 		(effects
@@
 	)
 	(label "MEMA14"
-		(at 196.85 279.4 0)
+		(at 196.85 292.1 0)
 		(fields_autoplaced yes)
 		(effects
@@
 	)
 	(label "MEMA18"
-		(at 247.65 292.1 0)
+		(at 247.65 254 0)
 		(fields_autoplaced yes)
 		(effects
@@
 	)
 	(label "RD2"
-		(at 243.84 248.92 180)
+		(at 243.84 254 180)
 		(fields_autoplaced yes)
 		(effects
@@
 	)
 	(label "RD6"
-		(at 294.64 246.38 180)
+		(at 294.64 261.62 180)
 		(fields_autoplaced yes)
 		(effects
@@
 	)
 	(label "RD4"
-		(at 294.64 251.46 180)
+		(at 294.64 254 180)
 		(fields_autoplaced yes)
 		(effects
@@
 	)
 	(label "RA9"
-		(at 247.65 261.62 0)
+		(at 247.65 266.7 0)
 		(fields_autoplaced yes)
 		(effects
@@
 	)
 	(label "MEMA18"
-		(at 196.85 289.56 0)
+		(at 196.85 274.32 0)
 		(fields_autoplaced yes)
 		(effects
@@
 	)
 	(label "RD1"
-		(at 243.84 246.38 180)
+		(at 243.84 261.62 180)
 		(fields_autoplaced yes)
 		(effects
@@
 	)
 	(label "RD6"
-		(at 243.84 259.08 180)
+		(at 243.84 243.84 180)
 		(fields_autoplaced yes)
 		(effects
@@
 	)
 	(label "RA11"
-		(at 247.65 256.54 0)
+		(at 247.65 259.08 0)
 		(fields_autoplaced yes)
 		(effects
