File: pcb_top/rev.A/zxevo1010_top.kicad_sch (KiCad schematic)
At the start: 199 parts, among them J1 Conn_02x05_Odd_Even, J2 Conn_02x05_Odd_Even, J3 Conn_02x05_Odd_Even, J4 PJ-320, J6 Conn_02x30_Row_Letter_First, Q1 BSS138, Q2 BC847, U1 ESP-12E, U10 EPM3064ATC100, U11 EP1K30TC144, U12 74AHCT1G125DB, U13 74AHCT1G125DB, U14 74AHCT1G125DB, U15 YMF288-M, U16 YMF288-M, U17 74LVC2G04DB, U18 MAX809LEUR, U2 CY62167EV30LL-45ZXI, U22 74LXC245, U23 MA8201, U25 1117-3.3, U26 1117-2.5, U27 PCM5102A, U28 1117-1.8, U29 EPM3128ATC100, U3 CY62167EV30LL-45ZXI, U30 LP2985-3.3, U31 LP2985-3.3, U32 PCM5102A, U4 Z84C0020FEC, U5 SAM2695, U6 29F040, U7 74LVC1G04DB, U8 74AHCT1G125DB, U9 VS1053b, X1 20 MHz, X2 24 MHz, X3 24 MHz, Y2 14 MHz

Commit message: wip pcb rev.A
Parts:
- added R23: 0, Resistor_SMD:R_1206_3216Metric, symbol Device:R
Connections:
- net +3V3: no longer C89.2, C90.2, U27.17 (XSMT), U27.20 (DVDD), U32.17 (XSMT), U32.20 (DVDD)
- net +3V3A: now also C89.2, C90.2, U27.17 (XSMT), U27.20 (DVDD), U32.17 (XSMT), U32.20 (DVDD)
- net +5V: now also R23.1, R23.2
Other:
- moved on the sheet: C49, C76, C77, C78, C79, C84, C89, C90, C91, C92, C93, C94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

Commit message: wip pcb rev.A
Parts:
- C42, C43: footprint Capacitor_SMD:C_0603_1608Metric_Pad1.08x0.95mm_HandSolder -> Capacitor_SMD:C_0805_2012Metric_Pad1.18x1.45mm_HandSolder
Connections:
- net +3V3: no longer R3.2, R36.2, R4.2, R42.2, R43.2, R44.2, R53.1, R54.1, R55.1, R56.1
- net +5V: now also R3.2, R36.2, R4.2, R42.2, R43.2, R44.2, R53.1, R54.1, R55.1, R56.1
- net TDI_FPGA: now also U10.73 (TDO); no longer J3.9 (Pin_9), R26.2
- net ~{RD}: now also U2.14 (~{BHE})
- net ~{WR}: now also U2.15 (~{BLE})
- net TDI_PSG: now reaches U29.4 (TDI)
- net TDI_PSG: now also U11.4 (TDO)
- net TDO: now reaches U29.73 (TDO)
- net TDO: now also J3.3 (Pin_3)
- net TDOFPGA_TDI3032 renamed TDI
- net TDI: now also J3.9 (Pin_9), R26.2; no longer U11.4 (TDO)
- removed net TDO_3032: J3.3 (Pin_3), U10.73 (TDO)
- no-connect marks 108 -> 106
Other:
- note added: "JTAG"
- note added: "traces passthrought"
- moved on the sheet: J3, R24, R26, R35

Commit message: wip pcb rev.A (almost done)
Parts:
- removed R23: 0, Resistor_SMD:R_1206_3216Metric, symbol Device:R
- removed U7: 74LVC1G04DB, Package_TO_SOT_SMD:SOT-23-5_HandSoldering, symbol 74xGxx:74LVC1G04
- removed Y2: 14 MHz, my:Crystal_SMD_3225-4Pin_3.2x2.5mm_HandSoldering, symbol Device:Crystal_GND24
- added U17: SN74LVC2G04DBVR, Package_TO_SOT_SMD:SOT-23-6_Handsoldering, symbol 74xGxx:74LVC2G04
- added Y1: 14 MHz, Crystal:Crystal_HC49-4H_Vertical, symbol Device:Crystal
- C4: renamed from C26; footprint Capacitor_SMD:C_0805_2012Metric_Pad1.18x1.45mm_HandSolder -> Capacitor_SMD:C_0603_1608Metric_Pad1.08x0.95mm_HandSolder
- JP2: renamed from JP1; Desc Boot -> (none)
- R49: renamed from R35; value 10k -> 6.8k
- U10: renamed from U17; value 74LVC2G04DB -> SN74LVC2G04DBVR
- U11: renamed from U13; value 74AHCT1G125DB -> SN74AHCT1G125DBVR
- U12: renamed from U14; value 74AHCT1G125DB -> SN74AHCT1G125DBVR
- U3: renamed from U10; value EPM3064ATC100 -> EPM3128ATC100; ValueAlt (none) -> EPM3064ATC100
- U7: renamed from U8; value 74AHCT1G125DB -> SN74AHCT1G125DBVR
- U8: renamed from U12; value 74AHCT1G125DB -> SN74AHCT1G125DBVR
- U9: renamed from U22; value 74LXC245 -> SN74LXC8T245PWR
- renumbered C36 to C1, C17 to C10, C18 to C11, C19 to C12, C20 to C13, C22 to C14, C23 to C15, C24 to C16, C25 to C17, C1 to C18, C2 to C19, C37 to C2, C3 to C20, C4 to C21, C9 to C22, C27 to C23, C11 to C24, C12 to C25, C13 to C26, C16 to C27, C84 to C28, C76 to C29, C38 to C3, C77 to C30, C78 to C31, C79 to C32, C91 to C33, C92 to C34, C93 to C35, C94 to C36, C95 to C37, C96 to C38, C90 to C39, C89 to C40, C14 to C41, C99 to C42, C21 to C43, C28 to C44, C29 to C45, C10 to C46, C15 to C47, C31 to C48, C33 to C49, C39 to C5, C35 to C50, C30 to C51, C32 to C52, C34 to C53, C42 to C54, C43 to C55, C44 to C56, C45 to C57, C46 to C58, C47 to C59, C40 to C6, C48 to C60, C59 to C61, C60 to C62, C61 to C63, C62 to C64, C63 to C65, C97 to C66, C98 to C67, C50 to C68, C51 to C69, C41 to C7, C52 to C70, C53 to C71, C54 to C72, C55 to C73, C56 to C74, C57 to C75, C58 to C76, C64 to C77, C65 to C78, C66 to C79, C67 to C80, C68 to C81, C69 to C82, C80 to C83, C81 to C84, C82 to C85, C49 to C89, C7 to C9, C70 to C90, C71 to C91, C72 to C92, C73 to C93, C74 to C94, C75 to C95, C5 to C96, C6 to C97, C83 to C98, C85 to C99, J6 to J1, J1 to J2, J2 to J3, J3 to J5, JP3 to JP1, Q2 to Q1, Q1 to Q2, R12 to R1, R45 to R10, R40 to R11, R16 to R12, R18 to R13, R19 to R14, R53 to R15, R46 to R16, R60 to R17, R58 to R18, R47 to R19, R37 to R2, R54 to R20, R41 to R21, R15 to R22, R17 to R23, R55 to R24, R20 to R25, R21 to R26, R22 to R27, R29 to R28, R30 to R29, R13 to R3, R31 to R30, R32 to R31, R56 to R32, R57 to R33, R3 to R34, R4 to R35, R48 to R36, R24 to R37, R26 to R38, R33 to R39, R42 to R4, R9 to R40, R5 to R41, R6 to R42, R36 to R43, R51 to R44, R49 to R45, R14 to R46, R50 to R47, R52 to R48, R43 to R5, R8 to R50, R10 to R51, R11 to R52, R1 to R53, R7 to R54, R2 to R55, R44 to R6, R38 to R7, R39 to R8, R59 to R9, TP2 to TP1, TP3 to TP2, TP1 to TP3, U32 to U1, U6 to U13, U4 to U14, U2 to U15, U3 to U16, U15 to U18, U16 to U19, U23 to U2, U5 to U20, U29 to U21, U27 to U22, U1 to U23, U25 to U24, U26 to U25, U28 to U26, U31 to U27, U30 to U28, U18 to U4, U11 to U5, U9 to U6
Connections:
- net +5V: now also U17.5 (VCC)
- net CLKOUT: now also U17.1
- net GND: now also U17.2 (GND), U17.3
- net MA_XTALI: now also Y1.2
- net MA_XTALO: now also Y1.1
- net ~{MEMOE}: now also U16.15 (~{BLE})
- net at R44.2, R46.2, R48.2: now also U17.6
Other:
- note added: "trace passthrought"
- moved on the sheet: C1, C10, C11, C12, C13, C14, C15, C16, C17, C18, C19, C2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

Commit message: wip pcb rev.A
Parts:
- added Q3: BSS138, Package_TO_SOT_SMD:SOT-23, symbol Transistor_FET:BSS138
- added R56, R57, R58: 6.8k, Resistor_SMD:R_0603_1608Metric_Pad0.98x0.95mm_HandSolder, symbol Device:R
- C25, C33, C34, C35, C36, C5: value 100n -> 2.2u
- C28: value 47u -> 22u; footprint Capacitor_Tantalum_SMD:CP_EIA-3528-21_Kemet-B_Pad1.50x2.35mm_HandSolder -> Capacitor_Tantalum_SMD:CP_EIA-3216-18_Kemet-A_Pad1.58x1.35mm_HandSolder
- C42: footprint Capacitor_SMD:CP_Elec_5x5.9 -> Capacitor_Tantalum_SMD:CP_EIA-6032-28_Kemet-C_Pad2.25x2.35mm_HandSolder
- Q1: value BC847 -> BSS138; symbol Transistor_BJT:BC847 -> Transistor_FET:BSS138
- R23, R31: value 47k -> 22k
- R25, R30: value 47k -> 18k
- R26, R27: value 10k -> 47k
- R28, R29: value 24k -> 47k
- R32: value 6.8k -> 1k
- R7: value 100 -> 120
- U27, U28: ValueAlt (none) -> LD3985M33R
- X3: value 24 MHz -> 32 MHz
Connections:
- net +3V3: now also Q3.1 (G), R56.2
- net +5V: now also R57.2, R58.2
- net GND: now also U18.16 (~{COM}), U19.16 (~{COM})
- net MIDI_DATA: now also U21.98 (I/O)
- net YMBCO0: now also U21.96 (I/O); no longer U21.100 (I/O)
- net YMDO0: now also U21.97 (I/O); no longer U21.99 (I/O)
- net YMLRO0: now also U21.99 (I/O); no longer U21.96 (I/O)
- net YMWCO0: now also U21.100 (I/O); no longer U21.97 (I/O)
- net ~{YMCS0}: now also U21.1 (I/O); no longer U21.98 (I/O)
- net at TP1.1: now also U21.63 (I/O); no longer U21.1 (I/O)
- net ~{ESP_RST}: now reaches J3.5 (Pin_5)
- net ~{ESP_RST}: now also Q3.3 (D)
- net at U19.22 (~{STBY}): now also R58.1
- net at U18.22 (~{STBY}): now also R57.1
- net RS: no longer names the net of J1.31 (Pin_31)
- net ZXA10: no longer names the net of J1.54 (Pin_54)
- net ZXA11: no longer names the net of J1.55 (Pin_55)
- net ZXA12: no longer names the net of J1.3 (Pin_3)
- net ZXA8: no longer names the net of J1.52 (Pin_52)
- net ZXA9: no longer names the net of J1.53 (Pin_53)
- net ~{RESET}: no longer names the net of U23.1 (~{RST})
- net ~{RESET}: now also Q3.2 (S), R56.1
- net ~{ZXRFSH}: no longer names the net of J1.50 (Pin_50)
- no-connect marks 106 -> 114
Other:
- note added: "Only for VS1053b"
- moved on the sheet: C18, C19, C20, C21, C22, C23, C24, C25, C26, C27, C8, C9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

Commit message: wip pcb rev.A
Parts:
- removed C1, C22, C25, C5: 2.2u, Capacitor_SMD:C_0603_1608Metric_Pad1.08x0.95mm_HandSolder, symbol Device:C
- removed C2, C23, C24, C3: 2.2n, Capacitor_SMD:C_0603_1608Metric_Pad1.08x0.95mm_HandSolder, symbol Device:C
- removed C39, C40: 100n, Capacitor_SMD:C_0603_1608Metric_Pad1.08x0.95mm_HandSolder, symbol Device:C
- removed U1, U22: PCM5102A, Package_SO:TSSOP-20_4.4x6.5mm_P0.65mm, symbol Audio:PCM5102A
- added C100: 100n, Capacitor_SMD:C_0603_1608Metric_Pad1.08x0.95mm_HandSolder, symbol Device:C
- added J6: PJ392, Connector_PinHeader_2.54mm:PinHeader_1x03_P2.54mm_Vertical, symbol Connector_Generic:Conn_01x03
- added R59: 51, Resistor_SMD:R_0603_1608Metric_Pad0.98x0.95mm_HandSolder, symbol Device:R
- added R60: 470, Resistor_SMD:R_0603_1608Metric_Pad0.98x0.95mm_HandSolder, symbol Device:R
- added U1, U22: UDA1334ATS, Package_SO:SSOP-16_4.4x5.2mm_P0.65mm, symbol Audio:UDA1334ATS
- added U29: SN74AHCT1G125DBVR, Package_TO_SOT_SMD:SOT-23-5_HandSoldering, symbol 74xGxx:74LVC1G125
- C33, C34, C35, C36: value 2.2u -> 1u
- C49, C52: value 100n -> 10n
- R1, R50: value 470 -> 6.8k; now not fitted
- R26, R27, R28, R29: value 47k -> 8.2k
- R3, R51: value 470 -> 6.8k
Connections:
- net +3V3A: now also R1.2, R50.2, U1.13 (VDDA), U1.4 (VDDD), U22.13 (VDDA), U22.4 (VDDD)
- net +5V: now also C100.2, R59.2, U29.5 (VCC)
- net DAC_BITCK: now also U1.1 (BCK)
- net DAC_DAT: now also U1.3 (DATAI)
- net DAC_LRCK: now also U1.2 (WS)
- net GND: now also R3.1, R51.1, C100.1, J6.3 (Pin_3), U1.10 (PLL0), U1.11 (SFOR0), U1.15 (VSSA), U1.5 (VSSD), U1.6 (SYSCLK/PLL1), U1.7 (SFOR1), U1.8 (MUTE), U22.10 (PLL0), U22.11 (SFOR0), U22.15 (VSSA), U22.5 (VSSD), U22.6 (SYSCLK/PLL1), U22.7 (SFOR1), U22.8 (MUTE), U29.1, U29.3 (GND)
- net MIDI_DATA: now also U21.99 (I/O), U29.2; no longer U21.98 (I/O)
- net NGS_AOL: now also U1.14 (VOUTL); no longer R1.2
- net NGS_AOR: now also U1.16 (VOUTR); no longer R3.2
- net PSG_BCK: now also U22.1 (BCK)
- net PSG_DIN: now also U21.27 (I/O), U22.3 (DATAI); no longer U21.28 (I/O)
- net PSG_L: now also U22.14 (VOUTL); no longer R50.2
- net PSG_LRCK: now also U21.28 (I/O), U22.2 (WS); no longer U21.27 (I/O)
- net PSG_R: now also U22.16 (VOUTR); no longer R51.2
- net YMLRO0: now also U21.100 (I/O); no longer U21.99 (I/O)
- net YMWCO0: now also U21.98 (I/O); no longer U21.100 (I/O)
- net at C26.2, C27.2: now also U22.12 (Vref(DAC))
- net at C6.2, C7.2: now also U1.12 (Vref(DAC))
- net MIDI_SENSE: now reaches U21.94 (I/O)
- net MIDI_SENSE: now also J6.1 (Pin_1), R60.2
- net at R50.1: now also R51.2, U22.9 (DEEM/CLKOUT)
- net at R1.1: now also R3.2, U1.9 (DEEM/CLKOUT)
- new net: J6.2 (Pin_2), R59.1
- new net: R60.1, U29.4
- no-connect marks 114 -> 113
Other:
- note added: "If MIDI equipment is connected - MIDI_SENSE is always '1' Otherwise MIDI_SENSE == MIDI_DATA"
- note added: "Type A jack connectors (MIDI standard) - https://minimidi.world/"
- moved on the sheet: C26, C27, C6, C68, C69, C7, C70, C71, C72, C73, C74, C75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

Commit message: wip pcb rev.A
Parts:
- removed R1, R3, R50, R51: 6.8k, Resistor_SMD:R_0603_1608Metric_Pad0.98x0.95mm_HandSolder, symbol Device:R
- added C1, C101: 100n, Capacitor_SMD:C_0603_1608Metric_Pad1.08x0.95mm_HandSolder, symbol Device:C
- added C2: 10u, Capacitor_SMD:C_0805_2012Metric_Pad1.18x1.45mm_HandSolder, symbol Device:C
- added C22, C23, C24, C25: 10u, Capacitor_Tantalum_SMD:CP_EIA-3216-18_Kemet-A_Pad1.58x1.35mm_HandSolder, symbol Device:C_Polarized
- added C3, C5: 10n, Capacitor_SMD:C_0603_1608Metric_Pad1.08x0.95mm_HandSolder, symbol Device:C
- added C39, C40: 1u, Capacitor_SMD:C_0603_1608Metric_Pad1.08x0.95mm_HandSolder, symbol Device:C
- added JP3, JP4, JP5: SolderJumper_3_Bridged12, Jumper:SolderJumper-3_P1.3mm_Bridged12_RoundedPad1.0x1.5mm, symbol Jumper:SolderJumper_3_Bridged12
- added R63, R64: 1k, Resistor_SMD:R_0603_1608Metric_Pad0.98x0.95mm_HandSolder, symbol Device:R
- added R65, R66, R67, R68: 8.2k, Resistor_SMD:R_0603_1608Metric_Pad0.98x0.95mm_HandSolder, symbol Device:R
- added U30: UDA1334ATS, Package_SO:SSOP-16_4.4x5.2mm_P0.65mm, symbol Audio:UDA1334ATS
- added U31: SN74LVC2G04DBVR, Package_TO_SOT_SMD:SOT-23-6_Handsoldering, symbol 74xGxx:74LVC2G04
- U21: symbol my:EPM3128ATC100 -> my:EPM3064ATC100
Connections:
- net +3V3A: now also U22.11 (SFOR0), C101.2, C39.2, C40.2, JP3.3 (B), JP4.3 (B), JP5.3 (B), U30.11 (SFOR0), U30.13 (VDDA), U30.4 (VDDD), U31.5 (VCC)
- net GND: now also C1.1, C101.1, C2.1, C3.1, C39.1, C40.1, C5.1, JP3.1 (A), JP4.1 (A), JP5.1 (A), U30.10 (PLL0), U30.15 (VSSA), U30.5 (VSSD), U30.6 (SYSCLK/PLL1), U30.7 (SFOR1), U30.8 (MUTE), U31.2 (GND); no longer U22.11 (SFOR0)
- net MIDI_DATA: now also U21.96 (I/O); no longer U21.99 (I/O)
- net MIXER_L: now also R65.1, R66.1
- net MIXER_R: now also R67.1, R68.1
- net YMA0: now also U21.19 (I/O); no longer U21.6 (I/O)
- net YMA1: now also U21.20 (I/O); no longer U21.7 (I/O)
- net YMBCO0: now also U22.1 (BCK); no longer U21.96 (I/O)
- net YMBCO1: now also U30.1 (BCK); no longer U21.9 (I/O)
- net YMCK: now also U21.21 (I/O); no longer U21.14 (I/O)
- net YMD0: now also U21.98 (I/O); no longer U21.16 (I/O)
- net YMD1: now also U21.99 (I/O); no longer U21.17 (I/O)
- net YMD2: now also U21.100 (I/O); no longer U21.19 (I/O)
- net YMD3: now also U21.97 (I/O); no longer U21.20 (I/O)
- net YMD4: now also U21.6 (I/O); no longer U21.21 (I/O)
- net YMD5: now also U21.8 (I/O); no longer U21.22 (I/O)
- net YMD6: now also U21.9 (I/O); no longer U21.23 (I/O)
- net YMD7: now also U21.10 (I/O); no longer U21.24 (I/O)
- net YMDO0: now also U22.3 (DATAI); no longer U21.97 (I/O)
- net YMDO1: now also U30.3 (DATAI); no longer U21.10 (I/O)
- net YMLRO0: now also U22.2 (WS); no longer U21.100 (I/O)
- net YMLRO1: now also U30.2 (WS); no longer U21.13 (I/O)
- net ZXA0: now also U21.60 (I/O); no longer U21.57 (I/O)
- net ZXA1: now also U21.58 (I/O); no longer U21.56 (I/O)
- net ZXA13: now also U21.61 (I/O); no longer U21.58 (I/O)
- net ZXA14: now also U21.63 (I/O); no longer U21.60 (I/O)
- net ZXA15: now also U21.64 (I/O); no longer U21.61 (I/O)
- net ZXA2: now also U21.57 (I/O); no longer U21.55 (I/O)
- net ZXA3: now also U21.56 (I/O); no longer U21.54 (I/O)
- net ZXA4: now also U21.44 (I/O); no longer U21.45 (I/O)
- net ZXA5: now also U21.45 (I/O); no longer U21.46 (I/O)
- net ZXA6: now also U21.46 (I/O); no longer U21.47 (I/O)
- net ZXA7: now also U21.47 (I/O); no longer U21.48 (I/O)
- net ZXD0: now also U21.31 (I/O); no longer U21.32 (I/O)
- net ZXD1: now also U21.32 (I/O); no longer U21.35 (I/O)
- net ZXD2: now also U21.35 (I/O); no longer U21.36 (I/O)
- net ZXD3: now also U21.40 (I/O); no longer U21.41 (I/O)
- net ZXD4: now also U21.41 (I/O); no longer U21.42 (I/O)
- net ZXD5: now also U21.37 (I/O); no longer U21.40 (I/O)
- net ZXD6: now also U21.36 (I/O); no longer U21.37 (I/O)
- net ZXD7: now also U21.30 (I/O); no longer U21.31 (I/O)
- net ~{YMCS0}: now also U21.13 (I/O); no longer U21.1 (I/O)
- net ~{YMCS1}: now also U21.14 (I/O); no longer U21.8 (I/O)
- net ~{YMRD}: now also U21.17 (I/O); no longer U21.5 (I/O)
- net ~{YMRST}: now also U21.12 (I/O); no longer U21.25 (I/O)
- net ~{YMWR}: now also U21.16 (I/O); no longer U21.2 (I/O)
- net ~{ZXM1}: now also U21.42 (I/O); no longer U21.44 (I/O)
- net ~{ZXMREQ}: now also U21.54 (I/O); no longer U21.52 (I/O)
- net ~{ZXRD}: now also U21.52 (I/O); no longer U21.50 (I/O)
- net ~{ZXWR}: now also U21.48 (I/O); no longer U21.49 (I/O)
- net at U1.9 (DEEM/CLKOUT): now also JP3.2 (C)
- net at TP3.1: now also U21.29 (I/O); no longer U21.30 (I/O)
- net at TP1.1: now also U21.67 (I/O); no longer U21.63 (I/O)
- net at U22.9 (DEEM/CLKOUT): now also JP4.2 (C)
- removed net PSG_BCK: U21.29 (I/O), U22.1 (BCK)
- net PSG_DIN: no longer names the net of U21.27 (I/O)
- net PSG_DIN: no longer U22.3 (DATAI)
- net PSG_L renamed SD_L
- net SD_L: now also C3.2, R63.1; no longer U22.14 (VOUTL)
- net PSG_LRCK: no longer names the net of U21.28 (I/O)
- net PSG_LRCK: no longer U22.2 (WS)
- net PSG_R renamed SD_R
- net SD_R: now also C5.2, R64.1; no longer U22.16 (VOUTR)
- net YMWCO0: no longer names the net of U18.25 (WCO)
- net YMWCO0: no longer U21.98 (I/O)
- net YMWCO1: no longer names the net of U19.25 (WCO)
- net YMWCO1: no longer U21.12 (I/O)
- new net: C23.2, R66.2
- new net: C25.2, R68.2
- new net: C1.2, C2.2, U30.12 (Vref(DAC))
- new net: C24.2, R67.2
- new net: JP5.2 (C), U30.9 (DEEM/CLKOUT)
- new net: R63.2, U31.6
- new net: R64.2, U31.4
- new net: C22.2, R65.2
- new net SD_L_1BIT: U21.25 (I/O), U31.1
- new net SD_R_1BIT: U21.23 (I/O), U31.3
- new net YMF_L0: C23.1, U22.14 (VOUTL)
- new net YMF_L1: C22.1, U30.14 (VOUTL)
- new net YMF_R0: C25.1, U22.16 (VOUTR)
- new net YMF_R1: C24.1, U30.16 (VOUTR)
- no-connect marks 113 -> 110
Other:
- moved on the sheet: C10, C11, C12, C13, C14, C15, C16, C17, C18, C19, C20, C21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

Commit message: pcb rev.A final versions
Parts:
- C49, C52: now not fitted
- J4: value PJ-320 -> PJ-322; footprint my:PJ-320A_D -> my:PJ-322
- U27, U28: value LP2985-3.3 -> TPS7A2033PDBVR; ValueAlt LD3985M33R -> NCP114ASN330T1G, LP2985-3.3, LD3985M33R
- U4: value MAX809LEUR -> MAX809MEUR; ValueAlt (none) -> STM809MWX6F, ADM809MART, TCM809MENB713, TPV809M, CAT809MTBI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
Changed lines of the file:
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@@
 			)
 		)
-		(property "Value" "PJ-320"
+		(property "Value" "PJ-322"
 			(at 461.137 169.9514 0)
 			(effects
@@
 			)
 		)
-		(property "Footprint" "my:PJ-320A_D"
+		(property "Footprint" "my:PJ-322"
 			(at 462.28 175.26 0)
 			(effects
@@
 			)
 		)
-		(property "Value" "LP2985-3.3"
+		(property "Value" "TPS7A2033PDBVR"
 			(at 149.86 504.444 0)
 			(effects
@@
 			)
 		)
-		(property "ValueAlt" "LD3985M33R"
+		(property "ValueAlt" "NCP114ASN330T1G, LP2985-3.3, LD3985M33R"
 			(at 149.606 506.222 0)
 			(effects
 				(font
-					(size 1 1)
+					(size 0.7 0.7)
 				)
 			)
@@
 		(in_bom yes)
 		(on_board yes)
-		(dnp no)
+		(dnp yes)
 		(property "Reference" "C49"
 			(at 165.735 513.08 0)
@@
 		(in_bom yes)
 		(on_board yes)
-		(dnp no)
+		(dnp yes)
 		(property "Reference" "C52"
 			(at 213.995 513.08 0)
@@
 			)
 		)
-		(property "Value" "LP2985-3.3"
+		(property "Value" "TPS7A2033PDBVR"
 			(at 198.12 504.444 0)
 			(effects
@@
 			)
 		)
-		(property "ValueAlt" "LD3985M33R"
+		(property "ValueAlt" "NCP114ASN330T1G, LP2985-3.3, LD3985M33R"
 			(at 197.866 506.222 0)
 			(effects
 				(font
-					(size 1 1)
+					(size 0.7 0.7)
 				)
 			)
@@
 		(dnp no)
 		(property "Reference" "U4"
-			(at 254.254 98.044 0)
+			(at 254.254 97.282 0)
 			(effects
 				(font
@@
 			)
 		)
-		(property "Value" "MAX809LEUR"
-			(at 254.254 99.822 0)
+		(property "Value" "MAX809MEUR"
+			(at 254.254 99.06 0)
 			(effects
 				(font
@@
 			)
 		)
+		(property "ValueAlt" "STM809MWX6F, ADM809MART, TCM809MENB713, TPV809M, CAT809MTBI, CBM809MST3, LM809M3-4.38, APX809S-44SA, SGM809-MXN3"
+			(at 269.494 100.584 0)
+			(effects
+				(font
+					(size 0.3 0.3)
+				)
+			)
+		)
