File: pcb_covers/rev.A/zxevo1010_covers.kicad_pcb (KiCad board)
At the start: 2 copper layers, 134.6 x 63 mm, 3 parts

Commit message: wip pcb rev.A
Other:
- outline, holes or cut-outs redrawn

Commit message: wip pcb rev.A
Parts:
- removed the G*** at (86.3, 114.5)
- removed the G*** at (202.7, 115.4)
- added G***: LOGO, LOGO, F.Cu at (85.7, 115.0)
- added G***: LOGO, LOGO, F.Cu at (201.9, 115.0)

Commit message: wip pcb rev.A
Changed lines of the file:
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@@
+		(layer "F.SilkS")
+	)
+	(gr_poly
+		(pts
+			(xy 130.4325 103.1) (xy 132.4325 103.1) (xy 131.4325 106.1) (xy 129.4325 106.1)
+		)
+		(stroke
+			(width 0.15)
+			(type solid)
+		)
+		(fill solid)
+		(layer "F.SilkS")
+	)
+	(gr_poly
+		(pts
+			(xy 157.575 103.112) (xy 159.575 103.112) (xy 158.575 106.112) (xy 156.575 106.112)
+		)
+		(stroke
+			(width 0.15)
+			(type solid)
+		)
+		(fill solid)
 		(layer "F.SilkS")
 	)
@@
 	(gr_poly
 		(pts
+			(xy 161.925 103.112) (xy 163.925 103.112) (xy 162.925 106.112) (xy 160.925 106.112)
+		)
+		(stroke
+			(width 0.15)
+			(type solid)
+		)
+		(fill solid)
+		(layer "F.SilkS")
+	)
+	(gr_poly
+		(pts
 			(xy 117.375 103.1) (xy 119.375 103.1) (xy 118.375 106.1) (xy 116.375 106.1)
 		)
@@
 		)
 		(stroke
-			(width 0.15)
-			(type solid)
-		)
-		(fill solid)
-		(layer "F.SilkS")
-	)
-	(gr_poly
-		(pts
-			(xy 161.925 103.112) (xy 163.925 103.112) (xy 162.925 106.112) (xy 160.925 106.112)
-		)
-		(stroke

Commit message: wip pcb rev.A
Other:
- outline, holes or cut-outs redrawn
- board text added: "MIDI OUT"

Commit message: pcb rev.A final versions
Other:
- outline, holes or cut-outs redrawn
